File: hardware/kicad/C_rf/dogrudan_sdr_C.kicad_pcb (KiCad board)
At the start: 2 copper layers, 350 x 235 mm, 445 parts, among them J1 SMA anten 1, J2 SMA anten 2, J3 SMA anten 3, J4 SMA anten 4, J80 A kartina, J81 A kartina #2, J82 RX1 -> A, J83 RX2 -> A, J84 RX3 -> A, J85 RX4 -> A, J86 TX1 <- A, J87 TX2 <- A, J88 TX3 <- A, J89 TX4 <- A, J90 D kartina, K11 G6KU-2F-Y, K12 G6KU-2F-Y, K13 G6KU-2F-Y, K14 G6KU-2F-Y, K15 G6KU-2F-Y, K16 G6KU-2F-Y, K17 G6KU-2F-Y, K21 G6KU-2F-Y, K22 G6KU-2F-Y, K23 G6KU-2F-Y, K24 G6KU-2F-Y, K25 G6KU-2F-Y, K26 G6KU-2F-Y, K27 G6KU-2F-Y, K31 G6KU-2F-Y, K32 G6KU-2F-Y, K33 G6KU-2F-Y, K34 G6KU-2F-Y, K35 G6KU-2F-Y, K36 G6KU-2F-Y, K37 G6KU-2F-Y, K41 G6KU-2F-Y, K42 G6KU-2F-Y, K43 G6KU-2F-Y, K44 G6KU-2F-Y, K45 G6KU-2F-Y, K46 G6KU-2F-Y, K47 G6KU-2F-Y, U40 PE4312C-Z, U41 PE4312C-Z, U42 PE4312C-Z, U43 PE4312C-Z, U60 74HC595D, U61 74HC595D, U62 74HC595D, U63 74HC595D, U64 74HC595D, U65 74HC595D, U66 74HC595D, U70 DRV8833PWPR, U71 DRV8833PWPR, U72 DRV8833PWPR, U73 DRV8833PWPR, U74 DRV8833PWPR, U75 DRV8833PWPR, U76 DRV8833PWPR, U77 DRV8833PWPR, U78 DRV8833PWPR, U79 DRV8833PWPR, U80 DRV8833PWPR, U81 DRV8833PWPR, U82 DRV8833PWPR, U83 DRV8833PWPR

Commit message: Update the hardware tools and add the gateware
This commit makes the public tree equal to the development tree. The
public tree was behind. It did not have the verification tools, the
build chain, or the FPGA source.

The hardware/kicad directory now has the full tool chain. This
includes yap.sh, which runs the steps in the correct order, and the
tools that check the boards.

The gateware directory is new. It has the Verilog source for the
Lattice ECP5, the test benches, and the synthesis script. The
gateware does the four-channel receive chain, the transmit chain, the
packet interface, and the control interface.

The internal Turkish documents stay in the development tree. The
documentation in this repository is English. The comments in the
source code stay in Turkish.
Parts:
- moved D115 313.4 mm to (17.0, 190.0), turned to 90 degrees
- moved D105 296.7 mm to (17.0, 80.0), turned to 90 degrees
- moved R107 218.9 mm to (31.0, 25.0), turned to 90 degrees
- moved R116 218.9 mm to (31.0, 80.0), turned to 90 degrees
- moved R125 218.9 mm to (31.0, 135.0), turned to 90 degrees
- moved R134 218.9 mm to (31.0, 190.0), turned to 90 degrees
- moved D114 197.4 mm to (122.2, 120.2)
- moved D106 193.2 mm to (122.2, 46.9)
- moved D110 146.7 mm to (17.0, 135.0), turned to 90 degrees
- moved E100 145.9 mm to (9.30, 28.8), turned to 90 degrees
- moved D124 142.0 mm to (173.9, 139.8)
- moved D133 140.9 mm to (173.9, 194.8)
- moved D123 138.7 mm to (173.0, 136.2)
- moved D132 137.1 mm to (173.0, 191.2)
- moved D101 48.8 mm to (109.7, 28.4)
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Routing:
- net RX1_B1_IN: track 0.00 -> 7.88 mm
- net RX2_B1_IN: track 0.00 -> 7.88 mm
- net RX4_B1_IN: track 0.00 -> 7.88 mm
- net RX3_B1_IN: track 0.00 -> 7.88 mm

Commit message: Connect the pads that had no net
A symbol pin number must agree with the footprint pad number. If the
numbers do not agree, the net goes nowhere. The netlist removes it
and gives no message. ERC examines the schematic and sees a wire. DRC
does not count an unconnected pad as a violation. All three boards
showed zero ERC violations while 31 pads had no net.

Two of these faults stopped a board.

The footprint of the Ethernet PHY was for a different part. The
project used QFN-48 6x6 mm with 0.4 mm pitch. The RTL8211F(I)-CG is
WQFN-40-EP 5x5 mm. You cannot solder the part to that pad pattern.

The 25 MHz crystal had a 2-pin symbol on a 4-pad footprint. On a 3225
crystal the terminals are the diagonal pads 1 and 3. Pads 2 and 4 are
the metal can. XO went to pad 2. There was no crystal between XI and
XO, and thus neither PHY could make a clock.

The paddle of the AD9251 was pin 0 in the symbol and pad 65 in the
footprint. The paddle of the PE4312 was Pad against pad 21. The gas
discharge tubes had one electrode unconnected, because
Device:GDT_2Pin uses pins 1 and 3 but the varistor footprint uses
pads 1 and 2. A local footprint with pads 1 and 3 corrects this.

ped_denetim.py finds these faults on the board. yap.sh runs it before
the DSN export. The chain stops if a pad has no net.

The DSN export also changed. It declared In1 and In4 as power layers
but did not export the copper on them. The router thus believed that
the two ground planes were empty. It routed the 289 pins of GND as
traces on the signal layers. The planes now go out as conduction
areas.
Parts:
- added C651: 100nF, C_0603_1608Metric, F.Cu at (245.6, 212.6)
- added C654: 100nF, C_0603_1608Metric, F.Cu at (305.6, 212.6)
- added C83: 10uF, C_1206_3216Metric, F.Cu at (14.3, 217.8)
- added C84: 100nF, C_0603_1608Metric, F.Cu at (10.0, 217.4)
- added R649: 0R, R_0603_1608Metric, F.Cu at (243.5, 215.2)
- added R650: 0R, R_0603_1608Metric, F.Cu at (243.5, 218.4)
- added R652: 0R, R_0603_1608Metric, F.Cu at (303.5, 214.3)
- added R653: 0R, R_0603_1608Metric, F.Cu at (303.5, 216.4)
- added U84: DRV8833PWPR, HTSSOP-16-1EP_4.4x5mm_P0.65mm_EP3.4x5mm_Mask2.46x2.31mm_ThermalVias, F.Cu at (240.0, 210.0)
- added U85: DRV8833PWPR, HTSSOP-16-1EP_4.4x5mm_P0.65mm_EP3.4x5mm_Mask2.46x2.31mm_ThermalVias, F.Cu at (300.0, 210.0)
- added U90: TPS62130, VQFN-16-1EP_3x3mm_P0.5mm_EP1.68x1.68mm, F.Cu at (10.0, 214.0)
- E100, E109, E118, E127: footprint RV_Disc_D12mm_W3.9mm_P7.5mm -> GDT_Disc_D12mm_W3.9mm_P7.5mm
- H1: value MountingHole_3.2mm_M3 -> MountingHole_3.2mm_M3_Pad; footprint MountingHole_3.2mm_M3 -> MountingHole_3.2mm_M3_Pad
- moved QT1 282.2 mm to (27.0, 12.0)
- moved QT2 282.2 mm to (27.0, 67.0)
- moved QT3 282.2 mm to (27.0, 122.0)
- moved QT4 282.2 mm to (27.0, 177.0)
- moved D102 281.5 mm to (30.5, 17.7)
- moved D111 281.5 mm to (30.5, 72.7)
- moved D120 281.5 mm to (30.5, 127.7)
- moved D129 281.5 mm to (30.5, 182.7)
- moved KT1 281.0 mm to (27.0, 25.0), turned to 90 degrees
- moved KT2 281.0 mm to (27.0, 80.0), turned to 90 degrees
- moved KT3 281.0 mm to (27.0, 135.0), turned to 90 degrees
- moved KT4 281.0 mm to (27.0, 190.0), turned to 90 degrees
- moved C618 263.1 mm to (305.6, 47.6)
- moved R616 261.8 mm to (303.5, 50.1)
- moved C602 261.6 mm to (295.2, 40.8)
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Connections:
- net FB_U80 renamed FB_U90
- U40 pad 21: (no net) -> GND
- U41 pad 21: (no net) -> GND
- U42 pad 21: (no net) -> GND
- U43 pad 21: (no net) -> GND
- U73 pad 10: Q15 -> GND
- U73 pad 5: K21_R -> unconnected-(U73-BOUT2-Pad5)
- U73 pad 7: K21_S -> unconnected-(U73-BOUT1-Pad7)
- U73 pad 9: Q14 -> GND
- U74 pad 10: Q19 -> Q17
- U74 pad 15: Q17 -> Q15
- U74 pad 16: Q16 -> Q14
- U74 pad 2: K22_S -> K21_S
- U74 pad 4: K22_R -> K21_R
- U74 pad 5: K23_R -> K22_R
- U74 pad 7: K23_S -> K22_S
- U74 pad 9: Q18 -> Q16
- U75 pad 10: Q23 -> Q21
- U75 pad 15: Q21 -> Q19
- U75 pad 16: Q20 -> Q18
- U75 pad 2: K24_S -> K23_S
- U75 pad 4: K24_R -> K23_R
- U75 pad 5: K25_R -> K24_R
- U75 pad 7: K25_S -> K24_S
- U75 pad 9: Q22 -> Q20
- U76 pad 10: Q27 -> Q25
- U76 pad 15: Q25 -> Q23
- U76 pad 16: Q24 -> Q22
- U76 pad 2: K26_S -> K25_S
- U76 pad 4: K26_R -> K25_R
- U76 pad 5: K27_R -> K26_R
- U76 pad 7: K27_S -> K26_S
- U76 pad 9: Q26 -> Q24
- U77 pad 10: Q31 -> GND
- U77 pad 15: Q29 -> Q27
- U77 pad 16: Q28 -> Q26
- U77 pad 2: K31_S -> K27_S
- U77 pad 4: K31_R -> K27_R
- U77 pad 5: K32_R -> unconnected-(U77-BOUT2-Pad5)
- U77 pad 7: K32_S -> unconnected-(U77-BOUT1-Pad7)
- U77 pad 9: Q30 -> GND
- U78 pad 10: Q35 -> Q31
- U78 pad 15: Q33 -> Q29
- U78 pad 16: Q32 -> Q28
- U78 pad 2: K33_S -> K31_S
- U78 pad 4: K33_R -> K31_R
- U78 pad 5: K34_R -> K32_R
- U78 pad 7: K34_S -> K32_S
- U78 pad 9: Q34 -> Q30
- U79 pad 10: Q39 -> Q35
- U79 pad 15: Q37 -> Q33
- U79 pad 16: Q36 -> Q32
- U79 pad 2: K35_S -> K33_S
- U79 pad 4: K35_R -> K33_R
- U79 pad 5: K36_R -> K34_R
- U79 pad 7: K36_S -> K34_S
- U79 pad 9: Q38 -> Q34
- U80 pad 1: Net-(L80-Pad1) -> +3V3
- U80 pad 10: VIN_PROT -> Q39
- U80 pad 12: VIN_PROT -> +5V
- U80 pad 13: VIN_PROT -> GND
- U80 pad 15: Q41 -> Q37
- U80 pad 16: Q40 -> Q36
- U80 pad 2: Net-(L80-Pad1) -> K35_S
- U80 pad 4: unconnected-(U80-PG-Pad4) -> K35_R
- U80 pad 5: K41_R -> K36_R
- U80 pad 7: K41_S -> K36_S
- U80 pad 9: unconnected-(U80-SS/TR-Pad9) -> Q38
- U81 pad 10: Q47 -> GND
- U81 pad 15: Q45 -> Q41
- U81 pad 16: Q44 -> Q40
- U81 pad 2: K42_S -> K37_S
- U81 pad 4: K42_R -> K37_R
- U81 pad 5: K43_R -> unconnected-(U81-BOUT2-Pad5)
- U81 pad 7: K43_S -> unconnected-(U81-BOUT1-Pad7)
- U81 pad 9: Q46 -> GND
- U82 pad 10: Q51 -> Q45
- U82 pad 15: Q49 -> Q43
- U82 pad 16: Q48 -> Q42
- U82 pad 2: K44_S -> K41_S
- U82 pad 4: K44_R -> K41_R
- U82 pad 5: K45_R -> K42_R
- U82 pad 7: K45_S -> K42_S
- U82 pad 9: Q50 -> Q44
- U83 pad 10: Q55 -> Q49
- U83 pad 15: Q53 -> Q47
- U83 pad 16: Q52 -> Q46
- U83 pad 2: K46_S -> K43_S
- U83 pad 4: K46_R -> K43_R
- U83 pad 5: K47_R -> K44_R
- U83 pad 7: K47_S -> K44_S
- U83 pad 9: Q54 -> Q48
Routing:
- net RX4_B1_IN: track 7.88 -> 12.7 mm
- net RX3_B1_IN: track 7.88 -> 12.7 mm
- net RX2_B1_IN: track 7.88 -> 12.7 mm
- net RX1_B1_IN: track 7.88 -> 12.7 mm
Other:
- board text added: "​15/10m"
- board text added: "​20/17m"
- board text added: "​40/30m"
- board text added: "​80/60m"
- board text added: "​BYPASS"
- board text added: "​CHASSIS GND - THIS HOLE ONLY"
- board text removed: "​12/10m"
- board text removed: "​17/15m"
- board text removed: "​30/20m"
- board text removed: "​40m"
- board text removed: "​80m"

Commit message: Correct the schematic faults that ERC cannot find
An agent examined the three schematics against the datasheets. ERC
reported zero violations before and after this work. None of these
faults are visible to ERC.

The comparator for the external 10 MHz reference was in shutdown. The
SHDN pin of the TLV3501 went to +3V3. Sixteen DRV8833 devices had VCP
and VINT unconnected. Without the charge pump none of the 28 filter
relays can latch. Seven regulators had no decoupling capacitor within
18 mm to 94 mm. On board D the nearest +12V capacitor to an LM358 was
227 mm away on a 275 mm board.

The PE4312 devices had no series 10k resistor on pin 3. The datasheet
makes this necessary for the attenuation accuracy. Their exposed pad
was 2.6 mm against 2.15 mm. The BOM did not give the load capacitance
of the crystal. This work added 60 parts and changed 4 footprints.

The worst fault was in the tool chain. lib/gen_symbols.py still made
the old pin numbers. The five corrections went into the symbol
library by hand and not into its generator. A new library would have
removed all of them.

The thermal vias are now a decision from the measured clearance and
the dissipation. This work removed them from the PE4312, the RTL8211F
and the ADCLK846. They stay on the DRV8833 and on the LM5164, which
is a 1 W buck converter.

Two checks are new. sema_denetim compares the pin names with the
nets. netlist_denetim locks 22 pin-to-net expectations from the
datasheets and does not need a board.

The boards were built again with these corrections. The chain now
adds the test points: 10 on board A, 7 on board C and 15 on board D.
Each board has 3 fiducials. Every pad has a net.
Parts:
- removed C406, C414, C415, C422, C423, C430, C431: 100nF, C_0402_1005Metric
- removed C612, C618, C627, C633, C642, C648: 100nF, C_0603_1608Metric
- removed R408, R416, R417, R425, R426: 10k, R_0603_1608Metric
- removed R610, R611, R614, R616, R619, R620, R625, R626, R629, R631, R634, R635, R640, R641, R644, R646, R649, R650: 0R, R_0603_1608Metric
- added C408: 100nF, C_0402_1005Metric, F.Cu at (80.7, 229.5)
- added C416: 100nF, C_0402_1005Metric, F.Cu at (126.7, 229.5)
- added C417: 100nF, C_0402_1005Metric, F.Cu at (172.7, 229.5)
- added C425: 100nF, C_0402_1005Metric, F.Cu at (218.7, 229.5)
- added C426: 100nF, C_0402_1005Metric, F.Cu at (264.7, 229.5)
- added C434: 100nF, C_0402_1005Metric, F.Cu at (310.7, 229.5)
- added C435: 100nF, C_0402_1005Metric, F.Cu at (75.2, 40.8)
- added C610: 2.2uF, C_0603_1608Metric, F.Cu at (89.4, 46.4)
- added C611: 100nF, C_0603_1608Metric, F.Cu at (85.6, 47.6)
- added C614: 10nF, C_0603_1608Metric, F.Cu at (163.5, 50.2)
- added C616: 100nF, C_0603_1608Metric, F.Cu at (165.6, 47.6)
- added C619: 10nF, C_0603_1608Metric, F.Cu at (243.5, 50.2)
- added C620: 2.2uF, C_0603_1608Metric, F.Cu at (247.1, 44.0)
- added C625: 2.2uF, C_0603_1608Metric, F.Cu at (307.1, 44.0)
- added C626: 100nF, C_0603_1608Metric, F.Cu at (305.6, 47.6)
- added C629: 10nF, C_0603_1608Metric, F.Cu at (89.4, 99.7)
- added C631: 100nF, C_0603_1608Metric, F.Cu at (85.6, 102.7)
- added C634: 10nF, C_0603_1608Metric, F.Cu at (163.5, 111.3)
- added C635: 2.2uF, C_0603_1608Metric, F.Cu at (167.1, 99.1)
- added C640: 2.2uF, C_0603_1608Metric, F.Cu at (247.1, 99.1)
- added C641: 100nF, C_0603_1608Metric, F.Cu at (245.6, 102.7)
- added C644: 10nF, C_0603_1608Metric, F.Cu at (303.5, 111.3)
- added C646: 100nF, C_0603_1608Metric, F.Cu at (305.6, 102.7)
- added C649: 10nF, C_0603_1608Metric, F.Cu at (83.5, 166.3)
- added C650: 2.2uF, C_0603_1608Metric, F.Cu at (89.4, 156.4)
- added C655: 2.2uF, C_0603_1608Metric, F.Cu at (169.4, 156.4)
- added C656: 100nF, C_0603_1608Metric, F.Cu at (165.6, 157.6)
- added C659: 10nF, C_0603_1608Metric, F.Cu at (243.5, 160.2)
- added C660: 2.2uF, C_0603_1608Metric, F.Cu at (249.4, 156.4)
- added C661: 100nF, C_0603_1608Metric, F.Cu at (245.6, 157.6)
- added C664: 10nF, C_0603_1608Metric, F.Cu at (303.5, 160.2)
- added C665: 2.2uF, C_0603_1608Metric, F.Cu at (309.4, 156.4)
- added C666: 100nF, C_0603_1608Metric, F.Cu at (305.6, 157.6)
- added C669: 10nF, C_0603_1608Metric, F.Cu at (89.4, 209.7)
- added C670: 2.2uF, C_0603_1608Metric, F.Cu at (89.4, 212.8)
- added C671: 100nF, C_0603_1608Metric, F.Cu at (85.6, 212.6)
- added C674: 10nF, C_0603_1608Metric, F.Cu at (161.8, 216.4)
- added C675: 2.2uF, C_0603_1608Metric, F.Cu at (167.1, 209.1)
- added C676: 100nF, C_0603_1608Metric, F.Cu at (165.6, 212.3)
- added C679: 10nF, C_0603_1608Metric, F.Cu at (243.5, 221.2)
- added C680: 2.2uF, C_0603_1608Metric, F.Cu at (247.1, 209.1)
- added C681: 100nF, C_0603_1608Metric, F.Cu at (245.6, 212.6)
- added C684: 10nF, C_0603_1608Metric, F.Cu at (301.8, 216.4)
- added C685: 2.2uF, C_0603_1608Metric, F.Cu at (307.1, 209.1)
- added C686: 100nF, C_0603_1608Metric, F.Cu at (305.6, 212.3)
- added FID1: ​FID, Fiducial_1mm_Mask2mm, F.Cu at (8.26, 12.6)
- added FID2: ​FID, Fiducial_1mm_Mask2mm, F.Cu at (346.4, 12.6)
- added FID3: ​FID, Fiducial_1mm_Mask2mm, F.Cu at (3.64, 222.4)
- added R406: 10k, R_0603_1608Metric, F.Cu at (204.8, 127.9)
- added R414: 10k, R_0603_1608Metric, F.Cu at (194.8, 167.2)
- added R415: 10k, R_0603_1608Metric, F.Cu at (196.0, 162.1)
- added R422: 10k, R_0603_1608Metric, F.Cu at (199.1, 167.9)
- added R423: 10k, R_0603_1608Metric, F.Cu at (196.9, 180.1)
- added R430: 10k, R_0603_1608Metric, F.Cu at (196.4, 211.0)
- added R431: 10k, R_0603_1608Metric, F.Cu at (195.5, 198.4)
- added R432: 10k, R_0603_1608Metric, F.Cu at (195.2, 201.4)
- added R433: 10k, R_0603_1608Metric, F.Cu at (199.8, 199.8)
- added R612: 0R, R_0603_1608Metric, F.Cu at (163.5, 56.3)
- added R618: 0R, R_0603_1608Metric, F.Cu at (243.5, 53.4)
- added R627: 0R, R_0603_1608Metric, F.Cu at (83.5, 108.4)
- added R633: 0R, R_0603_1608Metric, F.Cu at (163.5, 108.3)
- added R642: 0R, R_0603_1608Metric, F.Cu at (303.5, 105.2)
- added R648: 0R, R_0603_1608Metric, F.Cu at (83.5, 160.2)
- added R657: 0R, R_0603_1608Metric, F.Cu at (243.5, 163.2)
- added R658: 0R, R_0603_1608Metric, F.Cu at (243.5, 166.3)
- added R662: 0R, R_0603_1608Metric, F.Cu at (303.5, 163.2)
- added R663: 0R, R_0603_1608Metric, F.Cu at (303.5, 166.3)
- added R667: 0R, R_0603_1608Metric, F.Cu at (83.5, 218.3)
- added R668: 0R, R_0603_1608Metric, F.Cu at (83.5, 215.2)
- added R672: 0R, R_0603_1608Metric, F.Cu at (165.2, 216.4)
- added R673: 0R, R_0603_1608Metric, F.Cu at (163.3, 214.0)
- added R677: 0R, R_0603_1608Metric, F.Cu at (243.5, 215.2)
- added R678: 0R, R_0603_1608Metric, F.Cu at (243.5, 218.3)
- added R682: 0R, R_0603_1608Metric, F.Cu at (305.2, 216.4)
- added R683: 0R, R_0603_1608Metric, F.Cu at (303.3, 214.0)
- added TP1: ​+5V, TestPoint_Pad_D1.5mm, F.Cu at (309.2, 103.4)
- added TP2: ​+3V3, TestPoint_Pad_D1.5mm, F.Cu at (292.7, 100.0)
- added TP3: ​VIN_PROT, TestPoint_Pad_D1.5mm, F.Cu at (42.2, 232.3)
- added TP4: ​RX1_OUT, TestPoint_Pad_D1.5mm, F.Cu at (208.1, 119.5)
- added TP5: ​RX2_OUT, TestPoint_Pad_D1.5mm, F.Cu at (199.4, 153.8)
- added TP6: ​RX3_OUT, TestPoint_Pad_D1.5mm, F.Cu at (201.0, 182.8)
- added TP7: ​RX4_OUT, TestPoint_Pad_D1.5mm, F.Cu at (201.1, 187.9)
- C609, C624, C639, C654: value 100nF -> 10nF
- C615, C630, C645: value 100nF -> 2.2uF
- U40, U41, U42, U43: footprint QFN-20-1EP_4x4mm_P0.5mm_EP2.6x2.6mm_ThermalVias -> TQFN-20-1EP_4x4mm_P0.5mm_EP2.1x2.1mm
- moved C645 248.8 mm to (307.1, 99.1)
- moved R643 244.6 mm to (303.5, 108.3)
- moved R400 220.1 mm to (69.2, 227.0)
- moved R628 220.0 mm to (83.5, 105.2)
- moved C630 216.2 mm to (89.4, 102.8)
- moved C621 169.2 mm to (245.6, 47.6)
- moved C651 169.2 mm to (85.6, 157.6)
- moved R418 165.0 mm to (76.6, 230.1)
- moved R409 157.6 mm to (82.8, 223.1)
- moved R427 156.3 mm to (82.8, 226.2)
- moved R623 151.6 mm to (303.5, 50.1)
- moved C654 151.5 mm to (163.5, 160.2)
- moved R622 149.4 mm to (303.5, 53.1)
- moved R652 149.1 mm to (163.5, 163.2)
- moved R653 148.7 mm to (163.5, 166.3)
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Connections:
- C609 pad 1: +5V -> U70_VCP
- C609 pad 2: GND -> +5V
- C615 pad 1: +5V -> U71_VINT
- C624 pad 1: +5V -> U73_VCP
- C624 pad 2: GND -> +5V
- C630 pad 1: +5V -> U74_VINT
- C639 pad 1: +5V -> U76_VCP
- C639 pad 2: GND -> +5V
- C645 pad 1: +5V -> U77_VINT
- C654 pad 1: +5V -> U79_VCP
- C654 pad 2: GND -> +5V
- R400 pad 1: +3V3 -> ATT_DATA
- R400 pad 2: ATT1_C0 -> ATT1_DAT
- R401 pad 2: ATT1_C1 -> ATT1_C0
- R402 pad 2: ATT1_C2 -> ATT1_C1
- R403 pad 2: ATT1_C3 -> ATT1_C2
- R404 pad 2: ATT1_C4 -> ATT1_C3
- R405 pad 2: ATT1_C5 -> ATT1_C4
- R409 pad 1: +3V3 -> ATT_DATA
- R409 pad 2: ATT2_C1 -> ATT2_DAT
- R410 pad 2: ATT2_C2 -> ATT2_C0
- R411 pad 2: ATT2_C3 -> ATT2_C1
- R412 pad 2: ATT2_C4 -> ATT2_C2
- R413 pad 2: ATT2_C5 -> ATT2_C3
- R418 pad 1: +3V3 -> ATT_DATA
- R418 pad 2: ATT3_C2 -> ATT3_DAT
- R419 pad 2: ATT3_C3 -> ATT3_C0
- R420 pad 2: ATT3_C4 -> ATT3_C1
- R421 pad 2: ATT3_C5 -> ATT3_C2
- R424 pad 2: ATT4_C0 -> ATT3_C5
- R427 pad 1: +3V3 -> ATT_DATA
- R427 pad 2: ATT4_C3 -> ATT4_DAT
- R428 pad 2: ATT4_C4 -> ATT4_C0
- R429 pad 2: ATT4_C5 -> ATT4_C1
- R613 pad 1: U72_ISEN0 -> U71_ISEN1
- R617 pad 1: U73_ISEN1 -> U72_ISEN0
- R622 pad 1: U75_ISEN0 -> U73_ISEN0
- R623 pad 1: U75_ISEN1 -> U73_ISEN1
- R628 pad 1: U77_ISEN0 -> U74_ISEN1
- R632 pad 1: U78_ISEN1 -> U75_ISEN0
- R637 pad 1: U80_ISEN0 -> U76_ISEN0
- R638 pad 1: U80_ISEN1 -> U76_ISEN1
- R643 pad 1: U82_ISEN0 -> U77_ISEN1
- R647 pad 1: U83_ISEN1 -> U78_ISEN0
- R652 pad 1: U85_ISEN0 -> U79_ISEN0
- R653 pad 1: U85_ISEN1 -> U79_ISEN1
- U40 pad 3: ATT_DATA -> ATT1_DAT
- U41 pad 3: ATT_DATA -> ATT2_DAT
- U42 pad 3: ATT_DATA -> ATT3_DAT
- U43 pad 3: ATT_DATA -> ATT4_DAT
- U70 pad 11: unconnected-(U70-VCP-Pad11) -> U70_VCP
- U70 pad 14: unconnected-(U70-VINT-Pad14) -> U70_VINT
- U71 pad 11: unconnected-(U71-VCP-Pad11) -> U71_VCP
- U71 pad 14: unconnected-(U71-VINT-Pad14) -> U71_VINT
- U72 pad 11: unconnected-(U72-VCP-Pad11) -> U72_VCP
- U72 pad 14: unconnected-(U72-VINT-Pad14) -> U72_VINT
- U73 pad 11: unconnected-(U73-VCP-Pad11) -> U73_VCP
- U73 pad 14: unconnected-(U73-VINT-Pad14) -> U73_VINT
- U74 pad 11: unconnected-(U74-VCP-Pad11) -> U74_VCP
- U74 pad 14: unconnected-(U74-VINT-Pad14) -> U74_VINT
- U75 pad 11: unconnected-(U75-VCP-Pad11) -> U75_VCP
- U75 pad 14: unconnected-(U75-VINT-Pad14) -> U75_VINT
- U76 pad 11: unconnected-(U76-VCP-Pad11) -> U76_VCP
- U76 pad 14: unconnected-(U76-VINT-Pad14) -> U76_VINT
- U77 pad 11: unconnected-(U77-VCP-Pad11) -> U77_VCP
- U77 pad 14: unconnected-(U77-VINT-Pad14) -> U77_VINT
- U78 pad 11: unconnected-(U78-VCP-Pad11) -> U78_VCP
- U78 pad 14: unconnected-(U78-VINT-Pad14) -> U78_VINT
- U79 pad 11: unconnected-(U79-VCP-Pad11) -> U79_VCP
- U79 pad 14: unconnected-(U79-VINT-Pad14) -> U79_VINT
- U80 pad 11: unconnected-(U80-VCP-Pad11) -> U80_VCP
- U80 pad 14: unconnected-(U80-VINT-Pad14) -> U80_VINT
- U81 pad 11: unconnected-(U81-VCP-Pad11) -> U81_VCP
- U81 pad 14: unconnected-(U81-VINT-Pad14) -> U81_VINT
- U82 pad 11: unconnected-(U82-VCP-Pad11) -> U82_VCP
- U82 pad 14: unconnected-(U82-VINT-Pad14) -> U82_VINT
- U83 pad 11: unconnected-(U83-VCP-Pad11) -> U83_VCP
- U83 pad 14: unconnected-(U83-VINT-Pad14) -> U83_VINT
- U84 pad 11: unconnected-(U84-VCP-Pad11) -> U84_VCP
- U84 pad 14: unconnected-(U84-VINT-Pad14) -> U84_VINT
- U85 pad 11: unconnected-(U85-VCP-Pad11) -> U85_VCP
- U85 pad 14: unconnected-(U85-VINT-Pad14) -> U85_VINT

Commit message: Move each decoupling capacitor to the pin it serves
The audit found 14 chips with no decoupling capacitor within 15 mm.
Across the boards the nearest capacitor to a supply rail was a median
7.5 mm on A and 6.3 mm on C, and 91 mm in the worst case. A capacitor
45 mm from its pin has about 45 nH of loop inductance, near 2.8 ohm at
10 MHz, where milliohms are necessary. It is on the schematic, it is
in the BOM, it is fitted, and it does nothing.

The pass that moves capacitors ran before the fallback placer, so a
chip with no explicit rule was not yet placed and never entered the
pool. The fallback then gave every spare capacitor to the chip with
the most pins on the rail, which is the FPGA on +3V3. Small parts got
none. The pass now runs last.

A count of missing parts was also wrong. Every pad on a rail was
counted as a supply pin, including logic inputs tied high: SRCLR on
the 74HC595, SLEEP on the DRV8833, P/S on the PE4312. Counting only
pins the netlist marks power_in, board C has 15 supply pins and 15
capacitors. Four capacitors are missing across all three boards, not
59. The AD8318 has three supply pins and had one capacitor; it now
has three. The ADCLK846 has six and had five.
Parts:
- moved TP1 229.8 mm to (85.1, 52.4)
- moved C435 212.6 mm to (172.9, 229.6)
- moved C600 199.8 mm to (219.3, 230.0)
- moved C407 197.4 mm to (194.8, 114.0)
- moved C601 191.6 mm to (265.3, 230.0)
- moved C602 189.9 mm to (311.3, 230.0)
- moved C425 183.8 mm to (34.9, 229.6)
- moved C434 183.8 mm to (126.9, 229.6)
- moved C426 183.8 mm to (81.0, 230.1)
- moved TP4 161.6 mm to (340.8, 27.3)
- moved TP5 158.5 mm to (340.8, 82.3)
- moved TP6 147.0 mm to (340.8, 137.3)
- moved TP7 139.7 mm to (340.8, 192.3)
- moved C408 121.5 mm to (187.5, 171.4)
- moved C416 85.9 mm to (188.5, 169.8)
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
Commit message: Do not count a bulk capacitor as decoupling
The placement pass accepted any capacitor on the rail as sufficient.
On board A the flash memory had 10 uF at 5.5 mm and 47 uF at 16.3 mm,
so the pass was satisfied. Both are bulk. The nearest 100 nF was
17.0 mm away, and at that distance the loop inductance removes the
reason to fit it.

The audit tool already used a 10 uF ceiling for this. The placer did
not, so the two disagreed, and the placer was wrong.

The pass now treats only capacitors of 1 uF and below as decoupling,
both when it asks whether a pin is served and when it selects one to
move. It also searches a ring around the pin for free space instead
of using a fixed offset.

Findings fall from 14 to 4. Board A is clean.

Also: build.sh never ran bom.py, so BOM_*.csv were hand-made files
that no step regenerated and the BOM no longer matched the schematic.
Each board's build now writes its own.
Parts:
- moved TP5 168.4 mm to (192.1, 161.4)
- moved TP4 167.9 mm to (208.1, 130.2)
- moved TP3 124.0 mm to (133.2, 225.2)
- moved TP2 31.8 mm to (202.1, 163.9)
- moved TP1 13.9 mm to (84.4, 38.5)
- moved C666 8.95 mm to (302.9, 149.7)
- moved C686 8.95 mm to (302.9, 204.7)
- moved C626 8.95 mm to (302.9, 39.7)
- moved C646 8.95 mm to (302.9, 94.8)
- moved C426 5.44 mm to (82.5, 224.9)
- moved C611 5.06 mm to (87.7, 42.5)
- moved C616 5.06 mm to (167.7, 42.5)
- moved C621 5.06 mm to (247.7, 42.5)
- moved C651 5.06 mm to (87.7, 152.5)
- moved C656 5.06 mm to (167.7, 152.5)
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
Commit message: Let the placer, not the separator, own the capacitor position
Placing a capacitor beside its supply pin and then resolving overlaps
moves it away again. On board C the pass put a 100 nF 4.7 mm from the
attenuator's pin, the separator cleared 191 overlaps, and the
capacitor finished 17.9 mm away.

The pass now runs after separation and searches for free space around
the pin itself, so it does not need the separator afterwards. It
moves 21 capacitors on A, 26 on C and 12 on D.

Measured at the supply pin, the median distance is 2.8 mm on A,
5.4 mm on C and 4.6 mm on D. Board C's worst supply pin improves from
98.5 mm to 8.9 mm. Findings fall from 14 to 1.
Parts:
- moved TP1 239.9 mm to (242.2, 219.2)
- moved TP5 168.4 mm to (340.8, 82.3)
- moved TP3 123.2 mm to (10.0, 221.4)
- moved TP2 74.9 mm to (173.8, 233.2)
- moved C407 22.0 mm to (200.2, 135.3)
- moved C408 17.5 mm to (192.2, 188.2)
- moved C417 7.87 mm to (195.4, 206.2)
- moved C631 4.24 mm to (85.5, 93.8)
- moved C651 4.24 mm to (85.5, 148.8)
- moved C671 4.24 mm to (85.5, 203.8)
- moved C611 4.24 mm to (85.5, 38.9)
- moved C636 4.24 mm to (165.6, 93.8)
- moved C641 4.24 mm to (245.6, 93.8)
- moved C656 4.24 mm to (165.6, 148.8)
- moved C661 4.24 mm to (245.6, 148.8)
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
Commit message: Compare symbol pins against footprint pads before placement
Every fault that would have stopped a board in this work sits in one
layer: a symbol pin number that does not agree with a footprint pad
number. The ADC paddle was pin 0 against pad 65. The attenuator
paddle was named Pad against pad 21. The gas discharge tubes used
pins 1 and 3 against pads 1 and 2. The crystal had two pins on a
four-pad part, so XO went to the can. The Ethernet PHY carried the
footprint of a different package. Each was found separately, by hand,
after it had already cost placement and routing time.

temel_denetim checks the whole class at once. For each part it
reports pins with no pad, where the net goes nowhere while the
schematic looks correct; pads with no pin, where copper is left
unconnected; and a count mismatch, which is the quickest sign that a
footprint belongs to another part.

It reads the symbols embedded in the schematics and not the library
file, because the library was edited by hand while its generator
stayed behind.

yap.sh runs it after pcb_kur and before placement, and stops there. A
wrong schematic makes everything below it worthless.

All three boards report zero. The parts it cannot check are those
with no symbol: mounting holes, fiducials and test points.
Parts:
- moved TP5 168.4 mm to (192.1, 161.4)
- moved TP7 147.5 mm to (193.3, 191.8)
- moved TP1 135.9 mm to (311.1, 102.1)
- moved TP2 35.1 mm to (196.8, 206.7)
- moved C417 2.75 mm to (192.7, 206.7)
- moved TP3 2.52 mm to (12.1, 222.8)
