File: hardware/kicad/C_rf/dogrudan_sdr_C.kicad_pcb (KiCad board)
At the start: 2 copper layers, 350 x 235 mm, 502 parts, among them J1 SMA anten 1, J2 SMA anten 2, J3 SMA anten 3, J4 SMA anten 4, J80 A kartina, J81 A kartina #2, J82 RX1 -> A, J83 RX2 -> A, J84 RX3 -> A, J85 RX4 -> A, J86 TX1 <- A, J87 TX2 <- A, J88 TX3 <- A, J89 TX4 <- A, J90 D kartina, K11 G6KU-2F-Y, K12 G6KU-2F-Y, K13 G6KU-2F-Y, K14 G6KU-2F-Y, K15 G6KU-2F-Y, K16 G6KU-2F-Y, K17 G6KU-2F-Y, K21 G6KU-2F-Y, K22 G6KU-2F-Y, K23 G6KU-2F-Y, K24 G6KU-2F-Y, K25 G6KU-2F-Y, K26 G6KU-2F-Y, K27 G6KU-2F-Y, K31 G6KU-2F-Y, K32 G6KU-2F-Y, K33 G6KU-2F-Y, K34 G6KU-2F-Y, K35 G6KU-2F-Y, K36 G6KU-2F-Y, K37 G6KU-2F-Y, K41 G6KU-2F-Y, K42 G6KU-2F-Y, K43 G6KU-2F-Y, K44 G6KU-2F-Y, K45 G6KU-2F-Y, K46 G6KU-2F-Y, K47 G6KU-2F-Y, U40 PE4312C-Z, U41 PE4312C-Z, U42 PE4312C-Z, U43 PE4312C-Z, U60 74HC595D, U61 74HC595D, U62 74HC595D, U63 74HC595D, U64 74HC595D, U65 74HC595D, U66 74HC595D, U70 DRV8833PWPR, U71 DRV8833PWPR, U72 DRV8833PWPR, U73 DRV8833PWPR, U74 DRV8833PWPR, U75 DRV8833PWPR, U76 DRV8833PWPR, U77 DRV8833PWPR, U78 DRV8833PWPR, U79 DRV8833PWPR, U80 DRV8833PWPR, U81 DRV8833PWPR, U82 DRV8833PWPR, U83 DRV8833PWPR, U84 DRV8833PWPR, U85 DRV8833PWPR, U90 TPS62130

Commit message: Replace the receive band filters: they passed nothing
Simulation in ngspice shows all six filter positions peak below the
band they must pass, with the band itself 24 to 41 dB down. The
receiver would have been deaf on every band. No connectivity check
can find this: the netlist is correct and the values are wrong.

The cause is arithmetic. The three resonators were tuned as bare LC
pairs, but the coupling capacitors sit in parallel with them and pull
the frequency down. On 160m, 430 pF of resonator plus 270 pF of end
coupling plus 62 pF between resonators gives 762 pF, and with 16 uH
that is 1.44 MHz against a band at 1.8 to 2.0 MHz.

Compensation alone is not sufficient. Top coupling is a narrowband
structure and these positions are wide: 80+60 m spans 3.5 to
5.4 MHz, or 44%.

The structure is now a ladder bandpass, shunt resonator then series
resonator then shunt resonator, synthesised from a 3-pole 0.1 dB
Chebyshev prototype and verified with the values snapped to E12.

  band      loss   worst band edge   was
  160m      1.31   -1.71             -34
  80_60m    0.52   -0.97             -25
  40_30m    0.73   -1.49             -27
  20_17m    0.83   -1.04             -32
  15_10m    0.71   -1.00             -28
  6m        1.72   -2.37             -41

Board C falls from 502 parts to 406. The inductors are all SMD: the
toroids gave a Q of 150 against 40, which is one decibel on 160m
where atmospheric noise sets the receiver's floor, and they were 48
parts that a machine cannot place.
Parts:
- removed C1000, C1060, C1120, C1180, C1181: 270pF, C_0603_1608Metric
- removed C1002, C1062, C1122, C1182, C1183: 62pF, C_0603_1608Metric
- removed C1010, C1070, C1130, C1190, C1191: 390pF, C_0603_1608Metric
- removed C1012, C1072, C1132, C1192, C1193: 82pF, C_0603_1608Metric
- removed C1020, C1080, C1140, C1200, C1201: 160pF, C_0603_1608Metric
- removed C1022, C1082, C1142, C1202, C1203: 33pF, C_0603_1608Metric
- removed C1030, C1090, C1150, C1151, C1210, C1211: 56pF, C_0603_1608Metric
- removed C1032, C1092, C1152, C1153, C1212, C1213: 13pF, C_0603_1608Metric
- removed C1040, C1100, C1160, C1161, C1220, C1221: 47pF, C_0603_1608Metric
- removed C1042, C1102, C1162, C1163, C1222, C1223: 10pF, C_0603_1608Metric
- removed C1050, C1110, C1170, C1171, C1230, C1231: 5.6pF, C_0603_1608Metric
- removed C1052, C1112, C1172, C1173, C1232, C1233: 1.3pF, C_0603_1608Metric
- removed C1145, C1147, C1149, C1205, C1207, C1209: 91pF, C_0603_1608Metric
- removed C1155, C1157, C1159, C1215, C1217, C1219: 51pF, C_0603_1608Metric
- removed C1165, C1167, C1169, C1225, C1227, C1229: 30pF, C_0603_1608Metric
- removed C1175, C1177, C1179, C1235, C1237, C1239: 15pF, C_0603_1608Metric
- removed C1185, C1187, C1189: 430pF, C_0603_1608Metric
- removed C1195, C1197, C1199: 180pF, C_0603_1608Metric
- removed L1144, L1146, L1148, L1204, L1206, L1208: 3.9uH, L_0805_2012Metric
- removed L1154, L1156, L1158, L1214, L1216, L1218: 2uH, L_0805_2012Metric
- removed L1164, L1166, L1168, L1224, L1226, L1228: 1.3uH, L_0805_2012Metric
- removed L1174, L1176, L1178, L1234, L1236, L1238: 620nH, L_Toroid_T50_Vertical
- removed L1184, L1186, L1188: 16uH, L_Toroid_T50_Vertical
- removed L1194, L1196, L1198: 7.5uH, L_0805_2012Metric
- added L1000: 1uH, L_Toroid_T50_Vertical, F.Cu at (54.7, 11.0)
- added L1002: 1uH, L_Toroid_T50_Vertical, F.Cu at (69.0, 11.0)
- added L1010: 3.3uH, L_Toroid_T50_Vertical, F.Cu at (123.3, 11.0)
- added L1012: 470nH, L_Toroid_T50_Vertical, F.Cu at (134.7, 11.0)
- added L1020: 220nH, L_0805_2012Metric, F.Cu at (189.0, 11.0)
- added L1022: 1.5uH, L_0805_2012Metric, F.Cu at (193.1, 11.0)
- added L1030: 33nH, L_0805_2012Metric, F.Cu at (264.9, 11.0)
- added L1032: 33nH, L_0805_2012Metric, F.Cu at (269.0, 11.0)
- added L1040: 18uH, L_Toroid_T50_Vertical, F.Cu at (83.3, 66.0)
- added L1042: 1uH, L_Toroid_T50_Vertical, F.Cu at (94.7, 66.0)
- added L1050: 470nH, L_Toroid_T50_Vertical, F.Cu at (149.0, 66.0)
- added L1052: 2.2uH, L_Toroid_T50_Vertical, F.Cu at (163.3, 66.0)
- added L1060: 150nH, L_0805_2012Metric, F.Cu at (224.9, 66.0)
- added L1062: 150nH, L_0805_2012Metric, F.Cu at (229.0, 66.0)
- added L1070: 820nH, L_0805_2012Metric, F.Cu at (273.1, 66.0)
- added L1072: 1uH, L_Toroid_T50_Vertical, F.Cu at (54.7, 121.0)
- added L1080: 1uH, L_Toroid_T50_Vertical, F.Cu at (109.0, 121.0)
- added L1082: 3.3uH, L_Toroid_T50_Vertical, F.Cu at (123.3, 121.0)
- added L1090: 220nH, L_0805_2012Metric, F.Cu at (184.9, 121.0)
- added L1092: 220nH, L_0805_2012Metric, F.Cu at (189.0, 121.0)
- added L1100: 680nH, L_0805_2012Metric, F.Cu at (233.1, 121.0)
- added L1102: 33nH, L_0805_2012Metric, F.Cu at (264.9, 121.0)
- added L1110: 1uH, L_Toroid_T50_Vertical, F.Cu at (69.0, 176.0)
- added L1112: 18uH, L_Toroid_T50_Vertical, F.Cu at (83.3, 176.0)
- added L1120: 470nH, L_Toroid_T50_Vertical, F.Cu at (134.7, 176.0)
- added L1122: 470nH, L_Toroid_T50_Vertical, F.Cu at (149.0, 176.0)
- added L1130: 1.5uH, L_0805_2012Metric, F.Cu at (193.1, 176.0)
- added L1132: 150nH, L_0805_2012Metric, F.Cu at (224.9, 176.0)
- added L1140: 33nH, L_0805_2012Metric, F.Cu at (269.0, 176.0)
- added L1142: 820nH, L_0805_2012Metric, F.Cu at (273.1, 176.0)
- C1001: value 270pF -> 6800pF
- C1003: value 62pF -> 6800pF
- C1005: value 430pF -> 390pF
- C1007, C1009: value 430pF -> 1200pF
- C1013: value 82pF -> 680pF
- C1015: value 180pF -> 680pF
- C1019: value 180pF -> 470pF
- C1021: value 160pF -> 470pF
- C1023: value 33pF -> 68pF
- C1025, C1027: value 91pF -> 270pF
- C1029: value 91pF -> 56pF
- C1031: value 56pF -> 270pF
- C1033: value 13pF -> 270pF
- C1035: value 51pF -> 12pF
- C1037, C1039: value 51pF -> 6800pF
- C1041: value 47pF -> 390pF
- C1043: value 10pF -> 1200pF
- C1045: value 30pF -> 1200pF
- C1047: value 30pF -> 390pF
- C1049: value 30pF -> 680pF
- C1051: value 5.6pF -> 680pF
- C1053: value 1.3pF -> 180pF
- C1055, C1057: value 15pF -> 470pF
- C1059: value 15pF -> 68pF
- C1063: value 62pF -> 270pF
- C1065: value 430pF -> 56pF
- C1067, C1069: value 430pF -> 270pF
- C1071: value 390pF -> 12pF
- C1073: value 82pF -> 6800pF
- C1075: value 180pF -> 6800pF
- C1077: value 180pF -> 390pF
- C1079: value 180pF -> 1200pF
- C1081: value 160pF -> 1200pF
- C1083: value 33pF -> 390pF
- C1085, C1087: value 91pF -> 680pF
- C1089: value 91pF -> 180pF
- C1091: value 56pF -> 470pF
- C1093: value 13pF -> 470pF
- C1095: value 51pF -> 68pF
- C1097, C1099: value 51pF -> 270pF
- C1101: value 47pF -> 56pF
- C1103: value 10pF -> 270pF
- C1105: value 30pF -> 270pF
- C1107: value 30pF -> 12pF
- C1109: value 30pF -> 6800pF
- C1111: value 5.6pF -> 6800pF
- C1113: value 1.3pF -> 390pF
- C1115, C1117: value 15pF -> 1200pF
- C1119: value 15pF -> 390pF
- C1121: value 270pF -> 680pF
- C1123: value 62pF -> 680pF
- C1125: value 430pF -> 180pF
- C1127, C1129: value 430pF -> 470pF
- C1131: value 390pF -> 68pF
- C1133: value 82pF -> 270pF
- C1135, C1139: value 180pF -> 270pF
- C1137: value 180pF -> 56pF
- C1141: value 160pF -> 270pF
- C1143: value 33pF -> 12pF
- L1004: value 16uH -> 18uH
- L1006, L1008: value 16uH -> 1uH
- L1014: value 7.5uH -> 470nH; footprint L_0805_2012Metric -> L_Toroid_T50_Vertical
- L1016: value 7.5uH -> 2.2uH; footprint L_0805_2012Metric -> L_Toroid_T50_Vertical
- L1018: value 7.5uH -> 220nH
- L1024, L1026: value 3.9uH -> 150nH
- L1028: value 3.9uH -> 680nH
- L1034: value 2uH -> 820nH
- L1036, L1038: value 2uH -> 1uH; footprint L_0805_2012Metric -> L_Toroid_T50_Vertical
- L1044, L1108: value 1.3uH -> 1uH; footprint L_0805_2012Metric -> L_Toroid_T50_Vertical
- L1046: value 1.3uH -> 3.3uH; footprint L_0805_2012Metric -> L_Toroid_T50_Vertical
- L1048: value 1.3uH -> 470nH; footprint L_0805_2012Metric -> L_Toroid_T50_Vertical
- L1054, L1056: value 620nH -> 220nH; footprint L_Toroid_T50_Vertical -> L_0805_2012Metric
- L1058: value 620nH -> 1.5uH; footprint L_Toroid_T50_Vertical -> L_0805_2012Metric
- L1064: value 16uH -> 680nH; footprint L_Toroid_T50_Vertical -> L_0805_2012Metric
- L1066, L1068: value 16uH -> 33nH; footprint L_Toroid_T50_Vertical -> L_0805_2012Metric
- L1074, L1078: value 7.5uH -> 1uH; footprint L_0805_2012Metric -> L_Toroid_T50_Vertical
- L1076: value 7.5uH -> 18uH; footprint L_0805_2012Metric -> L_Toroid_T50_Vertical
- L1084, L1086: value 3.9uH -> 470nH; footprint L_0805_2012Metric -> L_Toroid_T50_Vertical
- L1088: value 3.9uH -> 2.2uH; footprint L_0805_2012Metric -> L_Toroid_T50_Vertical
- L1094: value 2uH -> 1.5uH
- L1096, L1098: value 2uH -> 150nH
- L1104: value 1.3uH -> 33nH
- L1106: value 1.3uH -> 820nH
- L1114, L1116: value 620nH -> 1uH
- L1118: value 620nH -> 3.3uH
- L1124: value 16uH -> 2.2uH
- L1126, L1128: value 16uH -> 220nH; footprint L_Toroid_T50_Vertical -> L_0805_2012Metric
- L1134: value 7.5uH -> 150nH
- L1136: value 7.5uH -> 680nH
- L1138: value 7.5uH -> 33nH
- moved C1113 234.4 mm to (80.0, 198.0)
- moved C1111 228.3 mm to (73.0, 198.0)
- moved L1108 209.6 mm to (54.7, 176.0)
- moved C1109 203.2 mm to (66.0, 198.0)
- moved L1066 195.9 mm to (264.9, 66.0), turned to 90 degrees
- moved L1114 194.2 mm to (94.7, 176.0)
- moved L1116 194.2 mm to (109.0, 176.0)
- moved L1118 194.2 mm to (123.3, 176.0)
- moved C1067 193.1 mm to (266.0, 88.0)
- moved C1069 193.1 mm to (273.0, 88.0)
- moved C1115 191.4 mm to (106.0, 198.0)
- moved C1117 191.4 mm to (113.0, 198.0)
- moved C1119 191.4 mm to (120.0, 198.0)
- moved L1068 185.7 mm to (269.0, 66.0), turned to 90 degrees
- moved L1064 178.4 mm to (233.1, 66.0)
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Connections:
- C1001 pad 1: N11_3 -> F11_A
- C1001 pad 2: F11_B -> GND
- C1003 pad 1: N11_2 -> F11_B
- C1003 pad 2: N11_3 -> GND
- C1005 pad 1: N11_1 -> N11_S
- C1005 pad 2: GND -> F11_B
- C1007 pad 1: N11_2 -> F12_A
- C1009 pad 1: N11_3 -> F12_B
- C1011 pad 1: N12_3 -> N12_S
- C1013 pad 1: N12_2 -> F13_A
- C1013 pad 2: N12_3 -> GND
- C1015 pad 1: N12_1 -> F13_B
- C1017 pad 1: N12_2 -> N13_S
- C1017 pad 2: GND -> F13_B
- C1019 pad 1: N12_3 -> F14_A
- C1021 pad 1: N13_3 -> F14_B
- C1021 pad 2: F13_B -> GND
- C1023 pad 1: N13_2 -> N14_S
- C1023 pad 2: N13_3 -> F14_B
- C1025 pad 1: N13_1 -> F15_A
- C1027 pad 1: N13_2 -> F15_B
- C1029 pad 1: N13_3 -> N15_S
- C1029 pad 2: GND -> F15_B
- C1031 pad 1: N14_3 -> F16_A
- C1031 pad 2: F14_B -> GND
- C1033 pad 1: N14_2 -> F16_B
- C1033 pad 2: N14_3 -> GND
- C1035 pad 1: N14_1 -> N16_S
- C1035 pad 2: GND -> F16_B
- C1037 pad 1: N14_2 -> F21_A
- C1039 pad 1: N14_3 -> F21_B
- C1041 pad 1: N15_3 -> N21_S
- C1041 pad 2: F15_B -> F21_B
- C1043 pad 1: N15_2 -> F22_A
- C1043 pad 2: N15_3 -> GND
- C1045 pad 1: N15_1 -> F22_B
- C1047 pad 1: N15_2 -> N22_S
- C1047 pad 2: GND -> F22_B
- C1049 pad 1: N15_3 -> F23_A
- C1051 pad 1: N16_3 -> F23_B
- C1051 pad 2: F16_B -> GND
- C1053 pad 1: N16_2 -> N23_S
- C1053 pad 2: N16_3 -> F23_B
- C1055 pad 1: N16_1 -> F24_A
- C1057 pad 1: N16_2 -> F24_B
- C1059 pad 1: N16_3 -> N24_S
- C1059 pad 2: GND -> F24_B
- C1061 pad 1: N21_3 -> F25_A
- C1061 pad 2: F21_B -> GND
- C1063 pad 1: N21_2 -> F25_B
- C1063 pad 2: N21_3 -> GND
- C1065 pad 1: N21_1 -> N25_S
- C1065 pad 2: GND -> F25_B
- C1067 pad 1: N21_2 -> F26_A
- C1069 pad 1: N21_3 -> F26_B
- C1071 pad 1: N22_3 -> N26_S
- C1071 pad 2: F22_B -> F26_B
- C1073 pad 1: N22_2 -> F31_A
- C1073 pad 2: N22_3 -> GND
- C1075 pad 1: N22_1 -> F31_B
- C1077 pad 1: N22_2 -> N31_S
- C1077 pad 2: GND -> F31_B
- C1079 pad 1: N22_3 -> F32_A
- C1081 pad 1: N23_3 -> F32_B
- C1081 pad 2: F23_B -> GND
- C1083 pad 1: N23_2 -> N32_S
- C1083 pad 2: N23_3 -> F32_B
- C1085 pad 1: N23_1 -> F33_A
- C1087 pad 1: N23_2 -> F33_B
- C1089 pad 1: N23_3 -> N33_S
- C1089 pad 2: GND -> F33_B
- C1091 pad 1: N24_3 -> F34_A
- C1091 pad 2: F24_B -> GND
- C1093 pad 1: N24_2 -> F34_B
- C1093 pad 2: N24_3 -> GND
- C1095 pad 1: N24_1 -> N34_S
- C1095 pad 2: GND -> F34_B
- C1097 pad 1: N24_2 -> F35_A
- C1099 pad 1: N24_3 -> F35_B
- C1101 pad 1: N25_3 -> N35_S
- C1101 pad 2: F25_B -> F35_B
- C1103 pad 1: N25_2 -> F36_A
- C1103 pad 2: N25_3 -> GND
- C1105 pad 1: N25_1 -> F36_B
- C1107 pad 1: N25_2 -> N36_S
- C1107 pad 2: GND -> F36_B
- C1109 pad 1: N25_3 -> F41_A
- C1111 pad 1: N26_3 -> F41_B
- C1111 pad 2: F26_B -> GND
- C1113 pad 1: N26_2 -> N41_S
- C1113 pad 2: N26_3 -> F41_B
- C1115 pad 1: N26_1 -> F42_A
- C1117 pad 1: N26_2 -> F42_B
- C1119 pad 1: N26_3 -> N42_S
- C1119 pad 2: GND -> F42_B
- C1121 pad 1: N31_3 -> F43_A
- C1121 pad 2: F31_B -> GND
- C1123 pad 1: N31_2 -> F43_B
- C1123 pad 2: N31_3 -> GND
- C1125 pad 1: N31_1 -> N43_S
- C1125 pad 2: GND -> F43_B
- C1127 pad 1: N31_2 -> F44_A
- C1129 pad 1: N31_3 -> F44_B
- C1131 pad 1: N32_3 -> N44_S
- C1131 pad 2: F32_B -> F44_B
- C1133 pad 1: N32_2 -> F45_A
- C1133 pad 2: N32_3 -> GND
- C1135 pad 1: N32_1 -> F45_B
- C1137 pad 1: N32_2 -> N45_S
- C1137 pad 2: GND -> F45_B
- C1139 pad 1: N32_3 -> F46_A
- C1141 pad 1: N33_3 -> F46_B
- C1141 pad 2: F33_B -> GND
- C1143 pad 1: N33_2 -> N46_S
- C1143 pad 2: N33_3 -> F46_B
- L1004 pad 1: N11_1 -> F11_A
- L1004 pad 2: GND -> N11_S
- L1006 pad 1: N11_2 -> F12_A
- L1008 pad 1: N11_3 -> F12_B
- L1014 pad 1: N12_1 -> F13_B
- L1016 pad 1: N12_2 -> F13_A
- L1016 pad 2: GND -> N13_S
- L1018 pad 1: N12_3 -> F14_A
- L1024 pad 1: N13_1 -> F15_A
- L1026 pad 1: N13_2 -> F15_B
- L1028 pad 1: N13_3 -> F15_A
- L1028 pad 2: GND -> N15_S
- L1034 pad 1: N14_1 -> F16_A
- L1034 pad 2: GND -> N16_S
- L1036 pad 1: N14_2 -> F21_A
- L1038 pad 1: N14_3 -> F21_B
- L1044 pad 1: N15_1 -> F22_B
- L1046 pad 1: N15_2 -> F22_A
- L1046 pad 2: GND -> N22_S
- L1048 pad 1: N15_3 -> F23_A
- L1054 pad 1: N16_1 -> F24_A
- L1056 pad 1: N16_2 -> F24_B
- L1058 pad 1: N16_3 -> F24_A
- L1058 pad 2: GND -> N24_S
- L1064 pad 1: N21_1 -> F25_A
- L1064 pad 2: GND -> N25_S
- L1066 pad 1: N21_2 -> F26_A
- L1068 pad 1: N21_3 -> F26_B
- L1074 pad 1: N22_1 -> F31_B
- L1076 pad 1: N22_2 -> F31_A
- L1076 pad 2: GND -> N31_S
- L1078 pad 1: N22_3 -> F32_A
- L1084 pad 1: N23_1 -> F33_A
- L1086 pad 1: N23_2 -> F33_B
- L1088 pad 1: N23_3 -> F33_A
- L1088 pad 2: GND -> N33_S
- L1094 pad 1: N24_1 -> F34_A
- L1094 pad 2: GND -> N34_S
- L1096 pad 1: N24_2 -> F35_A
- L1098 pad 1: N24_3 -> F35_B
- L1104 pad 1: N25_1 -> F36_B
- L1106 pad 1: N25_2 -> F36_A
- L1106 pad 2: GND -> N36_S
- L1108 pad 1: N25_3 -> F41_A
- L1114 pad 1: N26_1 -> F42_A
- L1116 pad 1: N26_2 -> F42_B
- L1118 pad 1: N26_3 -> F42_A
- L1118 pad 2: GND -> N42_S
- L1124 pad 1: N31_1 -> F43_A
- L1124 pad 2: GND -> N43_S
- L1126 pad 1: N31_2 -> F44_A
- L1128 pad 1: N31_3 -> F44_B
- L1134 pad 1: N32_1 -> F45_B
- L1136 pad 1: N32_2 -> F45_A
- L1136 pad 2: GND -> N45_S
- L1138 pad 1: N32_3 -> F46_A

Commit message: Replace the transmit filters: harmonic suppression was illegal
Simulation of the output filters shows second-harmonic suppression
between 3 and 30 dB, where 43 dB is necessary below 30 MHz and 60 dB
above. On the 80/60 m position the second harmonic of 3.5 MHz is
3.4 dB down: the filter barely touches it. The transmitter would have
been out of specification on every band, and the board gives no sign
of it. Output power, SWR and efficiency all read correctly while the
harmonic radiates.

The cause is the band grouping. One position must pass 5.37 MHz, so
its cutoff is at 6.0, and the second harmonic of the same position's
lowest band, 3.5 MHz, falls at 7.0. More poles do not help: by the
Chebyshev attenuation formula, nine poles give 32 dB there.

Each series inductor now has a parallel capacitor that places a
transmission zero on the harmonic. 80 m and 60 m are separate
positions, because a trap at 7.0 MHz also attenuates a 5.37 MHz
passband. That uses the seventh relay, which was a bypass; a
transmitter with no harmonic filter in line is not legal in any case.

  band      loss   2nd harmonic   was
  160m      0.61   -82.4          -25.2
  80m       0.64   -80.7          grouped
  60m       0.45   -81.9          grouped
  40_30m    1.45   -58.0          -9.5
  20_17m    0.88   -68.4          -18.2
  15_10m    1.35   -61.0          -14.1
  6m        1.14   -82.8          -30.2
Parts:
- moved TP1 250.7 mm to (82.2, 54.2)
- moved TP5 168.4 mm to (192.1, 161.4)
- moved TP4 167.9 mm to (340.8, 27.3)
- moved TP6 148.0 mm to (340.8, 137.3)
- moved TP7 147.5 mm to (340.8, 192.3)
- moved TP2 76.4 mm to (210.0, 117.9)

Commit message: Fit the filter bank and clear the overlaps
Board D's filter bank needs 285.6 mm of width with both inductors of
each band side by side, against about 236 mm available. Stacking them
vertically corrects the width and breaks the height: the strip
between the driver transformer and the relay row is 15.8 mm and a
stacked pair of T68 cores needs 37.7 mm.

Mapping the board in 10 mm bands gave the answer. Everything below
the relay row is the coupler and detector block at x above 250, while
the filter columns run from x 4 to 236. The space under them was
empty. The relay row moves from y 130 to 142 and its drivers from 155
to 172, with the filter block following. No board grew and the chain
stays in one row.

The separator never moves a part whose reference begins with U, J, T,
Y, L, Q, K or H, so two such parts overlapping cannot be separated
and the fix belongs in the placement rules. On A the XT60's courtyard
is 22.4 mm tall and snapped to the top edge, so it covered the
reverse-polarity MOSFET; the crystals and their inductors were placed
by the fallback and landed inside the PHY. All three now have
explicit positions.

The separator also gained a last resort: a movable part wedged so
that every push lands it in another part is relocated to the nearest
free position.

All three boards are at zero overlaps.
Parts:
- L1000, L1002, L1004, L1006, L1008, L1010, L1012, L1014, L1016, L1036, L1038, L1040, L1042, L1044, L1046, L1048, L1050, L1052, L1072, L1074, L1076, L1078, L1080, L1082, L1084, L1086, L1088, L1108, L1110, L1112, L1114, L1116, L1118, L1120, L1122, L1124: footprint L_Toroid_T50_Vertical -> L_0805_2012Metric
- moved TP1 218.2 mm to (299.8, 39.0)
- moved TP5 168.4 mm to (340.8, 82.3)
- moved TP7 147.5 mm to (193.3, 191.8)
- moved R690 111.2 mm to (154.4, 158.6)
- moved TP2 95.3 mm to (151.1, 43.0)
- moved R90 63.1 mm to (88.5, 151.1)
- moved L1000 10.2 mm to (64.9, 11.0)
- moved L1036 10.2 mm to (64.9, 66.0)
- moved L1072 10.2 mm to (64.9, 121.0)
- moved L1108 10.2 mm to (64.9, 176.0)
- moved L1012 10.2 mm to (144.9, 11.0)
- moved L1048 10.2 mm to (144.9, 66.0)
- moved L1084 10.2 mm to (144.9, 121.0)
- moved L1120 10.2 mm to (144.9, 176.0)
- moved L1010 10.2 mm to (113.1, 11.0)
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Routing:
- net RX2_B1_IN: track 12.7 -> 0.00 mm
- net RX1_B1_IN: track 12.7 -> 0.00 mm
- net RX4_B1_IN: track 12.7 -> 0.00 mm
- net RX3_B1_IN: track 12.7 -> 0.00 mm
Other:
- board text removed: "​!! 100W RF WHEN TRANSMITTING !!"
- board text removed: "​15/10m"
- board text removed: "​160m"
- board text removed: "​20/17m"
- board text removed: "​40/30m"
- board text removed: "​6m"
- board text removed: "​80/60m"
- board text removed: "​ANT 1"
- board text removed: "​ANT 2"
- board text removed: "​ANT 3"
- board text removed: "​ANT 4"
- board text removed: "​BYPASS"
- board text removed: "​CHASSIS GND - THIS HOLE ONLY"
- board text removed: "​CONTROL"
- board text removed: "​CONTROL 2"
- board text removed: "​RF FILTER BANK - 4 CH x 7 BANDS REV A"
- board text removed: "​RX1 -> A"
- board text removed: "​RX2 -> A"
- board text removed: "​RX3 -> A"
- board text removed: "​RX4 -> A"
- board text removed: "​TO BOARD D"
- board text removed: "​TX1 <- A"
- board text removed: "​TX2 <- A"
- board text removed: "​TX3 <- A"
- board text removed: "​TX4 <- A"

Commit message: Close the last overlaps and record the pass that undid the other
Board D reaches zero overlaps. Two remained after the relay row
moved: a T68 clipping the driver transformer by 1 x 2 mm, and two
2N7002 transistors two millimetres apart, which the separator was
never going to touch because both begin with Q.

One finding is left on D. Tracing a single capacitor through every
stage shows the mechanism:

  pcb_kur          121.2 mm from the chip
  placement          5.1 mm   correct
  separation        21.0 mm   pushed away
  decoupling pass   25.3 mm   handed to another chip

The placer puts the capacitor beside the pin that needs it, the
separator finds an overlap and moves it, and the decoupling pass then
reads it as the nearest free capacitor for somebody else. The chip
that began with a correct capacitor ends with none.

The two steps disagreed about what an overlap is: the pass used a
1.4 mm margin while the separator used its courtyard box. What one
called clear the other called a collision. The pass now uses the
separator's measure. Its guard against taking a chip's only capacitor
was also too broad, counting chips connected through a logic input
tied high; it now applies the same power_in test.

What remains is to decide which of the two passes owns the final
position.
Parts:
- moved TP1 282.5 mm to (82.2, 219.2)
- moved TP2 191.6 mm to (122.2, 232.4)
- moved TP5 168.4 mm to (192.1, 161.4)
- moved TP3 120.4 mm to (130.1, 225.6)
- moved R690 13.1 mm to (158.7, 146.2)
- moved C651 8.53 mm to (87.1, 157.1)
- moved C656 8.53 mm to (167.1, 157.1)
- moved C661 8.53 mm to (247.1, 157.1)
- moved C666 8.53 mm to (307.1, 157.1)
- moved C671 8.53 mm to (87.1, 212.1)
- moved C676 8.53 mm to (167.1, 212.1)
- moved C681 8.53 mm to (247.1, 212.1)
- moved C686 8.53 mm to (307.1, 212.1)
- moved C611 8.53 mm to (87.1, 47.1)
- moved C616 8.53 mm to (167.1, 47.1)
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
Commit message: Name the copyright holder and stamp it into the generated files
The repository had three licence files and no statement of who owns
the work. The only record of authorship was the git author field.

Copyleft depends on that statement. GPL and CERN-OHL-S work because
the holder grants permission on condition of reciprocity; with no
holder named there is nobody to require it from a downstream user.
Naming the author keeps the design open rather than closing it.

kicad/telif.py is the single source. The line reaches the schematics
through their title block and not through the generators, because
every schematic file is rewritten on each build and a header placed in
a generator would disappear at the first regeneration. All 23
schematics carry it. 109 source files have SPDX headers, split by the
project's own table: generators and the layout chain are hardware
under CERN-OHL-S-2.0, HDL and the audit tools are software under
GPL-3.0-only.

Board C's inductors also move to footprints that match parts that can
be bought. All of them sat on 0805 pads. Of the values this design
needs, 33 to 220 nH are 0603 parts, 470 and 820 nH are 0805, and
everything from 1000 nH upward is 1210, which is 3.2 by 2.5 mm and
does not fit an 0805 land. 32 inductors could not have been soldered.

A symbol-against-footprint check cannot find this. Those two agreed
with each other; what was wrong was the body size of the real part
behind the footprint.
Parts:
- L1000, L1002, L1004, L1006, L1008, L1010, L1016, L1022, L1028, L1034, L1036, L1038, L1040, L1042, L1044, L1046, L1052, L1058, L1064, L1070, L1072, L1074, L1076, L1078, L1080, L1082, L1088, L1094, L1100, L1106, L1108, L1110, L1112, L1114, L1116, L1118, L1124, L1130, L1136, L1142: footprint L_0805_2012Metric -> L_1210_3225Metric
- L1018, L1020, L1024, L1026, L1030, L1032, L1054, L1056, L1060, L1062, L1066, L1068, L1090, L1092, L1096, L1098, L1102, L1104, L1126, L1128, L1132, L1134, L1138, L1140: footprint L_0805_2012Metric -> L_0603_1608Metric
- moved TP1 217.7 mm to (299.8, 220.0)
- moved TP5 168.4 mm to (340.8, 82.3)
- moved R400 163.5 mm to (199.4, 126.0)
- moved TP7 147.5 mm to (340.8, 192.3)
- moved R409 130.2 mm to (188.1, 168.4)
- moved R418 124.5 mm to (191.3, 180.0)
- moved TP3 118.0 mm to (12.1, 222.8)
- moved R427 115.7 mm to (194.5, 204.2)
- moved TP2 37.0 mm to (85.3, 230.1)
- moved R690 17.5 mm to (141.2, 145.6)
- moved C407 7.49 mm to (198.1, 127.3)
- moved C408 6.61 mm to (188.9, 182.2)
- moved C417 5.43 mm to (188.8, 202.0)
- moved C636 3.21 mm to (166.9, 102.1)
- moved C641 3.21 mm to (246.9, 102.1)
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Routing:
- net RX2_B1_IN: track 0.00 -> 12.7 mm
- net RX1_B1_IN: track 0.00 -> 12.7 mm
- net RX4_B1_IN: track 0.00 -> 12.7 mm
- net RX3_B1_IN: track 0.00 -> 12.7 mm
Other:
- board text added: "​!! 100W RF WHEN TRANSMITTING !!"
- board text added: "​15/10m"
- board text added: "​160m"
- board text added: "​20/17m"
- board text added: "​40/30m"
- board text added: "​6m"
- board text added: "​80/60m"
- board text added: "​ANT 1"
- board text added: "​ANT 2"
- board text added: "​ANT 3"
- board text added: "​ANT 4"
- board text added: "​BYPASS"
- board text added: "​CHASSIS GND - THIS HOLE ONLY"
- board text added: "​CONTROL"
- board text added: "​CONTROL 2"
- board text added: "​RF FILTER BANK - 4 CH x 7 BANDS REV A"
- board text added: "​RX1 -> A"
- board text added: "​RX2 -> A"
- board text added: "​RX3 -> A"
- board text added: "​RX4 -> A"
- board text added: "​TO BOARD D"
- board text added: "​TX1 <- A"
- board text added: "​TX2 <- A"
- board text added: "​TX3 <- A"
- board text added: "​TX4 <- A"
