File: hardware/kicad/C_rf/01_power.kicad_sch (KiCad schematic)
At the start: 7 parts, among them U80 TPS62130

Commit message: Connect the pads that had no net
A symbol pin number must agree with the footprint pad number. If the
numbers do not agree, the net goes nowhere. The netlist removes it
and gives no message. ERC examines the schematic and sees a wire. DRC
does not count an unconnected pad as a violation. All three boards
showed zero ERC violations while 31 pads had no net.

Two of these faults stopped a board.

The footprint of the Ethernet PHY was for a different part. The
project used QFN-48 6x6 mm with 0.4 mm pitch. The RTL8211F(I)-CG is
WQFN-40-EP 5x5 mm. You cannot solder the part to that pad pattern.

The 25 MHz crystal had a 2-pin symbol on a 4-pad footprint. On a 3225
crystal the terminals are the diagonal pads 1 and 3. Pads 2 and 4 are
the metal can. XO went to pad 2. There was no crystal between XI and
XO, and thus neither PHY could make a clock.

The paddle of the AD9251 was pin 0 in the symbol and pad 65 in the
footprint. The paddle of the PE4312 was Pad against pad 21. The gas
discharge tubes had one electrode unconnected, because
Device:GDT_2Pin uses pins 1 and 3 but the varistor footprint uses
pads 1 and 2. A local footprint with pads 1 and 3 corrects this.

ped_denetim.py finds these faults on the board. yap.sh runs it before
the DSN export. The chain stops if a pad has no net.

The DSN export also changed. It declared In1 and In4 as power layers
but did not export the copper on them. The router thus believed that
the two ground planes were empty. It routed the 289 pins of GND as
traces on the signal layers. The planes now go out as conduction
areas.
Parts:
- removed U80: TPS62130, Package_DFN_QFN:VQFN-16-1EP_3x3mm_P0.5mm_EP1.68x1.68mm, symbol Regulator_Switching:TPS62130
- added C83: 10uF, Capacitor_SMD:C_1206_3216Metric, symbol Device:C
- added C84: 100nF, Capacitor_SMD:C_0603_1608Metric, symbol Device:C
- added U90: TPS62130, Package_DFN_QFN:VQFN-16-1EP_3x3mm_P0.5mm_EP1.68x1.68mm, symbol Regulator_Switching:TPS62130
Connections:
- net +5V: now also U90.14 (VOS)
- net GND: now also C83.2, C84.2, U90.15 (GND), U90.16 (GND), U90.17 (GND), U90.6 (GND), U90.7 (FSW), U90.8 (DEF)
- net VIN_PROT: now also C83.1, C84.1, U90.10 (VIN), U90.11 (VIN), U90.12 (VIN), U90.13 (EN)
- net at L80.1: now also U90.1 (SW), U90.2 (SW), U90.3 (SW)
- net FB_U80 renamed FB_U90
- net FB_U90: now also U90.5 (FB)
