File: hardware/kicad/C_rf/03_filter.kicad_sch (KiCad schematic)
At the start: 268 parts, among them K11 G6KU-2F-Y, K12 G6KU-2F-Y, K13 G6KU-2F-Y, K14 G6KU-2F-Y, K15 G6KU-2F-Y, K16 G6KU-2F-Y, K17 G6KU-2F-Y, K21 G6KU-2F-Y, K22 G6KU-2F-Y, K23 G6KU-2F-Y, K24 G6KU-2F-Y, K25 G6KU-2F-Y, K26 G6KU-2F-Y, K27 G6KU-2F-Y, K31 G6KU-2F-Y, K32 G6KU-2F-Y, K33 G6KU-2F-Y, K34 G6KU-2F-Y, K35 G6KU-2F-Y, K36 G6KU-2F-Y, K37 G6KU-2F-Y, K41 G6KU-2F-Y, K42 G6KU-2F-Y, K43 G6KU-2F-Y, K44 G6KU-2F-Y, K45 G6KU-2F-Y, K46 G6KU-2F-Y, K47 G6KU-2F-Y

Commit message: Replace the receive band filters: they passed nothing
Simulation in ngspice shows all six filter positions peak below the
band they must pass, with the band itself 24 to 41 dB down. The
receiver would have been deaf on every band. No connectivity check
can find this: the netlist is correct and the values are wrong.

The cause is arithmetic. The three resonators were tuned as bare LC
pairs, but the coupling capacitors sit in parallel with them and pull
the frequency down. On 160m, 430 pF of resonator plus 270 pF of end
coupling plus 62 pF between resonators gives 762 pF, and with 16 uH
that is 1.44 MHz against a band at 1.8 to 2.0 MHz.

Compensation alone is not sufficient. Top coupling is a narrowband
structure and these positions are wide: 80+60 m spans 3.5 to
5.4 MHz, or 44%.

The structure is now a ladder bandpass, shunt resonator then series
resonator then shunt resonator, synthesised from a 3-pole 0.1 dB
Chebyshev prototype and verified with the values snapped to E12.

  band      loss   worst band edge   was
  160m      1.31   -1.71             -34
  80_60m    0.52   -0.97             -25
  40_30m    0.73   -1.49             -27
  20_17m    0.83   -1.04             -32
  15_10m    0.71   -1.00             -28
  6m        1.72   -2.37             -41

Board C falls from 502 parts to 406. The inductors are all SMD: the
toroids gave a Q of 150 against 40, which is one decibel on 160m
where atmospheric noise sets the receiver's floor, and they were 48
parts that a machine cannot place.
Parts:
- removed C1000, C1060, C1120, C1180, C1181: 270pF, Capacitor_SMD:C_0603_1608Metric, symbol Device:C
- removed C1002, C1062, C1122, C1182, C1183: 62pF, Capacitor_SMD:C_0603_1608Metric, symbol Device:C
- removed C1010, C1070, C1130, C1190, C1191: 390pF, Capacitor_SMD:C_0603_1608Metric, symbol Device:C
- removed C1012, C1072, C1132, C1192, C1193: 82pF, Capacitor_SMD:C_0603_1608Metric, symbol Device:C
- removed C1020, C1080, C1140, C1200, C1201: 160pF, Capacitor_SMD:C_0603_1608Metric, symbol Device:C
- removed C1022, C1082, C1142, C1202, C1203: 33pF, Capacitor_SMD:C_0603_1608Metric, symbol Device:C
- removed C1030, C1090, C1150, C1151, C1210, C1211: 56pF, Capacitor_SMD:C_0603_1608Metric, symbol Device:C
- removed C1032, C1092, C1152, C1153, C1212, C1213: 13pF, Capacitor_SMD:C_0603_1608Metric, symbol Device:C
- removed C1040, C1100, C1160, C1161, C1220, C1221: 47pF, Capacitor_SMD:C_0603_1608Metric, symbol Device:C
- removed C1042, C1102, C1162, C1163, C1222, C1223: 10pF, Capacitor_SMD:C_0603_1608Metric, symbol Device:C
- removed C1050, C1110, C1170, C1171, C1230, C1231: 5.6pF, Capacitor_SMD:C_0603_1608Metric, symbol Device:C
- removed C1052, C1112, C1172, C1173, C1232, C1233: 1.3pF, Capacitor_SMD:C_0603_1608Metric, symbol Device:C
- removed C1145, C1147, C1149, C1205, C1207, C1209: 91pF, Capacitor_SMD:C_0603_1608Metric, symbol Device:C
- removed C1155, C1157, C1159, C1215, C1217, C1219: 51pF, Capacitor_SMD:C_0603_1608Metric, symbol Device:C
- removed C1165, C1167, C1169, C1225, C1227, C1229: 30pF, Capacitor_SMD:C_0603_1608Metric, symbol Device:C
- removed C1175, C1177, C1179, C1235, C1237, C1239: 15pF, Capacitor_SMD:C_0603_1608Metric, symbol Device:C
- removed C1185, C1187, C1189: 430pF, Capacitor_SMD:C_0603_1608Metric, symbol Device:C
- removed C1195, C1197, C1199: 180pF, Capacitor_SMD:C_0603_1608Metric, symbol Device:C
- removed L1144, L1146, L1148, L1204, L1206, L1208: 3.9uH, Inductor_SMD:L_0805_2012Metric, symbol Device:L
- removed L1154, L1156, L1158, L1214, L1216, L1218: 2uH, Inductor_SMD:L_0805_2012Metric, symbol Device:L
- removed L1164, L1166, L1168, L1224, L1226, L1228: 1.3uH, Inductor_SMD:L_0805_2012Metric, symbol Device:L
- removed L1174, L1176, L1178, L1234, L1236, L1238: 620nH, dogrudan-sdr:L_Toroid_T50_Vertical, symbol Device:L
- removed L1184, L1186, L1188: 16uH, dogrudan-sdr:L_Toroid_T50_Vertical, symbol Device:L
- removed L1194, L1196, L1198: 7.5uH, Inductor_SMD:L_0805_2012Metric, symbol Device:L
- added L1000, L1002, L1042, L1072, L1080, L1110: 1uH, dogrudan-sdr:L_Toroid_T50_Vertical, symbol Device:L
- added L1010, L1082: 3.3uH, dogrudan-sdr:L_Toroid_T50_Vertical, symbol Device:L
- added L1012, L1050, L1120, L1122: 470nH, dogrudan-sdr:L_Toroid_T50_Vertical, symbol Device:L
- added L1020, L1090, L1092: 220nH, Inductor_SMD:L_0805_2012Metric, symbol Device:L
- added L1022, L1130: 1.5uH, Inductor_SMD:L_0805_2012Metric, symbol Device:L
- added L1030, L1032, L1102, L1140: 33nH, Inductor_SMD:L_0805_2012Metric, symbol Device:L
- added L1040, L1112: 18uH, dogrudan-sdr:L_Toroid_T50_Vertical, symbol Device:L
- added L1052: 2.2uH, dogrudan-sdr:L_Toroid_T50_Vertical, symbol Device:L
- added L1060, L1062, L1132: 150nH, Inductor_SMD:L_0805_2012Metric, symbol Device:L
- added L1070, L1142: 820nH, Inductor_SMD:L_0805_2012Metric, symbol Device:L
- added L1100: 680nH, Inductor_SMD:L_0805_2012Metric, symbol Device:L
- C1001: value 270pF -> 6800pF
- C1003: value 62pF -> 6800pF
- C1005: value 430pF -> 390pF
- C1007, C1009: value 430pF -> 1200pF
- C1013: value 82pF -> 680pF
- C1015: value 180pF -> 680pF
- C1019: value 180pF -> 470pF
- C1021: value 160pF -> 470pF
- C1023: value 33pF -> 68pF
- C1025, C1027: value 91pF -> 270pF
- C1029: value 91pF -> 56pF
- C1031: value 56pF -> 270pF
- C1033: value 13pF -> 270pF
- C1035: value 51pF -> 12pF
- C1037, C1039: value 51pF -> 6800pF
- C1041: value 47pF -> 390pF
- C1043: value 10pF -> 1200pF
- C1045: value 30pF -> 1200pF
- C1047: value 30pF -> 390pF
- C1049: value 30pF -> 680pF
- C1051: value 5.6pF -> 680pF
- C1053: value 1.3pF -> 180pF
- C1055, C1057: value 15pF -> 470pF
- C1059: value 15pF -> 68pF
- C1063: value 62pF -> 270pF
- C1065: value 430pF -> 56pF
- C1067, C1069: value 430pF -> 270pF
- C1071: value 390pF -> 12pF
- C1073: value 82pF -> 6800pF
- C1075: value 180pF -> 6800pF
- C1077: value 180pF -> 390pF
- C1079: value 180pF -> 1200pF
- C1081: value 160pF -> 1200pF
- C1083: value 33pF -> 390pF
- C1085, C1087: value 91pF -> 680pF
- C1089: value 91pF -> 180pF
- C1091: value 56pF -> 470pF
- C1093: value 13pF -> 470pF
- C1095: value 51pF -> 68pF
- C1097, C1099: value 51pF -> 270pF
- C1101: value 47pF -> 56pF
- C1103: value 10pF -> 270pF
- C1105: value 30pF -> 270pF
- C1107: value 30pF -> 12pF
- C1109: value 30pF -> 6800pF
- C1111: value 5.6pF -> 6800pF
- C1113: value 1.3pF -> 390pF
- C1115, C1117: value 15pF -> 1200pF
- C1119: value 15pF -> 390pF
- C1121: value 270pF -> 680pF
- C1123: value 62pF -> 680pF
- C1125: value 430pF -> 180pF
- C1127, C1129: value 430pF -> 470pF
- C1131: value 390pF -> 68pF
- C1133: value 82pF -> 270pF
- C1135, C1139: value 180pF -> 270pF
- C1137: value 180pF -> 56pF
- C1141: value 160pF -> 270pF
- C1143: value 33pF -> 12pF
- L1004: value 16uH -> 18uH
- L1006, L1008: value 16uH -> 1uH
- L1014: value 7.5uH -> 470nH; footprint Inductor_SMD:L_0805_2012Metric -> dogrudan-sdr:L_Toroid_T50_Vertical
- L1016: value 7.5uH -> 2.2uH; footprint Inductor_SMD:L_0805_2012Metric -> dogrudan-sdr:L_Toroid_T50_Vertical
- L1018: value 7.5uH -> 220nH
- L1024, L1026: value 3.9uH -> 150nH
- L1028: value 3.9uH -> 680nH
- L1034: value 2uH -> 820nH
- L1036, L1038: value 2uH -> 1uH; footprint Inductor_SMD:L_0805_2012Metric -> dogrudan-sdr:L_Toroid_T50_Vertical
- L1044, L1108: value 1.3uH -> 1uH; footprint Inductor_SMD:L_0805_2012Metric -> dogrudan-sdr:L_Toroid_T50_Vertical
- L1046: value 1.3uH -> 3.3uH; footprint Inductor_SMD:L_0805_2012Metric -> dogrudan-sdr:L_Toroid_T50_Vertical
- L1048: value 1.3uH -> 470nH; footprint Inductor_SMD:L_0805_2012Metric -> dogrudan-sdr:L_Toroid_T50_Vertical
- L1054, L1056: value 620nH -> 220nH; footprint dogrudan-sdr:L_Toroid_T50_Vertical -> Inductor_SMD:L_0805_2012Metric
- L1058: value 620nH -> 1.5uH; footprint dogrudan-sdr:L_Toroid_T50_Vertical -> Inductor_SMD:L_0805_2012Metric
- L1064: value 16uH -> 680nH; footprint dogrudan-sdr:L_Toroid_T50_Vertical -> Inductor_SMD:L_0805_2012Metric
- L1066, L1068: value 16uH -> 33nH; footprint dogrudan-sdr:L_Toroid_T50_Vertical -> Inductor_SMD:L_0805_2012Metric
- L1074, L1078: value 7.5uH -> 1uH; footprint Inductor_SMD:L_0805_2012Metric -> dogrudan-sdr:L_Toroid_T50_Vertical
- L1076: value 7.5uH -> 18uH; footprint Inductor_SMD:L_0805_2012Metric -> dogrudan-sdr:L_Toroid_T50_Vertical
- L1084, L1086: value 3.9uH -> 470nH; footprint Inductor_SMD:L_0805_2012Metric -> dogrudan-sdr:L_Toroid_T50_Vertical
- L1088: value 3.9uH -> 2.2uH; footprint Inductor_SMD:L_0805_2012Metric -> dogrudan-sdr:L_Toroid_T50_Vertical
- L1094: value 2uH -> 1.5uH
- L1096, L1098: value 2uH -> 150nH
- L1104: value 1.3uH -> 33nH
- L1106: value 1.3uH -> 820nH
- L1114, L1116: value 620nH -> 1uH
- L1118: value 620nH -> 3.3uH
- L1124: value 16uH -> 2.2uH
- L1126, L1128: value 16uH -> 220nH; footprint dogrudan-sdr:L_Toroid_T50_Vertical -> Inductor_SMD:L_0805_2012Metric
- L1134: value 7.5uH -> 150nH
- L1136: value 7.5uH -> 680nH
- L1138: value 7.5uH -> 33nH
Connections:
- net N12_1 is gone; now on net F13_B: C1015.1, L1014.1
- net N13_1 is gone; now on net F15_A: C1025.1, L1024.1
- net N15_1 is gone; now on net F22_B: C1045.1, L1044.1
- net N16_1 is gone; now on net F24_A: C1055.1, L1054.1
- net N22_1 is gone; now on net F31_B: C1075.1, L1074.1
- net N23_1 is gone; now on net F33_A: C1085.1, L1084.1
- net N25_1 is gone; now on net F36_B: C1105.1, L1104.1
- net N26_1 is gone; now on net F42_A: C1115.1, L1114.1
- net N32_1 is gone; now on net F45_B: C1135.1, L1134.1
- net N33_3 is gone; now on net F46_B: C1141.1, C1143.2
- net F11_A: now also C1001.1, L1004.1, L1000.1
- net F11_B: now also C1003.1, C1005.2, L1002.1; no longer C1001.2
- net F12_A: now also C1007.1, L1006.1, L1010.1
- net F12_B: now also C1009.1, L1008.1
- net F13_A: now also C1013.1, L1016.1, L1012.1
- net F13_B: now also C1017.2; no longer C1021.2
- net F14_A: now also C1019.1, L1018.1, L1022.1
- net F14_B: now also C1021.1, C1023.2, L1020.1; no longer C1031.2
- net F15_A: now also L1028.1
- net F15_B: now also C1027.1, C1029.2, L1026.1; no longer C1041.2
- net F16_A: now also C1031.1, L1034.1, L1030.1
- net F16_B: now also C1033.1, C1035.2, L1032.1; no longer C1051.2
- net F21_A: now also C1037.1, L1036.1, L1040.1
- net F21_B: now also C1039.1, C1041.2, L1038.1; no longer C1061.2
- net F22_A: now also C1043.1, L1046.1, L1042.1
- net F22_B: now also C1047.2; no longer C1071.2
- net F23_A: now also C1049.1, L1048.1, L1052.1
- net F23_B: now also C1051.1, C1053.2, L1050.1; no longer C1081.2
- net F24_A: now also L1058.1
- net F24_B: now also C1057.1, C1059.2, L1056.1; no longer C1091.2
- net F25_A: now also C1061.1, L1064.1, L1060.1
- net F25_B: now also C1063.1, C1065.2, L1062.1; no longer C1101.2
- net F26_A: now also C1067.1, L1066.1, L1070.1
- net F26_B: now also C1069.1, C1071.2, L1068.1; no longer C1111.2
- net F31_A: now also C1073.1, L1076.1, L1072.1
- net F31_B: now also C1077.2; no longer C1121.2
- net F32_A: now also C1079.1, L1078.1, L1082.1
- net F32_B: now also C1081.1, C1083.2, L1080.1; no longer C1131.2
- net F33_A: now also L1088.1
- net F33_B: now also C1087.1, C1089.2, L1086.1; no longer C1141.2
- net F34_A: now also C1091.1, L1094.1, L1090.1
- net F34_B: now also C1093.1, C1095.2, L1092.1
- net F35_A: now also C1097.1, L1096.1, L1100.1
- net F35_B: now also C1099.1, C1101.2, L1098.1
- net F36_A: now also C1103.1, L1106.1, L1102.1
- net F36_B: now also C1107.2
- net F41_A: now also C1109.1, L1108.1, L1112.1
- net F41_B: now also C1111.1, C1113.2, L1110.1
- net F42_A: now also L1118.1
- net F42_B: now also C1117.1, C1119.2, L1116.1
- net F43_A: now also C1121.1, L1124.1, L1120.1
- net F43_B: now also C1123.1, C1125.2, L1122.1
- net F44_A: now also C1127.1, L1126.1, L1130.1
- net F44_B: now also C1129.1, C1131.2, L1128.1
- net F45_A: now also C1133.1, L1136.1, L1132.1
- net F45_B: now also C1137.2
- net F46_A: now also C1139.1, L1138.1, L1142.1
- net F46_B: now also L1140.1
- net GND: now also C1001.2, C1003.2, C1013.2, C1021.2, C1031.2, C1033.2, C1043.2, C1051.2, C1061.2, C1063.2, C1073.2, C1081.2, C1091.2, C1093.2, C1103.2, C1111.2, C1121.2, C1123.2, C1133.2, C1141.2, L1000.2, L1002.2, L1012.2, L1020.2, L1030.2, L1032.2, L1042.2, L1050.2, L1060.2, L1062.2, L1072.2, L1080.2, L1090.2, L1092.2, L1102.2, L1110.2, L1120.2, L1122.2, L1132.2, L1140.2; no longer C1005.2, C1017.2, C1029.2, C1035.2, C1047.2, C1059.2, C1065.2, C1077.2, C1089.2, C1095.2, C1107.2, C1119.2, C1125.2, C1137.2, L1004.2, L1016.2, L1028.2, L1034.2, L1046.2, L1058.2, L1064.2, L1076.2, L1088.2, L1094.2, L1106.2, L1118.2, L1124.2, L1136.2
- net N11_1 renamed N11_S
- net N11_S: now also L1004.2; no longer L1004.1
- removed net N11_2: C1003.1, C1007.1, L1006.1
- removed net N11_3: C1001.1, C1003.2, C1009.1, L1008.1
- removed net N12_2: C1013.1, C1017.1, L1016.1
- removed net N12_3: C1011.1, C1013.2, C1019.1, L1018.1
- removed net N13_2: C1023.1, C1027.1, L1026.1
- removed net N13_3: C1021.1, C1023.2, C1029.1, L1028.1
- net N14_1 renamed N16_S
- net N16_S: now also L1034.2; no longer L1034.1
- removed net N14_2: C1033.1, C1037.1, L1036.1
- removed net N14_3: C1031.1, C1033.2, C1039.1, L1038.1
- removed net N15_2: C1043.1, C1047.1, L1046.1
- removed net N15_3: C1041.1, C1043.2, C1049.1, L1048.1
- removed net N16_2: C1053.1, C1057.1, L1056.1
- removed net N16_3: C1051.1, C1053.2, C1059.1, L1058.1
- net N21_1 renamed N25_S
- net N25_S: now also L1064.2; no longer L1064.1
- removed net N21_2: C1063.1, C1067.1, L1066.1
- removed net N21_3: C1061.1, C1063.2, C1069.1, L1068.1
- removed net N22_2: C1073.1, C1077.1, L1076.1
- removed net N22_3: C1071.1, C1073.2, C1079.1, L1078.1
- removed net N23_2: C1083.1, C1087.1, L1086.1
- removed net N23_3: C1081.1, C1083.2, C1089.1, L1088.1
- net N24_1 renamed N34_S
- net N34_S: now also L1094.2; no longer L1094.1
- removed net N24_2: C1093.1, C1097.1, L1096.1
- removed net N24_3: C1091.1, C1093.2, C1099.1, L1098.1
- removed net N25_2: C1103.1, C1107.1, L1106.1
- removed net N25_3: C1101.1, C1103.2, C1109.1, L1108.1
- removed net N26_2: C1113.1, C1117.1, L1116.1
- removed net N26_3: C1111.1, C1113.2, C1119.1, L1118.1
- net N31_1 renamed N43_S
- net N43_S: now also L1124.2; no longer L1124.1
- removed net N31_2: C1123.1, C1127.1, L1126.1
- removed net N31_3: C1121.1, C1123.2, C1129.1, L1128.1
- removed net N32_2: C1133.1, C1137.1, L1136.1
- removed net N32_3: C1131.1, C1133.2, C1139.1, L1138.1
- net N33_2 renamed N46_S
- net N46_S: now also L1142.2
- new net N12_S: C1011.1, L1010.2
- new net N13_S: C1017.1, L1016.2
- new net N14_S: C1023.1, L1022.2
- new net N15_S: C1029.1, L1028.2
- new net N21_S: C1041.1, L1040.2
- new net N22_S: C1047.1, L1046.2
- new net N23_S: C1053.1, L1052.2
- new net N24_S: C1059.1, L1058.2
- new net N26_S: C1071.1, L1070.2
- new net N31_S: C1077.1, L1076.2
- new net N32_S: C1083.1, L1082.2
- new net N33_S: C1089.1, L1088.2
- new net N35_S: C1101.1, L1100.2
- new net N36_S: C1107.1, L1106.2
- new net N41_S: C1113.1, L1112.2
- new net N42_S: C1119.1, L1118.2
- new net N44_S: C1131.1, L1130.2
- new net N45_S: C1137.1, L1136.2

Commit message: Fit the filter bank and clear the overlaps
Board D's filter bank needs 285.6 mm of width with both inductors of
each band side by side, against about 236 mm available. Stacking them
vertically corrects the width and breaks the height: the strip
between the driver transformer and the relay row is 15.8 mm and a
stacked pair of T68 cores needs 37.7 mm.

Mapping the board in 10 mm bands gave the answer. Everything below
the relay row is the coupler and detector block at x above 250, while
the filter columns run from x 4 to 236. The space under them was
empty. The relay row moves from y 130 to 142 and its drivers from 155
to 172, with the filter block following. No board grew and the chain
stays in one row.

The separator never moves a part whose reference begins with U, J, T,
Y, L, Q, K or H, so two such parts overlapping cannot be separated
and the fix belongs in the placement rules. On A the XT60's courtyard
is 22.4 mm tall and snapped to the top edge, so it covered the
reverse-polarity MOSFET; the crystals and their inductors were placed
by the fallback and landed inside the PHY. All three now have
explicit positions.

The separator also gained a last resort: a movable part wedged so
that every push lands it in another part is relocated to the nearest
free position.

All three boards are at zero overlaps.
Parts:
- L1000, L1002, L1004, L1006, L1008, L1010, L1012, L1014, L1016, L1036, L1038, L1040, L1042, L1044, L1046, L1048, L1050, L1052, L1072, L1074, L1076, L1078, L1080, L1082, L1084, L1086, L1088, L1108, L1110, L1112, L1114, L1116, L1118, L1120, L1122, L1124: footprint dogrudan-sdr:L_Toroid_T50_Vertical -> Inductor_SMD:L_0805_2012Metric
