File: hardware/kicad/C_rf/03_filter.kicad_sch (KiCad schematic)
At the start: 172 parts, among them K11 G6KU-2F-Y, K12 G6KU-2F-Y, K13 G6KU-2F-Y, K14 G6KU-2F-Y, K15 G6KU-2F-Y, K16 G6KU-2F-Y, K17 G6KU-2F-Y, K21 G6KU-2F-Y, K22 G6KU-2F-Y, K23 G6KU-2F-Y, K24 G6KU-2F-Y, K25 G6KU-2F-Y, K26 G6KU-2F-Y, K27 G6KU-2F-Y, K31 G6KU-2F-Y, K32 G6KU-2F-Y, K33 G6KU-2F-Y, K34 G6KU-2F-Y, K35 G6KU-2F-Y, K36 G6KU-2F-Y, K37 G6KU-2F-Y, K41 G6KU-2F-Y, K42 G6KU-2F-Y, K43 G6KU-2F-Y, K44 G6KU-2F-Y, K45 G6KU-2F-Y, K46 G6KU-2F-Y, K47 G6KU-2F-Y

Commit message: Name the copyright holder and stamp it into the generated files
The repository had three licence files and no statement of who owns
the work. The only record of authorship was the git author field.

Copyleft depends on that statement. GPL and CERN-OHL-S work because
the holder grants permission on condition of reciprocity; with no
holder named there is nobody to require it from a downstream user.
Naming the author keeps the design open rather than closing it.

kicad/telif.py is the single source. The line reaches the schematics
through their title block and not through the generators, because
every schematic file is rewritten on each build and a header placed in
a generator would disappear at the first regeneration. All 23
schematics carry it. 109 source files have SPDX headers, split by the
project's own table: generators and the layout chain are hardware
under CERN-OHL-S-2.0, HDL and the audit tools are software under
GPL-3.0-only.

Board C's inductors also move to footprints that match parts that can
be bought. All of them sat on 0805 pads. Of the values this design
needs, 33 to 220 nH are 0603 parts, 470 and 820 nH are 0805, and
everything from 1000 nH upward is 1210, which is 3.2 by 2.5 mm and
does not fit an 0805 land. 32 inductors could not have been soldered.

A symbol-against-footprint check cannot find this. Those two agreed
with each other; what was wrong was the body size of the real part
behind the footprint.
Parts:
- L1000, L1002, L1004, L1006, L1008, L1010, L1016, L1022, L1028, L1034, L1036, L1038, L1040, L1042, L1044, L1046, L1052, L1058, L1064, L1070, L1072, L1074, L1076, L1078, L1080, L1082, L1088, L1094, L1100, L1106, L1108, L1110, L1112, L1114, L1116, L1118, L1124, L1130, L1136, L1142: footprint Inductor_SMD:L_0805_2012Metric -> Inductor_SMD:L_1210_3225Metric
- L1018, L1020, L1024, L1026, L1030, L1032, L1054, L1056, L1060, L1062, L1066, L1068, L1090, L1092, L1096, L1098, L1102, L1104, L1126, L1128, L1132, L1134, L1138, L1140: footprint Inductor_SMD:L_0805_2012Metric -> Inductor_SMD:L_0603_1608Metric

Commit message: Add a transmission zero to two preselector positions
The receiver samples at 80 MSPS. Nyquist is 40 MHz. A signal above
40 MHz folds onto the band as |f - 80|. After the fold, the receiver
cannot tell it from the wanted signal. Digital processing cannot
remove it. The preselector is the only protection.

A new tool measures the full chain. It goes from the antenna to the
ADC pin. It includes the attenuator, the transformer, the series
resistors and the ADC input capacitance. A filter alone gives the
wrong answer, because each block sees the impedance of its neighbour.

The tool found two weak bands:

  15 m to 10 m   50.3 MHz folds onto 29.7 MHz    24 dB
  6 m            30.0 MHz folds onto 50.0 MHz    36 dB

The first one is serious. 50.3 MHz is inside the 6 m band. If the
station transmits on 6 m, the signal lands on the 10 m receiver.

The two problems need different solutions. On 15 m to 10 m the
interference is above the band. A capacitor across the series
inductor puts a zero there. On 6 m the interference is below the
band. A series-arm trap cannot help, because it always puts the zero
above the passband. A capacitor in series with the shunt inductor
gives a zero below the band.

A search program found the values. It is not possible to calculate
them: a new zero also changes the passband. The program examines all
values together against two limits. It uses an analytical model, and
then ngspice confirms the result.

  15 m to 10 m   24 dB to 55 dB    loss 2.63 dB to 2.39 dB
  6 m            36 dB to 68 dB    loss 5.45 dB to 3.73 dB

The chain tool now reads the filter table from the generator. A
manual copy caused a fault before: a verification tool measured an
old design that the board no longer had.
Parts:
- removed C1031, C1061, C1063, C1067, C1133, C1135, C1139, C1141: 270pF, Capacitor_SMD:C_0603_1608Metric, symbol Device:C
- removed C1037, C1039, C1073, C1109: 6800pF, Capacitor_SMD:C_0603_1608Metric, symbol Device:C
- removed C1041, C1047, C1119: 390pF, Capacitor_SMD:C_0603_1608Metric, symbol Device:C
- removed C1043, C1045, C1115, C1117: 1200pF, Capacitor_SMD:C_0603_1608Metric, symbol Device:C
- removed C1049, C1051, C1121, C1123: 680pF, Capacitor_SMD:C_0603_1608Metric, symbol Device:C
- removed C1053, C1125: 180pF, Capacitor_SMD:C_0603_1608Metric, symbol Device:C
- removed C1055, C1057, C1127, C1129: 470pF, Capacitor_SMD:C_0603_1608Metric, symbol Device:C
- removed C1059, C1131: 68pF, Capacitor_SMD:C_0603_1608Metric, symbol Device:C
- removed C1065, C1137: 56pF, Capacitor_SMD:C_0603_1608Metric, symbol Device:C
- removed C1143: 12pF, Capacitor_SMD:C_0603_1608Metric, symbol Device:C
- removed L1030, L1032, L1066, L1068, L1138, L1140: 33nH, Inductor_SMD:L_0603_1608Metric, symbol Device:L
- removed L1036, L1038, L1042, L1044, L1072, L1074, L1108, L1110, L1114, L1116: 1uH, Inductor_SMD:L_1210_3225Metric, symbol Device:L
- removed L1040: 18uH, Inductor_SMD:L_1210_3225Metric, symbol Device:L
- removed L1046, L1118: 3.3uH, Inductor_SMD:L_1210_3225Metric, symbol Device:L
- removed L1048, L1050, L1120, L1122: 470nH, Inductor_SMD:L_0805_2012Metric, symbol Device:L
- removed L1052, L1124: 2.2uH, Inductor_SMD:L_1210_3225Metric, symbol Device:L
- removed L1054, L1056, L1126, L1128: 220nH, Inductor_SMD:L_0603_1608Metric, symbol Device:L
- removed L1058, L1130: 1.5uH, Inductor_SMD:L_1210_3225Metric, symbol Device:L
- removed L1060, L1062, L1132, L1134: 150nH, Inductor_SMD:L_0603_1608Metric, symbol Device:L
- removed L1064, L1136: 680nH, Inductor_SMD:L_1210_3225Metric, symbol Device:L
- removed L1142: 820nH, Inductor_SMD:L_1210_3225Metric, symbol Device:L
- added C1030, C1108, C1147: 15pF, Capacitor_SMD:C_0603_1608Metric, symbol Device:C
- added C1032, C1046, C1048, C1074, C1110, C1124, C1126, C1149, C1152: 1200pF, Capacitor_SMD:C_0603_1608Metric, symbol Device:C
- added C1036, C1052, C1054, C1072, C1114, C1130, C1132, C1150, C1153: 680pF, Capacitor_SMD:C_0603_1608Metric, symbol Device:C
- added C1038, C1116, C1155: 8.2pF, Capacitor_SMD:C_0603_1608Metric, symbol Device:C
- added C1040, C1042, C1118, C1120: 6800pF, Capacitor_SMD:C_0603_1608Metric, symbol Device:C
- added C1044, C1050, C1122, C1128: 390pF, Capacitor_SMD:C_0603_1608Metric, symbol Device:C
- added C1056, C1134: 180pF, Capacitor_SMD:C_0603_1608Metric, symbol Device:C
- added C1058, C1060, C1136, C1138: 470pF, Capacitor_SMD:C_0603_1608Metric, symbol Device:C
- added C1062, C1140: 68pF, Capacitor_SMD:C_0603_1608Metric, symbol Device:C
- added C1064, C1066, C1142, C1144: 560pF, Capacitor_SMD:C_0603_1608Metric, symbol Device:C
- added C1068, C1146: 56pF, Capacitor_SMD:C_0603_1608Metric, symbol Device:C
- added L1031, L1073, L1109, L1148, L1151: 22nH, Inductor_SMD:L_0603_1608Metric, symbol Device:L
- added L1037, L1115, L1154: 1.2uH, Inductor_SMD:L_1210_3225Metric, symbol Device:L
- added L1039, L1041, L1045, L1047, L1117, L1119, L1123, L1125: 1uH, Inductor_SMD:L_1210_3225Metric, symbol Device:L
- added L1043, L1121: 18uH, Inductor_SMD:L_1210_3225Metric, symbol Device:L
- added L1049, L1127: 3.3uH, Inductor_SMD:L_1210_3225Metric, symbol Device:L
- added L1051, L1053, L1129, L1131: 470nH, Inductor_SMD:L_0805_2012Metric, symbol Device:L
- added L1055, L1133: 2.2uH, Inductor_SMD:L_1210_3225Metric, symbol Device:L
- added L1057, L1059, L1135, L1137: 220nH, Inductor_SMD:L_0603_1608Metric, symbol Device:L
- added L1061, L1139: 1.5uH, Inductor_SMD:L_1210_3225Metric, symbol Device:L
- added L1063, L1065, L1141, L1143: 82nH, Inductor_SMD:L_0603_1608Metric, symbol Device:L
- added L1067, L1145: 560nH, Inductor_SMD:L_0805_2012Metric, symbol Device:L
- C1025, C1027, C1103, C1105: value 270pF -> 560pF
- C1033: value 270pF -> 680pF
- C1035, C1071: value 12pF -> 1200pF
- C1069: value 270pF -> 15pF
- C1075, C1111: value 6800pF -> 680pF
- C1077: value 390pF -> 8.2pF
- C1079, C1081: value 1200pF -> 6800pF
- C1085, C1087: value 680pF -> 1200pF
- C1089: value 180pF -> 390pF
- C1091, C1093: value 470pF -> 680pF
- C1095: value 68pF -> 180pF
- C1097, C1099: value 270pF -> 470pF
- C1101: value 56pF -> 68pF
- C1107: value 12pF -> 56pF
- C1113: value 390pF -> 1200pF
- L1024, L1026: value 150nH -> 82nH
- L1028: value 680nH -> 560nH; footprint Inductor_SMD:L_1210_3225Metric -> Inductor_SMD:L_0805_2012Metric
- L1034, L1070: value 820nH -> 22nH; footprint Inductor_SMD:L_1210_3225Metric -> Inductor_SMD:L_0603_1608Metric
- L1076: value 18uH -> 1.2uH
- L1082: value 3.3uH -> 18uH
- L1084, L1086: value 470nH -> 1uH; footprint Inductor_SMD:L_0805_2012Metric -> Inductor_SMD:L_1210_3225Metric
- L1088: value 2.2uH -> 3.3uH
- L1090, L1092: value 220nH -> 470nH; footprint Inductor_SMD:L_0603_1608Metric -> Inductor_SMD:L_0805_2012Metric
- L1094: value 1.5uH -> 2.2uH
- L1096, L1098: value 150nH -> 220nH
- L1100: value 680nH -> 1.5uH
- L1102, L1104: value 33nH -> 82nH
- L1106: value 820nH -> 560nH; footprint Inductor_SMD:L_1210_3225Metric -> Inductor_SMD:L_0805_2012Metric
- L1112: value 18uH -> 22nH; footprint Inductor_SMD:L_1210_3225Metric -> Inductor_SMD:L_0603_1608Metric
Connections:
- net F15_A: now also C1030.1
- net F16_A: now also C1033.1, L1031.1, L1037.1; no longer L1034.1
- net F16_B: now also L1034.1, C1036.1, C1038.2; no longer C1033.1, C1035.2
- net F21_A: now also C1040.1, L1039.1, L1043.1
- net F21_B: now also C1042.1, C1044.2, L1041.1
- net F22_A: now also C1046.1, L1045.1, L1049.1
- net F22_B: now also C1048.1, C1050.2, L1047.1
- net F23_A: now also C1052.1, L1051.1, L1055.1
- net F23_B: now also C1054.1, C1056.2, L1053.1
- net F24_A: now also C1058.1, L1057.1, L1061.1
- net F24_B: now also C1060.1, C1062.2, L1059.1
- net F25_A: now also C1069.1, C1064.1, L1063.1, L1067.1
- net F25_B: now also C1066.1, C1068.2, L1065.1
- net F26_A: now also L1076.1, C1072.1
- net F26_B: now also C1075.1, C1077.2, L1073.1; no longer C1069.1, C1071.2
- net F31_A: now also C1079.1, L1078.1, L1082.1; no longer L1076.1
- net F31_B: now also C1081.1, C1083.2, L1080.1; no longer C1075.1, C1077.2
- net F32_A: now also C1085.1, L1084.1, L1088.1; no longer C1079.1, L1078.1, L1082.1
- net F32_B: now also C1087.1, C1089.2, L1086.1; no longer C1081.1, C1083.2, L1080.1
- net F33_A: now also C1091.1, L1090.1, L1094.1; no longer C1085.1, L1084.1, L1088.1
- net F33_B: now also C1093.1, C1095.2, L1092.1; no longer C1087.1, C1089.2, L1086.1
- net F34_A: now also C1097.1, L1096.1, L1100.1; no longer C1091.1, L1090.1, L1094.1
- net F34_B: now also C1099.1, C1101.2, L1098.1; no longer C1093.1, C1095.2, L1092.1
- net F35_A: now also C1103.1, L1102.1, L1106.1, C1108.1; no longer C1097.1, L1096.1, L1100.1
- net F35_B: now also C1105.1, C1107.2, L1104.1; no longer C1099.1, C1101.2, L1098.1
- net F36_A: now also C1111.1, L1109.1, L1115.1; no longer C1103.1, L1102.1, L1106.1
- net F36_B: now also L1112.1, C1114.1, C1116.2; no longer C1105.1, C1107.2, L1104.1
- net F41_A: now also C1118.1, L1117.1, L1121.1; no longer L1112.1
- net F41_B: now also C1120.1, C1122.2, L1119.1; no longer C1111.1, C1113.2
- net F42_A: now also C1124.1, L1123.1, L1127.1
- net F42_B: now also C1126.1, C1128.2, L1125.1
- net F43_A: now also C1130.1, L1129.1, L1133.1
- net F43_B: now also C1132.1, C1134.2, L1131.1
- net F44_A: now also C1136.1, L1135.1, L1139.1
- net F44_B: now also C1138.1, C1140.2, L1137.1
- net F45_A: now also C1142.1, C1147.1, L1141.1, L1145.1
- net F45_B: now also C1144.1, C1146.2, L1143.1
- net F46_A: now also C1150.1, L1148.1, L1154.1
- net F46_B: now also C1153.1, C1155.2, L1151.1
- net GND: now also C1035.2, C1071.2, C1113.2, C1032.2, C1036.2, C1040.2, C1042.2, C1046.2, C1048.2, C1052.2, C1054.2, C1058.2, C1060.2, C1064.2, C1066.2, C1072.2, C1074.2, C1110.2, C1114.2, C1118.2, C1120.2, C1124.2, C1126.2, C1130.2, C1132.2, C1136.2, C1138.2, C1142.2, C1144.2, C1149.2, C1150.2, C1152.2, C1153.2, L1039.2, L1041.2, L1045.2, L1047.2, L1051.2, L1053.2, L1057.2, L1059.2, L1063.2, L1065.2, L1117.2, L1119.2, L1123.2, L1125.2, L1129.2, L1131.2, L1135.2, L1137.2, L1141.2, L1143.2; no longer C1069.2
- net N15_S: now also C1030.2
- net N16_S: now also C1038.1, L1037.2; no longer C1035.1, L1034.2
- net N21_S: now also C1044.1, L1043.2
- net N22_S: now also C1050.1, L1049.2
- net N23_S: now also C1056.1, L1055.2
- net N24_S: now also C1062.1, L1061.2
- net N25_S: now also C1069.2, C1068.1, L1067.2
- net N26_S: now also C1077.1, L1076.2; no longer C1071.1, L1070.2
- net N31_S: now also C1083.1, L1082.2; no longer C1077.1, L1076.2
- net N32_S: now also C1089.1, L1088.2; no longer C1083.1, L1082.2
- net N33_S: now also C1095.1, L1094.2; no longer C1089.1, L1088.2
- net N34_S: now also C1101.1, L1100.2; no longer C1095.1, L1094.2
- net N35_S: now also C1107.1, L1106.2, C1108.2; no longer C1101.1, L1100.2
- net N36_S: now also C1116.1, L1115.2; no longer C1107.1, L1106.2
- net N41_S: now also C1122.1, L1121.2; no longer C1113.1, L1112.2
- net N42_S: now also C1128.1, L1127.2
- net N43_S: now also C1134.1, L1133.2
- net N44_S: now also C1140.1, L1139.2
- net N45_S: now also C1146.1, C1147.2, L1145.2
- net N46_S: now also C1155.1, L1154.2
- new net X16A: C1032.1, L1031.2
- new net X16B: C1035.1, L1034.2
- new net X26A: C1071.1, L1070.2
- new net X26B: C1074.1, L1073.2
- new net X36A: C1110.1, L1109.2
- new net X36B: C1113.1, L1112.2
- new net X46A: C1149.1, L1148.2
- new net X46B: C1152.1, L1151.2

Commit message: Design for tolerance, not for nominal values
Every measurement until now used nominal component values, and all
six bands passed. But no component is nominal. A design that passes
at nominal values and fails in production is the most expensive kind
of fault, because it appears only after the boards arrive.

A new tool measures the same design with real parts: capacitors at
±5 %, inductors at ±5 %, temperature from −20 °C to +60 °C. It does
two things. Worst-case analysis puts every part at its worst end at
the same time. Monte Carlo gives the fraction of boards that pass.

The result was bad:

  6 m               54 % of boards pass, flatness 1.8 dB to 10.2 dB
  15 m to 10 m      77.5 %, flatness up to 6.3 dB

The cause is not a bad design. The band is narrow: 6 m is 50 MHz to
54 MHz, which is 7.7 % fractional bandwidth. A ±5 % tolerance moves
the resonance by about 5 %, and the band edge leaves the flat region.
A nominal measurement cannot show this.

A sensitivity analysis showed that all six components matter on 6 m.
So no single value correction can solve it.

The solution is to design the filter for a band that is wider than
the necessary band, by the tolerance. The shift then keeps the band
inside the flat region.

  15 m to 10 m   alias rejection 54.7 dB to 51.3 dB, pass 77.5 % to 100 %
  6 m            alias rejection 68.6 dB to 55.6 dB, pass 54 % to 99.9 %

The nominal rejection decreased. The fraction of good boards
increased. The second number is the important one: a filter that
gives 68 dB at nominal values but fails half the boards does not beat
a filter that gives 55 dB and passes all of them.

Worst-case analysis also passes on all six bands now.

Two errors in the tool were corrected. The insertion-loss limit was
8.5 dB for all bands, and 160 m failed. That limit was arbitrary. The
sensitivity of a receiver comes from the noise floor, not from the
front-end loss, and at the low end of HF the atmosphere sets the
floor: ITU-R P.372 gives about 60 dB ab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
Parts:
- C1029, C1068, C1107, C1146: value 56pF -> 82pF
- C1030, C1069, C1108, C1147: value 15pF -> 22pF
- C1033, C1036, C1072, C1075, C1111, C1114, C1150, C1153: value 680pF -> 390pF
- C1038, C1077, C1116, C1155: value 8.2pF -> 12pF
- L1024, L1026, L1063, L1065, L1102, L1104, L1141, L1143: value 82nH -> 68nH
- L1028, L1067, L1106, L1145: value 560nH -> 390nH
- L1031, L1034, L1070, L1073, L1109, L1112, L1148, L1151: value 22nH -> 33nH
- L1037, L1076, L1115, L1154: value 1.2uH -> 820nH
