File: hardware/kicad/C_rf/04_atten.kicad_sch (KiCad schematic)
At the start: 36 parts, among them U40 PE4312C-Z, U41 PE4312C-Z, U42 PE4312C-Z, U43 PE4312C-Z

Commit message: Connect the pads that had no net
A symbol pin number must agree with the footprint pad number. If the
numbers do not agree, the net goes nowhere. The netlist removes it
and gives no message. ERC examines the schematic and sees a wire. DRC
does not count an unconnected pad as a violation. All three boards
showed zero ERC violations while 31 pads had no net.

Two of these faults stopped a board.

The footprint of the Ethernet PHY was for a different part. The
project used QFN-48 6x6 mm with 0.4 mm pitch. The RTL8211F(I)-CG is
WQFN-40-EP 5x5 mm. You cannot solder the part to that pad pattern.

The 25 MHz crystal had a 2-pin symbol on a 4-pad footprint. On a 3225
crystal the terminals are the diagonal pads 1 and 3. Pads 2 and 4 are
the metal can. XO went to pad 2. There was no crystal between XI and
XO, and thus neither PHY could make a clock.

The paddle of the AD9251 was pin 0 in the symbol and pad 65 in the
footprint. The paddle of the PE4312 was Pad against pad 21. The gas
discharge tubes had one electrode unconnected, because
Device:GDT_2Pin uses pins 1 and 3 but the varistor footprint uses
pads 1 and 2. A local footprint with pads 1 and 3 corrects this.

ped_denetim.py finds these faults on the board. yap.sh runs it before
the DSN export. The chain stops if a pad has no net.

The DSN export also changed. It declared In1 and In4 as power layers
but did not export the copper on them. The router thus believed that
the two ground planes were empty. It routed the 289 pins of GND as
traces on the signal layers. The planes now go out as conduction
areas.
Connections:
- net GND: now also U40.21 (GND), U41.21 (GND), U42.21 (GND), U43.21 (GND); no longer U40.Pad (GND), U41.Pad (GND), U42.Pad (GND), U43.Pad (GND)

Commit message: Remove the pads that have no copper from the DSN export
The router reported the same 220 clearance violations in each pass.
At the same time the number of unrouted connections decreased. The
violations were thus in the input and not in the routing.

The -1EP footprints of KiCad put four paste apertures on the exposed
pad. These apertures stop full paste coverage and they have no copper
layer. The DSN export put them on the top copper layer. The image of
U51 in the DSN had 21 pins: 17 correct pins and four unconnected
copper islands in the exposed pad. These islands are always in
conflict with the pad and they close the area below it.

The export now removes a pad that has no copper layer. The image of
U51 has 17 pins. The violations on board D decreased from 220 to 152.
Parts:
- removed C406, C414, C415, C422, C423, C430, C431: 100nF, Capacitor_SMD:C_0402_1005Metric, symbol Device:C
- removed R408, R416, R417, R425, R426: 10k, Resistor_SMD:R_0603_1608Metric, symbol Device:R
- added C408, C416, C417, C425, C426, C434, C435: 100nF, Capacitor_SMD:C_0402_1005Metric, symbol Device:C
- added R406, R414, R415, R422, R423, R430, R431, R432, R433: 10k, Resistor_SMD:R_0603_1608Metric, symbol Device:R
- U40, U41, U42, U43: footprint Package_DFN_QFN:QFN-20-1EP_4x4mm_P0.5mm_EP2.6x2.6mm_ThermalVias -> Package_DFN_QFN:TQFN-20-1EP_4x4mm_P0.5mm_EP2.1x2.1mm_ThermalVias
Connections:
- net +3V3: now also C408.1, C416.1, C417.1, C425.1, C426.1, C434.1, C435.1, R406.1, R414.1, R415.1, R422.1, R423.1, R430.1, R431.1, R432.1, R433.1; no longer R400.1, R409.1, R418.1, R427.1
- net ATT1_C0: now also R401.2; no longer R400.2
- net ATT1_C1: now also R402.2; no longer R401.2
- net ATT1_C2: now also R403.2; no longer R402.2
- net ATT1_C3: now also R404.2; no longer R403.2
- net ATT1_C4: now also R405.2; no longer R404.2
- net ATT1_C5: now also R406.2; no longer R405.2
- net ATT2_C0: now also R410.2
- net ATT2_C1: now also R411.2; no longer R409.2
- net ATT2_C2: now also R412.2; no longer R410.2
- net ATT2_C3: now also R413.2; no longer R411.2
- net ATT2_C4: now also R414.2; no longer R412.2
- net ATT2_C5: now also R415.2; no longer R413.2
- net ATT3_C0: now also R419.2
- net ATT3_C1: now also R420.2
- net ATT3_C2: now also R421.2; no longer R418.2
- net ATT3_C3: now also R422.2; no longer R419.2
- net ATT3_C4: now also R423.2; no longer R420.2
- net ATT3_C5: now also R424.2; no longer R421.2
- net ATT4_C0: now also R428.2; no longer R424.2
- net ATT4_C1: now also R429.2
- net ATT4_C2: now also R430.2
- net ATT4_C3: now also R431.2; no longer R427.2
- net ATT4_C4: now also R432.2; no longer R428.2
- net ATT4_C5: now also R433.2; no longer R429.2
- net ATT_DATA: now also R400.1, R409.1, R418.1, R427.1; no longer U40.3 (Data), U41.3 (Data), U42.3 (Data), U43.3 (Data)
- net GND: now also C408.2, C416.2, C417.2, C425.2, C426.2, C434.2, C435.2
- new net ATT1_DAT: R400.2, U40.3 (Data)
- new net ATT2_DAT: R409.2, U41.3 (Data)
- new net ATT3_DAT: R418.2, U42.3 (Data)
- new net ATT4_DAT: R427.2, U43.3 (Data)

Commit message: Correct the clearance test for the pre-routed traces
The clearance test used a circle for each pad. The radius was
max(width, height)/2. The corner of a rectangle is at
hypot(width, height)/2 from the center. The test thus made the pad
smaller than it is. On the 2.5 x 4.5 mm gate pad of a TO-247 the
difference is 2.250 mm against 2.574 mm.

The DRN_A trace was on the gate pad of Q10 with an overlap of 35 um.
This is a short circuit between the 50 V drain rail and the gate of a
100 W device. The search that finds the tee offset accepted this
route. The overlap is at a corner and 35 um wide. You cannot see it
on a plot.

The test now uses the real shape of the pad and the collision test of
pcbnew. It also uses the 300 um clearance and not only an overlap. A
trace that is 50 um from a pad is also not possible to manufacture.

Board D was built again. No trace is below 300 um and the smallest
gap is 0.537 mm. Boards A and C were correct.
Parts:
- U40, U41, U42, U43: footprint Package_DFN_QFN:TQFN-20-1EP_4x4mm_P0.5mm_EP2.1x2.1mm_ThermalVias -> Package_DFN_QFN:TQFN-20-1EP_4x4mm_P0.5mm_EP2.1x2.1mm
