File: hardware/kicad/C_rf/05_driver.kicad_sch (KiCad schematic)
At the start: 71 parts, among them U60 74HC595D, U61 74HC595D, U62 74HC595D, U63 74HC595D, U64 74HC595D, U65 74HC595D, U66 74HC595D, U70 DRV8833PWPR, U71 DRV8833PWPR, U72 DRV8833PWPR, U73 DRV8833PWPR, U74 DRV8833PWPR, U75 DRV8833PWPR, U76 DRV8833PWPR, U77 DRV8833PWPR, U78 DRV8833PWPR, U79 DRV8833PWPR, U80 DRV8833PWPR, U81 DRV8833PWPR, U82 DRV8833PWPR, U83 DRV8833PWPR

Commit message: Connect the pads that had no net
A symbol pin number must agree with the footprint pad number. If the
numbers do not agree, the net goes nowhere. The netlist removes it
and gives no message. ERC examines the schematic and sees a wire. DRC
does not count an unconnected pad as a violation. All three boards
showed zero ERC violations while 31 pads had no net.

Two of these faults stopped a board.

The footprint of the Ethernet PHY was for a different part. The
project used QFN-48 6x6 mm with 0.4 mm pitch. The RTL8211F(I)-CG is
WQFN-40-EP 5x5 mm. You cannot solder the part to that pad pattern.

The 25 MHz crystal had a 2-pin symbol on a 4-pad footprint. On a 3225
crystal the terminals are the diagonal pads 1 and 3. Pads 2 and 4 are
the metal can. XO went to pad 2. There was no crystal between XI and
XO, and thus neither PHY could make a clock.

The paddle of the AD9251 was pin 0 in the symbol and pad 65 in the
footprint. The paddle of the PE4312 was Pad against pad 21. The gas
discharge tubes had one electrode unconnected, because
Device:GDT_2Pin uses pins 1 and 3 but the varistor footprint uses
pads 1 and 2. A local footprint with pads 1 and 3 corrects this.

ped_denetim.py finds these faults on the board. yap.sh runs it before
the DSN export. The chain stops if a pad has no net.

The DSN export also changed. It declared In1 and In4 as power layers
but did not export the copper on them. The router thus believed that
the two ground planes were empty. It routed the 289 pins of GND as
traces on the signal layers. The planes now go out as conduction
areas.
Parts:
- added C651, C654: 100nF, Capacitor_SMD:C_0603_1608Metric, symbol Device:C
- added R649, R650, R652, R653: 0R, Resistor_SMD:R_0603_1608Metric, symbol Device:R
- added U84, U85: DRV8833PWPR, Package_SO:HTSSOP-16-1EP_4.4x5mm_P0.65mm_EP3.4x5mm_Mask2.46x2.31mm_ThermalVias, symbol Driver_Motor:DRV8833PWP
Connections:
- net +3V3: now also U84.1 (~{SLEEP}), U85.1 (~{SLEEP})
- net +5V: now also C651.1, C654.1, U84.12 (VM), U85.12 (VM)
- net GND: now also U73.10 (BIN2), U73.9 (BIN1), U77.10 (BIN2), U77.9 (BIN1), U81.10 (BIN2), U81.9 (BIN1), C651.2, C654.2, R649.2, R650.2, R652.2, R653.2, U84.13 (GND), U84.17 (GND), U85.10 (BIN2), U85.13 (GND), U85.17 (GND), U85.9 (BIN1)
- net K21_R: now also U74.4 (AOUT2); no longer U73.5 (BOUT2)
- net K21_S: now also U74.2 (AOUT1); no longer U73.7 (BOUT1)
- net K22_R: now also U74.5 (BOUT2); no longer U74.4 (AOUT2)
- net K22_S: now also U74.7 (BOUT1); no longer U74.2 (AOUT1)
- net K23_R: now also U75.4 (AOUT2); no longer U74.5 (BOUT2)
- net K23_S: now also U75.2 (AOUT1); no longer U74.7 (BOUT1)
- net K24_R: now also U75.5 (BOUT2); no longer U75.4 (AOUT2)
- net K24_S: now also U75.7 (BOUT1); no longer U75.2 (AOUT1)
- net K25_R: now also U76.4 (AOUT2); no longer U75.5 (BOUT2)
- net K25_S: now also U76.2 (AOUT1); no longer U75.7 (BOUT1)
- net K26_R: now also U76.5 (BOUT2); no longer U76.4 (AOUT2)
- net K26_S: now also U76.7 (BOUT1); no longer U76.2 (AOUT1)
- net K27_R: now also U77.4 (AOUT2); no longer U76.5 (BOUT2)
- net K27_S: now also U77.2 (AOUT1); no longer U76.7 (BOUT1)
- net K31_R: now also U78.4 (AOUT2); no longer U77.4 (AOUT2)
- net K31_S: now also U78.2 (AOUT1); no longer U77.2 (AOUT1)
- net K32_R: now also U78.5 (BOUT2); no longer U77.5 (BOUT2)
- net K32_S: now also U78.7 (BOUT1); no longer U77.7 (BOUT1)
- net K33_R: now also U79.4 (AOUT2); no longer U78.4 (AOUT2)
- net K33_S: now also U79.2 (AOUT1); no longer U78.2 (AOUT1)
- net K34_R: now also U79.5 (BOUT2); no longer U78.5 (BOUT2)
- net K34_S: now also U79.7 (BOUT1); no longer U78.7 (BOUT1)
- net K35_R: now also U80.4 (AOUT2); no longer U79.4 (AOUT2)
- net K35_S: now also U80.2 (AOUT1); no longer U79.2 (AOUT1)
- net K36_R: now also U80.5 (BOUT2); no longer U79.5 (BOUT2)
- net K36_S: now also U80.7 (BOUT1); no longer U79.7 (BOUT1)
- net K37_R: now also U81.4 (AOUT2); no longer U80.4 (AOUT2)
- net K37_S: now also U81.2 (AOUT1); no longer U80.2 (AOUT1)
- net K41_R: now also U82.4 (AOUT2); no longer U80.5 (BOUT2)
- net K41_S: now also U82.2 (AOUT1); no longer U80.7 (BOUT1)
- net K42_R: now also U82.5 (BOUT2); no longer U81.4 (AOUT2)
- net K42_S: now also U82.7 (BOUT1); no longer U81.2 (AOUT1)
- net K43_R: now also U83.4 (AOUT2); no longer U81.5 (BOUT2)
- net K43_S: now also U83.2 (AOUT1); no longer U81.7 (BOUT1)
- net K44_R: now also U83.5 (BOUT2); no longer U82.4 (AOUT2)
- net K44_S: now also U83.7 (BOUT1); no longer U82.2 (AOUT1)
- net K45_R: now also U84.4 (AOUT2); no longer U82.5 (BOUT2)
- net K45_S: now also U84.2 (AOUT1); no longer U82.7 (BOUT1)
- net K46_R: now also U84.5 (BOUT2); no longer U83.4 (AOUT2)
- net K46_S: now also U84.7 (BOUT1); no longer U83.2 (AOUT1)
- net K47_R: now also U85.4 (AOUT2); no longer U83.5 (BOUT2)
- net K47_S: now also U85.2 (AOUT1); no longer U83.7 (BOUT1)
- net Q14: now also U74.16 (AIN1); no longer U73.9 (BIN1)
- net Q15: now also U74.15 (AIN2); no longer U73.10 (BIN2)
- net Q16: now also U74.9 (BIN1); no longer U74.16 (AIN1)
- net Q17: now also U74.10 (BIN2); no longer U74.15 (AIN2)
- net Q18: now also U75.16 (AIN1); no longer U74.9 (BIN1)
- net Q19: now also U75.15 (AIN2); no longer U74.10 (BIN2)
- net Q20: now also U75.9 (BIN1); no longer U75.16 (AIN1)
- net Q21: now also U75.10 (BIN2); no longer U75.15 (AIN2)
- net Q22: now also U76.16 (AIN1); no longer U75.9 (BIN1)
- net Q23: now also U76.15 (AIN2); no longer U75.10 (BIN2)
- net Q24: now also U76.9 (BIN1); no longer U76.16 (AIN1)
- net Q25: now also U76.10 (BIN2); no longer U76.15 (AIN2)
- net Q26: now also U77.16 (AIN1); no longer U76.9 (BIN1)
- net Q27: now also U77.15 (AIN2); no longer U76.10 (BIN2)
- net Q28: now also U78.16 (AIN1); no longer U77.16 (AIN1)
- net Q29: now also U78.15 (AIN2); no longer U77.15 (AIN2)
- net Q30: now also U78.9 (BIN1); no longer U77.9 (BIN1)
- net Q31: now also U78.10 (BIN2); no longer U77.10 (BIN2)
- net Q32: now also U79.16 (AIN1); no longer U78.16 (AIN1)
- net Q33: now also U79.15 (AIN2); no longer U78.15 (AIN2)
- net Q34: now also U79.9 (BIN1); no longer U78.9 (BIN1)
- net Q35: now also U79.10 (BIN2); no longer U78.10 (BIN2)
- net Q36: now also U80.16 (AIN1); no longer U79.16 (AIN1)
- net Q37: now also U80.15 (AIN2); no longer U79.15 (AIN2)
- net Q38: now also U80.9 (BIN1); no longer U79.9 (BIN1)
- net Q39: now also U80.10 (BIN2); no longer U79.10 (BIN2)
- net Q40: now also U81.16 (AIN1); no longer U80.16 (AIN1)
- net Q41: now also U81.15 (AIN2); no longer U80.15 (AIN2)
- net Q42: now also U82.16 (AIN1); no longer U80.9 (BIN1)
- net Q43: now also U82.15 (AIN2); no longer U80.10 (BIN2)
- net Q44: now also U82.9 (BIN1); no longer U81.16 (AIN1)
- net Q45: now also U82.10 (BIN2); no longer U81.15 (AIN2)
- net Q46: now also U83.16 (AIN1); no longer U81.9 (BIN1)
- net Q47: now also U83.15 (AIN2); no longer U81.10 (BIN2)
- net Q48: now also U83.9 (BIN1); no longer U82.16 (AIN1)
- net Q49: now also U83.10 (BIN2); no longer U82.15 (AIN2)
- net Q50: now also U84.16 (AIN1); no longer U82.9 (BIN1)
- net Q51: now also U84.15 (AIN2); no longer U82.10 (BIN2)
- net Q52: now also U84.9 (BIN1); no longer U83.16 (AIN1)
- net Q53: now also U84.10 (BIN2); no longer U83.15 (AIN2)
- net Q54: now also U85.16 (AIN1); no longer U83.9 (BIN1)
- net Q55: now also U85.15 (AIN2); no longer U83.10 (BIN2)
- net RLY_FAULT: now also U84.8 (~{FAULT}), U85.8 (~{FAULT})
- new net U84_ISEN0: R649.1, U84.3 (AISEN)
- new net U84_ISEN1: R650.1, U84.6 (BISEN)
- new net U85_ISEN0: R652.1, U85.3 (AISEN)
- new net U85_ISEN1: R653.1, U85.6 (BISEN)
- no-connect marks 28 -> 40
Other:
- note added: "G6KU TEK SARIMLI kilitlenen: bobine verilen gerilimin YONU konumu belirliyor. Acik drenaj surucu (TPIC6B595) YETMEZ — akimi sadece bir yonde cekebilir. H koprusu sart. Zincir: A kartindan 3 hat -> 8 x 74HC595 (64 lojik cikis) 56 lojik -> 16 x DRV8833 (kanal basina dort) 28 H koprusu kanali -> 28 filtre rolesi 74HC595 yetiyor cunku bobin akimini DRV8833 veriyor; yazmacin surdugu sey sadece lojik g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"
- note removed: "G6KU TEK SARIMLI kilitlenen: bobine verilen gerilimin YONU konumu belirliyor. Acik drenaj surucu (TPIC6B595) YETMEZ — akimi sadece bir yonde cekebilir. H koprusu sart. Zincir: A kartindan 3 hat -> 8 x 74HC595 (64 lojik cikis) 56 lojik -> 14 x DRV8833 (her biri cift H koprusu) 28 H koprusu kanali -> 28 filtre rolesi 74HC595 yetiyor cunku bobin akimini DRV8833 veriyor; yazmacin surdugu sey sadece l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"

Commit message: Remove the pads that have no copper from the DSN export
The router reported the same 220 clearance violations in each pass.
At the same time the number of unrouted connections decreased. The
violations were thus in the input and not in the routing.

The -1EP footprints of KiCad put four paste apertures on the exposed
pad. These apertures stop full paste coverage and they have no copper
layer. The DSN export put them on the top copper layer. The image of
U51 in the DSN had 21 pins: 17 correct pins and four unconnected
copper islands in the exposed pad. These islands are always in
conflict with the pad and they close the area below it.

The export now removes a pad that has no copper layer. The image of
U51 has 17 pins. The violations on board D decreased from 220 to 152.
Parts:
- removed C612, C618, C627, C633, C642, C648: 100nF, Capacitor_SMD:C_0603_1608Metric, symbol Device:C
- removed R610, R611, R614, R616, R619, R620, R625, R626, R629, R631, R634, R635, R640, R641, R644, R646, R649, R650: 0R, Resistor_SMD:R_0603_1608Metric, symbol Device:R
- added C610, C620, C625, C635, C640, C650, C655, C660, C665, C670, C675, C680, C685: 2.2uF, Capacitor_SMD:C_0603_1608Metric, symbol Device:C
- added C611, C616, C626, C631, C641, C646, C656, C661, C666, C671, C676, C681, C686: 100nF, Capacitor_SMD:C_0603_1608Metric, symbol Device:C
- added C614, C619, C629, C634, C644, C649, C659, C664, C669, C674, C679, C684: 10nF, Capacitor_SMD:C_0603_1608Metric, symbol Device:C
- added R612, R618, R627, R633, R642, R648, R657, R658, R662, R663, R667, R668, R672, R673, R677, R678, R682, R683: 0R, Resistor_SMD:R_0603_1608Metric, symbol Device:R
- C609, C624, C639, C654: value 100nF -> 10nF
- C615, C630, C645: value 100nF -> 2.2uF
Connections:
- net +5V: now also C609.2, C624.2, C639.2, C654.2, C611.1, C614.2, C616.1, C619.2, C626.1, C629.2, C631.1, C634.2, C641.1, C644.2, C646.1, C649.2, C656.1, C659.2, C661.1, C664.2, C666.1, C669.2, C671.1, C674.2, C676.1, C679.2, C681.1, C684.2, C686.1; no longer C609.1, C615.1, C624.1, C630.1, C639.1, C645.1, C654.1
- net GND: now also C610.2, C611.2, C616.2, C620.2, C625.2, C626.2, C631.2, C635.2, C640.2, C641.2, C646.2, C650.2, C655.2, C656.2, C660.2, C661.2, C665.2, C666.2, C670.2, C671.2, C675.2, C676.2, C680.2, C681.2, C685.2, C686.2, R612.2, R618.2, R627.2, R633.2, R642.2, R648.2, R657.2, R658.2, R662.2, R663.2, R667.2, R668.2, R672.2, R673.2, R677.2, R678.2, R682.2, R683.2; no longer C609.2, C624.2, C639.2, C654.2
- net U71_ISEN0: now also R612.1
- net U71_ISEN1: now also R613.1
- net U72_ISEN0: now also R617.1; no longer R613.1
- net U72_ISEN1: now also R618.1
- net U73_ISEN0: now also R622.1
- net U73_ISEN1: now also R623.1; no longer R617.1
- net U74_ISEN0: now also R627.1
- net U74_ISEN1: now also R628.1
- net U75_ISEN0: now also R632.1; no longer R622.1
- net U75_ISEN1: now also R633.1; no longer R623.1
- net U76_ISEN0: now also R637.1
- net U76_ISEN1: now also R638.1
- net U77_ISEN0: now also R642.1; no longer R628.1
- net U77_ISEN1: now also R643.1
- net U78_ISEN0: now also R647.1
- net U78_ISEN1: now also R648.1; no longer R632.1
- net U79_ISEN0: now also R652.1
- net U79_ISEN1: now also R653.1
- net U80_ISEN0: now also R657.1; no longer R637.1
- net U80_ISEN1: now also R658.1; no longer R638.1
- net U81_ISEN0: now also R662.1
- net U81_ISEN1: now also R663.1
- net U82_ISEN0: now also R667.1; no longer R643.1
- net U82_ISEN1: now also R668.1
- net U83_ISEN0: now also R672.1
- net U83_ISEN1: now also R673.1; no longer R647.1
- net U84_ISEN0: now also R677.1
- net U84_ISEN1: now also R678.1
- net U85_ISEN0: now also R682.1; no longer R652.1
- net U85_ISEN1: now also R683.1; no longer R653.1
- net U70_VCP: now reaches U70.11 (VCP)
- net U70_VCP: now also C609.1
- net U70_VINT: now reaches U70.14 (VINT)
- net U70_VINT: now also C610.1
- net U81_VCP: now reaches U81.11 (VCP)
- net U81_VCP: now also C664.1
- net U81_VINT: now reaches U81.14 (VINT)
- net U81_VINT: now also C665.1
- net U72_VCP: now reaches U72.11 (VCP)
- net U72_VCP: now also C619.1
- net U72_VINT: now reaches U72.14 (VINT)
- net U72_VINT: now also C620.1
- net U85_VCP: now reaches U85.11 (VCP)
- net U85_VCP: now also C684.1
- net U85_VINT: now reaches U85.14 (VINT)
- net U85_VINT: now also C685.1
- net U75_VCP: now reaches U75.11 (VCP)
- net U75_VCP: now also C634.1
- net U75_VINT: now reaches U75.14 (VINT)
- net U75_VINT: now also C635.1
- net U74_VCP: now reaches U74.11 (VCP)
- net U74_VCP: now also C629.1
- net U74_VINT: now reaches U74.14 (VINT)
- net U74_VINT: now also C630.1
- net U73_VCP: now reaches U73.11 (VCP)
- net U73_VCP: now also C624.1
- net U73_VINT: now reaches U73.14 (VINT)
- net U73_VINT: now also C625.1
- net U78_VCP: now reaches U78.11 (VCP)
- net U78_VCP: now also C649.1
- net U78_VINT: now reaches U78.14 (VINT)
- net U78_VINT: now also C650.1
- net U77_VCP: now reaches U77.11 (VCP)
- net U77_VCP: now also C644.1
- net U77_VINT: now reaches U77.14 (VINT)
- net U77_VINT: now also C645.1
- net U80_VCP: now reaches U80.11 (VCP)
- net U80_VCP: now also C659.1
- net U80_VINT: now reaches U80.14 (VINT)
- net U80_VINT: now also C660.1
- net U83_VCP: now reaches U83.11 (VCP)
- net U83_VCP: now also C674.1
- net U83_VINT: now reaches U83.14 (VINT)
- net U83_VINT: now also C675.1
- net U71_VCP: now reaches U71.11 (VCP)
- net U71_VCP: now also C614.1
- net U71_VINT: now reaches U71.14 (VINT)
- net U71_VINT: now also C615.1
- net U84_VCP: now reaches U84.11 (VCP)
- net U84_VCP: now also C679.1
- net U84_VINT: now reaches U84.14 (VINT)
- net U84_VINT: now also C680.1
- net U82_VCP: now reaches U82.11 (VCP)
- net U82_VCP: now also C669.1
- net U82_VINT: now reaches U82.14 (VINT)
- net U82_VINT: now also C670.1
- net U79_VCP: now reaches U79.11 (VCP)
- net U79_VCP: now also C654.1
- net U79_VINT: now reaches U79.14 (VINT)
- net U79_VINT: now also C655.1
- net U76_VCP: now reaches U76.11 (VCP)
- net U76_VCP: now also C639.1
- net U76_VINT: now reaches U76.14 (VINT)
- net U76_VINT: now also C640.1
- no-connect marks 40 -> 8
Other:
- note added: "SARJ POMPASI VE IC REGULATOR KONDANSATORLERI — SURUCU BASINA IKI"
