File: hardware/kicad/D_pa/02_final.kicad_sch (KiCad schematic)
At the start: 24 parts, among them Q10 IRFP250N, Q11 IRFP250N, Q12 IRFP250N, Q13 IRFP250N, T10 BN43-202 3:1, T11 BN43-3312 2:4

Commit message: Connect the pads that had no net
A symbol pin number must agree with the footprint pad number. If the
numbers do not agree, the net goes nowhere. The netlist removes it
and gives no message. ERC examines the schematic and sees a wire. DRC
does not count an unconnected pad as a violation. All three boards
showed zero ERC violations while 31 pads had no net.

Two of these faults stopped a board.

The footprint of the Ethernet PHY was for a different part. The
project used QFN-48 6x6 mm with 0.4 mm pitch. The RTL8211F(I)-CG is
WQFN-40-EP 5x5 mm. You cannot solder the part to that pad pattern.

The 25 MHz crystal had a 2-pin symbol on a 4-pad footprint. On a 3225
crystal the terminals are the diagonal pads 1 and 3. Pads 2 and 4 are
the metal can. XO went to pad 2. There was no crystal between XI and
XO, and thus neither PHY could make a clock.

The paddle of the AD9251 was pin 0 in the symbol and pad 65 in the
footprint. The paddle of the PE4312 was Pad against pad 21. The gas
discharge tubes had one electrode unconnected, because
Device:GDT_2Pin uses pins 1 and 3 but the varistor footprint uses
pads 1 and 2. A local footprint with pads 1 and 3 corrects this.

ped_denetim.py finds these faults on the board. yap.sh runs it before
the DSN export. The chain stops if a pad has no net.

The DSN export also changed. It declared In1 and In4 as power layers
but did not export the copper on them. The router thus believed that
the two ground planes were empty. It routed the 289 pins of GND as
traces on the signal layers. The planes now go out as conduction
areas.
Parts:
- removed C210: 100nF, Capacitor_SMD:C_1206_3216Metric, symbol Device:C
- removed C211: 1uF, Capacitor_SMD:C_1206_3216Metric, symbol Device:C
- removed C212: 100uF, Capacitor_SMD:C_1206_3216Metric, symbol Device:C
- removed C214, C216: 1nF, Capacitor_SMD:C_1206_3216Metric, symbol Device:C
- removed L10: 10uH bogucu, dogrudan-sdr:L_Toroid_T50_Vertical, symbol Device:L
- removed R202, R204, R206, R208: 10R, Resistor_SMD:R_0603_1608Metric, symbol Device:R
- removed R203, R209: 1k, Resistor_SMD:R_0603_1608Metric, symbol Device:R
- removed R213, R215: 820R, Resistor_SMD:R_2512_6332Metric, symbol Device:R
- removed T10: BN43-202 3:1, dogrudan-sdr:XFMR_Toroid_4P_Vertical, symbol Device:Transformer_1P_1S
- removed T11: BN43-3312 2:4, dogrudan-sdr:XFMR_Toroid_4P_Vertical, symbol Device:Transformer_1P_1S
- added C202: 100nF, Capacitor_SMD:C_1206_3216Metric, symbol Device:C
- added C203: 1uF, Capacitor_SMD:C_1206_3216Metric, symbol Device:C
- added C204: 10uF, Capacitor_SMD:C_1206_3216Metric, symbol Device:C
- added C206, C208: 1nF, Capacitor_SMD:C_1206_3216Metric, symbol Device:C
- added C230, C231, C232, C233: 100nF, Capacitor_SMD:C_0603_1608Metric, symbol Device:C
- added L20: 10uH bogucu, dogrudan-sdr:L_Toroid_T50_Vertical, symbol Device:L
- added R240, R241, R242, R243: 10R, Resistor_SMD:R_0603_1608Metric, symbol Device:R
- added R244, R245, R246, R247: 1k, Resistor_SMD:R_0603_1608Metric, symbol Device:R
- added T30: BN43-202 3:1, dogrudan-sdr:XFMR_Toroid_4P_Vertical, symbol Device:Transformer_1P_1S
- added T31: BN43-3312 2:4 CT, dogrudan-sdr:XFMR_Toroid_5P_Vertical, symbol dogrudan-sdr:XFMR_CT
- R205, R207: value 1k -> 820R; footprint Resistor_SMD:R_0603_1608Metric -> Resistor_SMD:R_2512_6332Metric
Connections:
- net +50V: now also L20.1
- net DRN_A: now also R205.1, T31.1 (PRI_A)
- net DRN_B: now also R207.1, T31.2 (PRI_B)
- net DRN_CT: now also C202.1, C203.1, C204.1, L20.2, T31.5 (PRI_CT)
- net DRV_OUT: now also T30.1 (AA)
- net FB_A: now also R205.2, C206.1
- net FB_B: now also R207.2, C208.1
- net G10: now also R240.2, R244.2
- net G11: now also R241.2, R245.2; no longer R205.2
- net G12: now also R242.2, R246.2; no longer R207.2
- net G13: now also R243.2, R247.2
- net GATE1: now also R244.1
- net GATE2: now also R245.1; no longer R205.1
- net GATE3: now also R246.1; no longer R207.1
- net GATE4: now also R247.1
- net GIN_A: now also C206.2, C230.1, C231.1, T30.3 (SA)
- net GIN_B: now also C208.2, C232.1, C233.1, T30.4 (SB)
- net GND: now also C202.2, C203.2, C204.2, T30.2 (AB), T31.4 (SEC_B)
- net PA_OUT: now also T31.3 (SEC_A)
- new net GC10: C230.2, R240.1
- new net GC11: C231.2, R241.1
- new net GC12: C232.2, R242.1
- new net GC13: C233.2, R243.1
Other:
- note added: "SARIMLAR — manyetik_hesap.py T31 cikis: BN43-3312, birincil 2 sarim ORTA UCLU, ikincil 4. R_dd = Vcc^2/(2*Pout) = 12.5 ohm, yuk 50 -> 1:4 empedans. Sarim sayisi iki sarttan buyugu: endüktans (0.9) ve DOYMA (1.4). 2 sarimda B = 34.6 mT, ferrit-43'un 50 mT sinirinin altinda. Birincil akim 2.8 A rms -> AWG 18. IKI YARIM SARIM SIMETRIK: asimetri cift harmonik iptalini bozar, push-pull'un tek kazandir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"
- note removed: "SARIMLAR — manyetik_hesap.py T11 cikis: BN43-3312, birincil 2 sarim ORTA UCLU, ikincil 4. R_dd = Vcc^2/(2*Pout) = 12.5 ohm, yuk 50 -> 1:4 empedans. Sarim sayisi iki sarttan buyugu: endüktans (0.9) ve DOYMA (1.4). 2 sarimda B = 34.6 mT, ferrit-43'un 50 mT sinirinin altinda. Birincil akim 2.8 A rms -> AWG 18. IKI YARIM SARIM SIMETRIK: asimetri cift harmonik iptalini bozar, push-pull'un tek kazandir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"
