File: hardware/kicad/D_pa/05_lpf.kicad_sch (KiCad schematic)
At the start: 72 parts

Commit message: Correct the transmit envelope and add a third zero on 15 m to 10 m
The unit has no reconstruction filter. A comment on board A said that
the filter is on board C. Board C has no such filter: the transmit
signal enters through an SMA connector and goes to the transmit and
receive relay. The datasheet also gave a cutoff frequency for this
filter that does not exist.

A sampling DAC does not make one frequency. It makes images at
|k*fs +/- fd|. The zero-order hold gives each image a different
level, and the function falls slowly. If the carrier is near Nyquist,
an image at a lower frequency can be stronger than the carrier.

A new tool measures this. It uses the harmonic filter of board D,
because that filter is the only one in the transmit path.

  15 m to 10 m   4-channel   image at 10.3 MHz is 10.4 dB stronger
  6 m            4-channel   image is 14.2 dB stronger
  6 m            2-channel   image is 7.4 dB stronger
  20 m, 17 m     4-channel   -12.0 dBc, the limit is -43 dBc
  15 m to 10 m   2-channel   -40.4 dBc, the limit is -43 dBc

Only the last one is correctable.

That filter position must attenuate three frequencies: 42 MHz (the
second harmonic of 21 MHz), 63 MHz (the third harmonic) and 50.3 MHz
(the DAC image). A five-pole filter has two traps. No pair of trap
frequencies gives more than 1.9 dB of margin, and 1.9 dB is not a
margin: one E24 rounding already cost 19 dB in this project.

A shunt series-LC at the output adds a third zero. The image goes
from -40.4 dBc to -47.3 dBc, and the margin becomes 23 dB. Above
resonance the branch is capacitive and attenuates the whole stopband,
so the harmonics also improve. The passband loss falls from 1.35 dB
to 0.99 dB.

The transmit envelope is now written honestly. The RTL said "Nyquist
is 20 MHz, so 160 m to 17 m". Nyquist alone is not enough: the images
must also be filtered, and the real limit is lower.

  4-channel   160 m to 30 m
  2-channel   160 m to 10 m
  6 m         no transmit. Receive works, with 68 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
Parts:
- removed C554, C562: 62pF, Capacitor_THT:C_Disc_D7.5mm_W5.0mm_P5.00mm, symbol Device:C
- removed C558: 110pF, Capacitor_THT:C_Disc_D7.5mm_W5.0mm_P5.00mm, symbol Device:C
- removed L555, L559: T50-6 7s, dogrudan-sdr:L_Toroid_T50_Vertical, symbol Device:L
- added C555: 15pF, Capacitor_THT:C_Disc_D7.5mm_W5.0mm_P5.00mm, symbol Device:C
- added C559: 13pF, Capacitor_THT:C_Disc_D7.5mm_W5.0mm_P5.00mm, symbol Device:C
- added C563: 3.3pF, Capacitor_THT:C_Disc_D7.5mm_W5.0mm_P5.00mm, symbol Device:C
- added C564: 3pF, Capacitor_SMD:C_0603_1608Metric, symbol Device:C
- added C565: 62pF, Capacitor_THT:C_Disc_D7.5mm_W5.0mm_P5.00mm, symbol Device:C
- added L554: T50-6 10s, dogrudan-sdr:L_Toroid_T50_Vertical, symbol Device:L
- added L558, L562: T50-6 7s, dogrudan-sdr:L_Toroid_T50_Vertical, symbol Device:L
- C556: value 13pF -> 15pF; footprint Capacitor_THT:C_Disc_D7.5mm_W5.0mm_P5.00mm -> Capacitor_SMD:C_0603_1608Metric
- C557: value 1.1pF -> 62pF; footprint Capacitor_SMD:C_0603_1608Metric -> Capacitor_THT:C_Disc_D7.5mm_W5.0mm_P5.00mm
- C560: value 3.3pF -> 1.1pF; footprint Capacitor_THT:C_Disc_D7.5mm_W5.0mm_P5.00mm -> Capacitor_SMD:C_0603_1608Metric
- C561: value 3pF -> 110pF; footprint Capacitor_SMD:C_0603_1608Metric -> Capacitor_THT:C_Disc_D7.5mm_W5.0mm_P5.00mm
Connections:
- net GND: now also C556.2, C557.2, C561.2, C555.2, C565.2
- net LF6_B: now also L554.1
- net LF7_A: now also C560.1, C559.1, L558.1; no longer C556.1
- net LF7_B: now also C563.2, C564.2, C565.1, L562.2; no longer C560.2, C561.2
- net N7_1: now also C560.2, C559.2, C563.1, C564.1, L558.2, L562.1; no longer C556.2, C557.2, C560.1
- new net NCEN6: C555.1, C556.1, L554.2
