File: hardware/kicad/D_pa/dogrudan_sdr_D.kicad_pcb (KiCad board)
At the start: 2 copper layers, 240 x 185 mm, 187 parts, among them J10 A kartindan TX1, J20 DPD -> C karti, J30 50V giris, J31 A kartina, J32 C kartindan, J40 ANTEN -> panel SO-239, K20 G6K-2F-Y, Q10 IRFP250N, Q11 IRFP250N, Q12 IRFP250N, Q13 IRFP250N, Q20 IRF530N, Q21 IRF530N, Q30 IRF9540N, Q31 2N7002, Q32 2N7002, T10 BN43-202 3:1, T11 BN43-3312 2:4, T12 BN43-202 2:3, T20 FT50-43 1:32, T21 FT50-43 1:32, U10 PE4312C-Z, U11 PGA-103+, U20 MCP4922-E/SL, U21 MCP4922-E/SL, U30 AD8318ACPZ, U31 AD8318ACPZ, U32 INA240A1DR, U33 INA240A1DR, U34 INA240A1DR, U41 LM358, U42 LM358, U50 LM5164DDAR, U51 TPS62130, U55 MCP9700AT, U56 74HC595D, U57 MCP3208T-CI/SL

Commit message: Update the hardware tools and add the gateware
This commit makes the public tree equal to the development tree. The
public tree was behind. It did not have the verification tools, the
build chain, or the FPGA source.

The hardware/kicad directory now has the full tool chain. This
includes yap.sh, which runs the steps in the correct order, and the
tools that check the boards.

The gateware directory is new. It has the Verilog source for the
Lattice ECP5, the test benches, and the synthesis script. The
gateware does the four-channel receive chain, the transmit chain, the
packet interface, and the control interface.

The internal Turkish documents stay in the development tree. The
documentation in this repository is English. The comments in the
source code stay in Turkish.
Parts:
- added J33: sonraki PA, PinHeader_2x10_P2.54mm_Vertical, F.Cu at (136.0, 179.7)
- moved C611 212.9 mm to (35.4, 167.1)
- moved U33 177.6 mm to (52.0, 164.0)
- moved U32 172.2 mm to (30.0, 164.0)
- moved U34 171.5 mm to (74.0, 164.0)
- moved C612 148.9 mm to (57.4, 167.1)
- moved C624 128.1 mm to (122.2, 161.2)
- moved Q31 126.8 mm to (178.0, 164.0)
- moved R310 101.7 mm to (91.3, 130.8)
- moved R314 101.7 mm to (91.3, 134.0)
- moved U57 98.9 mm to (100.0, 164.0)
- moved U55 88.6 mm to (125.0, 164.0)
- moved R208 85.8 mm to (184.4, 17.0), turned to 90 degrees
- moved C216 80.6 mm to (155.3, 57.2)
- moved RS1 73.6 mm to (117.5, 24.0), turned to 90 degrees
- moved R206 72.7 mm to (164.4, 17.0), turned to 90 degrees
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Connections:
- U56 pad 9: unconnected-(U56-QH'-Pad9) -> RLY_SER_NEXT
Routing:
- net G13: track 0.00 -> 14.5 mm
- net G12: track 0.00 -> 14.5 mm
- net G11: track 0.00 -> 14.5 mm
- net G10: track 0.00 -> 14.5 mm
- net D2_GA_S: track 0.00 -> 12.3 mm
- net D2_GB_S: track 0.00 -> 12.3 mm

Commit message: Connect the pads that had no net
A symbol pin number must agree with the footprint pad number. If the
numbers do not agree, the net goes nowhere. The netlist removes it
and gives no message. ERC examines the schematic and sees a wire. DRC
does not count an unconnected pad as a violation. All three boards
showed zero ERC violations while 31 pads had no net.

Two of these faults stopped a board.

The footprint of the Ethernet PHY was for a different part. The
project used QFN-48 6x6 mm with 0.4 mm pitch. The RTL8211F(I)-CG is
WQFN-40-EP 5x5 mm. You cannot solder the part to that pad pattern.

The 25 MHz crystal had a 2-pin symbol on a 4-pad footprint. On a 3225
crystal the terminals are the diagonal pads 1 and 3. Pads 2 and 4 are
the metal can. XO went to pad 2. There was no crystal between XI and
XO, and thus neither PHY could make a clock.

The paddle of the AD9251 was pin 0 in the symbol and pad 65 in the
footprint. The paddle of the PE4312 was Pad against pad 21. The gas
discharge tubes had one electrode unconnected, because
Device:GDT_2Pin uses pins 1 and 3 but the varistor footprint uses
pads 1 and 2. A local footprint with pads 1 and 3 corrects this.

ped_denetim.py finds these faults on the board. yap.sh runs it before
the DSN export. The chain stops if a pad has no net.

The DSN export also changed. It declared In1 and In4 as power layers
but did not export the copper on them. The router thus believed that
the two ground planes were empty. It routed the 289 pins of GND as
traces on the signal layers. The planes now go out as conduction
areas.
Parts:
- removed C210: 100nF, C_1206_3216Metric
- removed C211: 1uF, C_1206_3216Metric
- removed C212: 100uF, C_1206_3216Metric
- removed C214, C216: 1nF, C_1206_3216Metric
- removed C603, C606, C612, C616, C624: 100nF, C_0603_1608Metric
- removed C605, C611: 22uF, C_0603_1608Metric
- removed D30: 15V, D_SOD-323
- removed D617, D618, D619, D620, D621, D622, D623: 1N4148WS, D_SOD-323
- removed R202, R204, R206, R208: 10R, R_0603_1608Metric
- removed R203, R209: 1k, R_0603_1608Metric
- removed R213, R215: 820R, R_2512_6332Metric
- removed R600, R613, R615: 100k, R_0603_1608Metric
- removed R607: 140k, R_0603_1608Metric
- removed R609: 105k, R_0603_1608Metric
- removed R610: 20k, R_0603_1608Metric
- removed T11: BN43-3312 2:4, XFMR_Toroid_4P_Vertical
- removed U30: AD8318ACPZ, NXP_VQFN-16-1EP_4x4mm_P0.65mm_EP2.1x2.1mm
- added C202: 100nF, C_1206_3216Metric, F.Cu at (140.7, 56.4)
- added C203: 1uF, C_1206_3216Metric, F.Cu at (140.9, 52.6)
- added C204: 10uF, C_1206_3216Metric, F.Cu at (137.7, 61.4)
- added C206: 1nF, C_1206_3216Metric, F.Cu at (136.2, 65.7)
- added C208: 1nF, C_1206_3216Metric, F.Cu at (172.7, 65.8)
- added C230: 100nF, C_0603_1608Metric, F.Cu at (108.5, 17.0)
- added C231: 100nF, C_0603_1608Metric, F.Cu at (146.4, 17.0)
- added C232: 100nF, C_0603_1608Metric, F.Cu at (158.4, 17.0)
- added C233: 100nF, C_0603_1608Metric, F.Cu at (196.4, 17.0)
- added C600: 100nF, C_0603_1608Metric, F.Cu at (247.6, 65.7)
- added C609: 100nF, C_0603_1608Metric, F.Cu at (95.6, 62.3)
- added C617: 100nF, C_0603_1608Metric, F.Cu at (122.2, 161.2)
- added C650: 10uF, C_1206_3216Metric, F.Cu at (253.8, 71.7)
- added C651: 100nF, C_0603_1608Metric, F.Cu at (253.4, 76.0)
- added C660: 100nF, C_0603_1608Metric, F.Cu at (262.1, 29.0)
- added C661: 22nF, C_0805_2012Metric, F.Cu at (242.4, 32.5)
- added C662: 100nF, C_0805_2012Metric, F.Cu at (255.2, 58.0)
- added C663: 2.2uF, C_1210_3225Metric, F.Cu at (255.9, 53.4)
- added C664: 22uF, C_1206_3216Metric, F.Cu at (240.3, 53.6)
- added C665: 100nF, C_0603_1608Metric, F.Cu at (240.8, 58.0)
- added C666: 22uF, C_0603_1608Metric, F.Cu at (242.3, 72.5)
- added C667: 100nF, C_0603_1608Metric, F.Cu at (242.3, 76.0)
- added D31: SMBJ54A, D_SMB, F.Cu at (266.7, 35.8)
- added D607: 1N4148WS, D_SOD-323, F.Cu at (234.7, 124.5)
- added D610: 1N4148WS, D_SOD-323, F.Cu at (30.6, 147.3)
- added D611: 1N4148WS, D_SOD-323, F.Cu at (81.7, 147.3)
- added D612: 1N4148WS, D_SOD-323, F.Cu at (126.3, 147.3)
- added D613: 1N4148WS, D_SOD-323, F.Cu at (164.6, 147.3)
- added D615: 1N4148WS, D_SOD-323, F.Cu at (226.5, 147.3)
- added D616: 1N4148WS, D_SOD-323, F.Cu at (248.3, 147.3)
- added L20: 10uH bogucu, L_Toroid_T50_Vertical, F.Cu at (127.4, 51.0)
- added R240: 10R, R_0603_1608Metric, F.Cu at (114.5, 17.0)
- added R241: 10R, R_0603_1608Metric, F.Cu at (140.4, 17.0)
- added R242: 10R, R_0603_1608Metric, F.Cu at (164.4, 17.0)
- added R243: 10R, R_0603_1608Metric, F.Cu at (190.4, 17.0)
- added R244: 1k, R_0603_1608Metric, F.Cu at (111.5, 17.0)
- added R245: 1k, R_0603_1608Metric, F.Cu at (143.4, 17.0)
- added R246: 1k, R_0603_1608Metric, F.Cu at (161.4, 17.0)
- added R247: 1k, R_0603_1608Metric, F.Cu at (193.4, 17.0)
- added R601: 100k, R_0603_1608Metric, F.Cu at (247.6, 71.5)
- added R602: 140k, R_0603_1608Metric, F.Cu at (247.6, 63.1)
- added R603: 10k, R_0603_1608Metric, F.Cu at (247.6, 68.6)
- added R605: 20k, R_0603_1608Metric, F.Cu at (255.2, 83.5)
- added R606: 100k, R_0603_1608Metric, F.Cu at (193.5, 168.1)
- added T30: BN43-202 3:1, XFMR_Toroid_4P_Vertical, F.Cu at (152.4, 49.5)
- added T31: BN43-3312 2:4 CT, XFMR_Toroid_5P_Vertical, F.Cu at (147.0, 34.0)
- added U52: LM74700QDBVRQ1, SOT-23-6, F.Cu at (252.0, 30.0)
- added U60: AD8318ACPZ, NXP_VQFN-16-1EP_4x4mm_P0.65mm_EP2.1x2.1mm, F.Cu at (266.0, 136.0)
- added U61: AD8318ACPZ, NXP_VQFN-16-1EP_4x4mm_P0.65mm_EP2.1x2.1mm, F.Cu at (266.0, 158.0)
- C110: footprint C_0603_1608Metric -> C_1206_3216Metric
- C601, C602: footprint CP_Radial_D10.0mm_P5.00mm -> CP_Radial_D16.0mm_P7.50mm
- L10: value 10uH bogucu -> 1uH bogucu; footprint L_Toroid_T50_Vertical -> L_0805_2012Metric
- L501, L503, L506, L508: footprint L_Toroid_T50_Vertical -> L_Toroid_T94_Vertical
- L511, L513, L516, L518: footprint L_Toroid_T50_Vertical -> L_Toroid_T68_Vertical
- Q30: value IRF9540N -> IRFB4110PBF
- R205, R207: value 1k -> 820R; footprint R_0603_1608Metric -> R_2512_6332Metric
- R404, R408: value 61R9 -> 19R1
- R604: value 100k -> 105k
- R608: value 10k -> 100k
- T10: value BN43-202 3:1 -> BN43-202 2:1
- T12: value BN43-202 2:3 -> BN43-202 2:3 CT; footprint XFMR_Toroid_4P_Vertical -> XFMR_Toroid_5P_Vertical
- U31: value AD8318ACPZ -> INA240A1DR; footprint NXP_VQFN-16-1EP_4x4mm_P0.65mm_EP2.1x2.1mm -> SOIC-8_3.9x4.9mm_P1.27mm
- moved U33 188.1 mm to (176.4, 23.0)
- moved U34 186.7 mm to (196.4, 23.0)
- moved U32 182.9 mm to (146.4, 23.0)
- moved R608 167.8 mm to (121.5, 177.0)
- moved C411 160.0 mm to (150.8, 2.42)
- moved U31 146.8 mm to (126.5, 23.0)
- moved C407 143.6 mm to (130.8, 2.42)
- moved C303 112.3 mm to (43.5, 172.1)
- moved C307 108.5 mm to (43.5, 168.9)
- moved C110 104.3 mm to (166.5, 68.5)
- moved U41 103.2 mm to (40.0, 164.0)
- moved L11 98.6 mm to (168.4, 65.0)
- moved C311 83.0 mm to (65.5, 172.1)
- moved U42 81.4 mm to (62.0, 164.0)
- moved C315 78.6 mm to (65.5, 168.9)
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Connections:
- D614 pad 1: DPD_EN_LO -> KL5_LO
- D614 pad 2: +5V -> +12V
- R205 pad 1: GATE2 -> DRN_A
- R205 pad 2: G11 -> FB_A
- R207 pad 1: GATE3 -> DRN_B
- R207 pad 2: G12 -> FB_B
- R400 pad 2: GND -> CPL_COM
- R402 pad 2: GND -> CPL_COM
- R604 pad 1: RON_12V -> +5V
- R604 pad 2: GND -> FB_5V
- R608 pad 1: FB_12V -> PA_INHIBIT
- T10 pad 1: DRV_OUT -> D2_IN
- T10 pad 3: GIN_A -> D2_GA
- T10 pad 4: GIN_B -> D2_GB
- T20 pad 4: GND -> REV_RAW
- T21 pad 1: ANT_OUT -> CPL_COM
- T21 pad 2: ANT_OUT -> GND
- T21 pad 3: REV_RAW -> ANT_OUT
- U10 pad 21: (no net) -> GND
- U31 pad 5: REV_CLPF -> IMEAS1
- U31 pad 6: REV_LOG -> +5V
- U31 pad 7: REV_LOG -> GND
Routing:
- net DRN_B: track 0.00 -> 24.4 mm
- net DRN_A: track 0.00 -> 24.4 mm
- net G13: track 14.5 -> 11.5 mm
- net G12: track 14.5 -> 11.5 mm
- net G11: track 14.5 -> 11.5 mm
- net G10: track 14.5 -> 11.5 mm
Other:
- board size 240 x 185 mm -> 275 x 185 mm
- board text added: "​12V->5V"
- board text added: "​15/10m"
- board text added: "​20/17m"
- board text added: "​40/30m"
- board text added: "​50V->12V"
- board text added: "​80/60m"
- board text added: "​BIAS INT 1-2"
- board text added: "​BIAS INT 3-4"
- board text added: "​BYPASS"
- board text added: "​DRV CHOKE"
- board text added: "​DRV IN XFMR"
- board text added: "​FINAL CHOKE"
- board text added: "​FINAL IN XFMR"
- board text added: "​HOLES UNPLATED - CHASSIS BOND ON BOARD C"
- board text added: "​IDEAL DIODE"
- board text added: "​INPUT TVS"
- board text added: "​ISENSE 1"
- board text added: "​ISENSE 2"
- board text added: "​ISENSE 3"
- board text added: "​ISENSE 4"
- board text added: "​REV POLARITY"
- board text removed: "​12/10m"
- board text removed: "​17/15m"
- board text removed: "​30/20m"
- board text removed: "​40m"
- board text removed: "​80m"

Commit message: Correct the clearance test for the pre-routed traces
The clearance test used a circle for each pad. The radius was
max(width, height)/2. The corner of a rectangle is at
hypot(width, height)/2 from the center. The test thus made the pad
smaller than it is. On the 2.5 x 4.5 mm gate pad of a TO-247 the
difference is 2.250 mm against 2.574 mm.

The DRN_A trace was on the gate pad of Q10 with an overlap of 35 um.
This is a short circuit between the 50 V drain rail and the gate of a
100 W device. The search that finds the tee offset accepted this
route. The overlap is at a corner and 35 um wide. You cannot see it
on a plot.

The test now uses the real shape of the pad and the collision test of
pcbnew. It also uses the 300 um clearance and not only an overlap. A
trace that is 50 um from a pad is also not possible to manufacture.

Board D was built again. No trace is below 300 um and the smallest
gap is 0.537 mm. Boards A and C were correct.
Parts:
- added C111: 100nF, C_0603_1608Metric, F.Cu at (23.1, 73.8)
- added C441: 100nF, C_0603_1608Metric, F.Cu at (180.8, 2.42)
- added C442: 100nF, C_0603_1608Metric, F.Cu at (201.8, 26.1)
- added C443: 100nF, C_0603_1608Metric, F.Cu at (257.0, 73.1)
- added C444: 100nF, C_0603_1608Metric, F.Cu at (261.8, 138.5)
- added C460: 100nF, C_0603_1608Metric, F.Cu at (44.4, 160.2)
- added C461: 100nF, C_0603_1608Metric, F.Cu at (66.4, 160.2)
- added C690: 100nF, C_0603_1608Metric, F.Cu at (105.3, 157.9)
- added R99: 10k, R_0603_1608Metric, F.Cu at (89.7, 123.7)
- U10: footprint QFN-20-1EP_4x4mm_P0.5mm_EP2.6x2.6mm_ThermalVias -> TQFN-20-1EP_4x4mm_P0.5mm_EP2.1x2.1mm_ThermalVias
- moved C609 102.4 mm to (122.2, 161.2)
- moved C300 76.2 mm to (95.6, 50.3)
- moved C617 34.3 mm to (155.3, 170.1)
- moved R690 22.6 mm to (153.3, 132.4)
- moved C301 12.0 mm to (95.6, 62.3)
- moved R104 7.79 mm to (29.2, 77.8)
- moved R105 7.02 mm to (32.2, 72.0)
- moved R101 3.02 mm to (36.6, 72.7)
- moved R102 0.75 mm to (27.6, 74.9)
- moved C601 0.51 mm to (261.3, 64.0)
Connections:
- U10 pad 3: ATT_DATA -> ATT_DAT_Q
Routing:
- net DRN_B: track 24.4 -> 26.9 mm
- net DRN_A: track 24.4 -> 26.9 mm

Commit message: Correct the schematic faults that ERC cannot find
An agent examined the three schematics against the datasheets. ERC
reported zero violations before and after this work. None of these
faults are visible to ERC.

The comparator for the external 10 MHz reference was in shutdown. The
SHDN pin of the TLV3501 went to +3V3. Sixteen DRV8833 devices had VCP
and VINT unconnected. Without the charge pump none of the 28 filter
relays can latch. Seven regulators had no decoupling capacitor within
18 mm to 94 mm. On board D the nearest +12V capacitor to an LM358 was
227 mm away on a 275 mm board.

The PE4312 devices had no series 10k resistor on pin 3. The datasheet
makes this necessary for the attenuation accuracy. Their exposed pad
was 2.6 mm against 2.15 mm. The BOM did not give the load capacitance
of the crystal. This work added 60 parts and changed 4 footprints.

The worst fault was in the tool chain. lib/gen_symbols.py still made
the old pin numbers. The five corrections went into the symbol
library by hand and not into its generator. A new library would have
removed all of them.

The thermal vias are now a decision from the measured clearance and
the dissipation. This work removed them from the PE4312, the RTL8211F
and the ADCLK846. They stay on the DRV8833 and on the LM5164, which
is a 1 W buck converter.

Two checks are new. sema_denetim compares the pin names with the
nets. netlist_denetim locks 22 pin-to-net expectations from the
datasheets and does not need a board.

The boards were built again with these corrections. The chain now
adds the test points: 10 on board A, 7 on board C and 15 on board D.
Each board has 3 fiducials. Every pad has a net.
Parts:
- added FID1: ​FID, Fiducial_1mm_Mask2mm, F.Cu at (8.26, 12.6)
- added FID2: ​FID, Fiducial_1mm_Mask2mm, F.Cu at (271.4, 12.6)
- added FID3: ​FID, Fiducial_1mm_Mask2mm, F.Cu at (3.64, 172.4)
- added TP1: ​+50V, TestPoint_Pad_D1.5mm, F.Cu at (244.4, 38.6)
- added TP10: ​IMEAS1, TestPoint_Pad_D1.5mm, F.Cu at (130.5, 29.7)
- added TP11: ​IMEAS2, TestPoint_Pad_D1.5mm, F.Cu at (93.9, 134.7)
- added TP12: ​IMEAS3, TestPoint_Pad_D1.5mm, F.Cu at (180.5, 29.7)
- added TP13: ​IMEAS4, TestPoint_Pad_D1.5mm, F.Cu at (109.5, 137.0)
- added TP14: ​FWD_LOG, TestPoint_Pad_D1.5mm, F.Cu at (272.3, 137.8)
- added TP15: ​REV_LOG, TestPoint_Pad_D1.5mm, F.Cu at (91.6, 162.9)
- added TP2: ​+12V, TestPoint_Pad_D1.5mm, F.Cu at (238.8, 49.6)
- added TP3: ​+5V, TestPoint_Pad_D1.5mm, F.Cu at (262.3, 142.1)
- added TP4: ​+3V3, TestPoint_Pad_D1.5mm, F.Cu at (92.0, 66.5)
- added TP5: ​DRN_CT, TestPoint_Pad_D1.5mm, F.Cu at (136.9, 50.1)
- added TP6: ​GATE1, TestPoint_Pad_D1.5mm, F.Cu at (112.2, 21.7)
- added TP7: ​GATE2, TestPoint_Pad_D1.5mm, F.Cu at (111.1, 72.6)
- added TP8: ​GATE3, TestPoint_Pad_D1.5mm, F.Cu at (103.6, 119.7)
- added TP9: ​GATE4, TestPoint_Pad_D1.5mm, F.Cu at (114.3, 119.7)
- U10: footprint TQFN-20-1EP_4x4mm_P0.5mm_EP2.1x2.1mm_ThermalVias -> TQFN-20-1EP_4x4mm_P0.5mm_EP2.1x2.1mm
- moved C602 1.49 mm to (250.3, 40.1)
- moved C661 0.79 mm to (243.0, 33.1)
- moved C660 0.10 mm to (262.0, 29.0)

Commit message: Move each decoupling capacitor to the pin it serves
The audit found 14 chips with no decoupling capacitor within 15 mm.
Across the boards the nearest capacitor to a supply rail was a median
7.5 mm on A and 6.3 mm on C, and 91 mm in the worst case. A capacitor
45 mm from its pin has about 45 nH of loop inductance, near 2.8 ohm at
10 MHz, where milliohms are necessary. It is on the schematic, it is
in the BOM, it is fitted, and it does nothing.

The pass that moves capacitors ran before the fallback placer, so a
chip with no explicit rule was not yet placed and never entered the
pool. The fallback then gave every spare capacitor to the chip with
the most pins on the rail, which is the FPGA on +3V3. Small parts got
none. The pass now runs last.

A count of missing parts was also wrong. Every pad on a rail was
counted as a supply pin, including logic inputs tied high: SRCLR on
the 74HC595, SLEEP on the DRV8833, P/S on the PE4312. Counting only
pins the netlist marks power_in, board C has 15 supply pins and 15
capacitors. Four capacitors are missing across all three boards, not
59. The AD8318 has three supply pins and had one capacitor; it now
has three. The ADCLK846 has six and had five.
Parts:
- removed C410: 220pF, C_0603_1608Metric
- removed C411: 100nF, C_0603_1608Metric
- removed R408: 19R1, R_0603_1608Metric
- removed R409: 247R, R_0603_1608Metric
- removed R412: 51R, R_0603_1608Metric
- added C408: 100nF, C_0603_1608Metric, F.Cu at (151.3, 2.42)
- added C409: 100nF, C_0603_1608Metric, F.Cu at (209.0, 26.1)
- added C412: 220pF, C_0603_1608Metric, F.Cu at (268.7, 161.5)
- added C413: 100nF, C_0603_1608Metric, F.Cu at (201.8, 26.3)
- added C414: 100nF, C_0603_1608Metric, F.Cu at (256.6, 72.3)
- added C415: 100nF, C_0603_1608Metric, F.Cu at (261.7, 137.9)
- added R410: 19R1, R_0603_1608Metric, F.Cu at (271.8, 106.3)
- added R411: 247R, R_0603_1608Metric, F.Cu at (267.2, 126.4)
- added R416: 51R, R_0603_1608Metric, F.Cu at (267.7, 84.1)
- moved C441 177.0 mm to (261.7, 159.9)
- moved TP12 164.0 mm to (99.8, 172.5)
- moved C442 128.5 mm to (262.2, 139.6)
- moved TP8 114.1 mm to (162.2, 21.7)
- moved TP2 104.0 mm to (201.4, 146.6)
- moved C443 88.6 mm to (262.2, 161.6)
- moved TP9 67.0 mm to (164.2, 74.9)
- moved TP4 65.6 mm to (27.3, 77.4)
- moved TP7 51.2 mm to (91.0, 119.7)
- moved TP11 30.9 mm to (91.6, 165.4)
- moved C602 20.5 mm to (231.3, 32.4)
- moved R308 19.7 mm to (88.2, 127.4)
- moved R302 14.5 mm to (85.8, 145.5)
- moved R402 14.2 mm to (269.5, 108.7)
- moved C203 13.7 mm to (145.1, 65.6)
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
Commit message: Do not count a bulk capacitor as decoupling
The placement pass accepted any capacitor on the rail as sufficient.
On board A the flash memory had 10 uF at 5.5 mm and 47 uF at 16.3 mm,
so the pass was satisfied. Both are bulk. The nearest 100 nF was
17.0 mm away, and at that distance the loop inductance removes the
reason to fit it.

The audit tool already used a 10 uF ceiling for this. The placer did
not, so the two disagreed, and the placer was wrong.

The pass now treats only capacitors of 1 uF and below as decoupling,
both when it asks whether a pin is served and when it selects one to
move. It also searches a ring around the pin for free space instead
of using a fixed offset.

Findings fall from 14 to 4. Board A is clean.

Also: build.sh never ran bom.py, so BOM_*.csv were hand-made files
that no step regenerated and the BOM no longer matched the schematic.
Each board's build now writes its own.
Parts:
- C110: value 10uF -> 100nF; footprint C_1206_3216Metric -> C_0603_1608Metric
- moved TP15 166.1 mm to (257.7, 159.8)
- moved TP12 163.9 mm to (178.9, 28.9)
- moved TP2 143.6 mm to (58.2, 157.5)
- moved TP10 123.3 mm to (89.8, 147.0)
- moved TP8 114.1 mm to (103.6, 119.7)
- moved TP3 67.5 mm to (258.8, 76.7)
- moved TP13 36.5 mm to (100.5, 172.4)
- moved TP11 29.0 mm to (92.3, 136.4)
- moved TP1 17.8 mm to (250.3, 52.1)
- moved C507 11.0 mm to (89.5, 118.1)
- moved TP4 8.96 mm to (36.3, 77.6)
- moved C602 8.39 mm to (237.8, 37.7)
- moved R690 7.55 mm to (153.3, 122.2)
- moved C461 7.31 mm to (62.6, 159.0)
- moved C460 7.27 mm to (40.7, 159.0)
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
Commit message: Let the placer, not the separator, own the capacitor position
Placing a capacitor beside its supply pin and then resolving overlaps
moves it away again. On board C the pass put a 100 nF 4.7 mm from the
attenuator's pin, the separator cleared 191 overlaps, and the
capacitor finished 17.9 mm away.

The pass now runs after separation and searches for free space around
the pin itself, so it does not need the separator afterwards. It
moves 21 capacitors on A, 26 on C and 12 on D.

Measured at the supply pin, the median distance is 2.8 mm on A,
5.4 mm on C and 4.6 mm on D. Board C's worst supply pin improves from
98.5 mm to 8.9 mm. Findings fall from 14 to 1.
Parts:
- moved TP2 176.1 mm to (233.9, 146.6)
- moved TP14 171.3 mm to (91.6, 161.6)
- moved TP15 166.2 mm to (91.6, 165.8)
- moved TP12 130.9 mm to (100.8, 133.9)
- moved TP11 127.6 mm to (152.8, 24.1)
- moved TP7 123.5 mm to (141.9, 13.1)
- moved TP8 114.1 mm to (162.2, 21.7)
- moved TP9 67.1 mm to (191.9, 13.1)
- moved TP3 57.8 mm to (236.5, 130.0)
- moved TP6 55.6 mm to (89.8, 72.6)
- moved TP13 36.5 mm to (109.5, 137.0)
- moved TP1 30.4 mm to (259.0, 22.9)
- moved C409 30.1 mm to (178.9, 28.2)
- moved C407 27.1 mm to (151.6, 17.1)
- moved C662 10.4 mm to (249.2, 66.5), turned to 0 degrees
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