File: hardware/kicad/D_pa/dogrudan_sdr_D.kicad_pcb (KiCad board)
At the start: 2 copper layers, 275 x 185 mm, 232 parts, among them J10 A kartindan TX1, J20 DPD -> C karti, J30 50V giris, J31 A kartina, J32 C kartindan, J33 sonraki PA, J40 ANTEN -> panel SO-239, K20 G6K-2F-Y, Q10 IRFP250N, Q11 IRFP250N, Q12 IRFP250N, Q13 IRFP250N, Q20 IRF530N, Q21 IRF530N, Q30 IRFB4110PBF, Q31 2N7002, Q32 2N7002, T10 BN43-202 2:1, T12 BN43-202 2:3 CT, T20 FT50-43 1:32, T21 FT50-43 1:32, T30 BN43-202 3:1, T31 BN43-3312 2:4 CT, U10 PE4312C-Z, U11 PGA-103+, U20 MCP4922-E/SL, U21 MCP4922-E/SL, U31 INA240A1DR, U32 INA240A1DR, U33 INA240A1DR, U34 INA240A1DR, U41 LM358, U42 LM358, U50 LM5164DDAR, U51 TPS62130, U52 LM74700QDBVRQ1, U55 MCP9700AT, U56 74HC595D, U57 MCP3208T-CI/SL, U60 AD8318ACPZ, U61 AD8318ACPZ

Commit message: Compare symbol pins against footprint pads before placement
Every fault that would have stopped a board in this work sits in one
layer: a symbol pin number that does not agree with a footprint pad
number. The ADC paddle was pin 0 against pad 65. The attenuator
paddle was named Pad against pad 21. The gas discharge tubes used
pins 1 and 3 against pads 1 and 2. The crystal had two pins on a
four-pad part, so XO went to the can. The Ethernet PHY carried the
footprint of a different package. Each was found separately, by hand,
after it had already cost placement and routing time.

temel_denetim checks the whole class at once. For each part it
reports pins with no pad, where the net goes nowhere while the
schematic looks correct; pads with no pin, where copper is left
unconnected; and a count mismatch, which is the quickest sign that a
footprint belongs to another part.

It reads the symbols embedded in the schematics and not the library
file, because the library was edited by hand while its generator
stayed behind.

yap.sh runs it after pcb_kur and before placement, and stops there. A
wrong schematic makes everything below it worthless.

All three boards report zero. The parts it cannot check are those
with no symbol: mounting holes, fiducials and test points.
Parts:
- C110: value 100nF -> 10uF; footprint C_0603_1608Metric -> C_1206_3216Metric
- moved TP11 154.0 mm to (91.6, 165.4)
- moved TP9 131.8 mm to (114.3, 119.7)
- moved TP12 129.3 mm to (177.4, 29.7)
- moved TP10 124.5 mm to (128.9, 28.9)
- moved TP7 123.5 mm to (93.0, 126.5)
- moved TP3 115.0 mm to (181.2, 29.2)
- moved TP4 107.0 mm to (39.2, 175.7)
- moved TP2 73.9 mm to (258.2, 76.8)
- moved TP8 61.2 mm to (134.6, 76.3)
- moved TP6 56.0 mm to (68.8, 124.5)
- moved TP1 26.8 mm to (254.4, 49.3)
- moved TP15 10.9 mm to (95.2, 155.5)
- moved C409 10.2 mm to (178.9, 18.1)
- moved TP5 8.07 mm to (140.8, 44.1)
- moved R690 7.55 mm to (153.3, 129.8)
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
Commit message: Replace the transmit filters: harmonic suppression was illegal
Simulation of the output filters shows second-harmonic suppression
between 3 and 30 dB, where 43 dB is necessary below 30 MHz and 60 dB
above. On the 80/60 m position the second harmonic of 3.5 MHz is
3.4 dB down: the filter barely touches it. The transmitter would have
been out of specification on every band, and the board gives no sign
of it. Output power, SWR and efficiency all read correctly while the
harmonic radiates.

The cause is the band grouping. One position must pass 5.37 MHz, so
its cutoff is at 6.0, and the second harmonic of the same position's
lowest band, 3.5 MHz, falls at 7.0. More poles do not help: by the
Chebyshev attenuation formula, nine poles give 32 dB there.

Each series inductor now has a parallel capacitor that places a
transmission zero on the harmonic. 80 m and 60 m are separate
positions, because a trap at 7.0 MHz also attenuates a 5.37 MHz
passband. That uses the seventh relay, which was a bypass; a
transmitter with no harmonic filter in line is not legal in any case.

  band      loss   2nd harmonic   was
  160m      0.61   -82.4          -25.2
  80m       0.64   -80.7          grouped
  60m       0.45   -81.9          grouped
  40_30m    1.45   -58.0          -9.5
  20_17m    0.88   -68.4          -18.2
  15_10m    1.35   -61.0          -14.1
  6m        1.14   -82.8          -30.2
Parts:
- removed C504: 1600pF, C_Disc_D7.5mm_W5.0mm_P5.00mm
- removed C515, C522: 200pF, C_Disc_D7.5mm_W5.0mm_P5.00mm
- removed C525, C529: 68pF, C_Disc_D7.5mm_W5.0mm_P5.00mm
- removed L503: T94-2 25s, L_Toroid_T94_Vertical
- removed L506: T94-2 15s, L_Toroid_T94_Vertical
- removed L513: T68-2 13s, L_Toroid_T68_Vertical
- removed L516: T68-2 10s, L_Toroid_T68_Vertical
- removed L521, L523: T50-6 10s, L_Toroid_T50_Vertical
- removed L526, L528: T50-6 8s, L_Toroid_T50_Vertical
- added C503: 2700pF, C_Disc_D7.5mm_W5.0mm_P5.00mm, F.Cu at (44.0, 119.3)
- added C506: 1600pF, C_Disc_D7.5mm_W5.0mm_P5.00mm, F.Cu at (55.2, 118.2)
- added C513: 820pF, C_Disc_D7.5mm_W5.0mm_P5.00mm, F.Cu at (106.3, 120.5)
- added C516: 120pF, C_Disc_D7.5mm_W5.0mm_P5.00mm, F.Cu at (140.4, 118.1)
- added C521: 270pF, C_Disc_D7.5mm_W5.0mm_P5.00mm, F.Cu at (166.3, 116.0)
- added C523: 180pF, C_Disc_D7.5mm_W5.0mm_P5.00mm, F.Cu at (185.2, 114.9)
- added C526: 75pF, C_Disc_D7.5mm_W5.0mm_P5.00mm, F.Cu at (193.1, 122.4)
- added C528: 160pF, C_Disc_D7.5mm_W5.0mm_P5.00mm, F.Cu at (204.5, 114.9)
- added C530: 68pF, C_Disc_D7.5mm_W5.0mm_P5.00mm, F.Cu at (223.3, 115.0)
- added C531: 270pF, C_Disc_D7.5mm_W5.0mm_P5.00mm, F.Cu at (225.6, 123.2)
- added C533: 30pF, C_Disc_D7.5mm_W5.0mm_P5.00mm, F.Cu at (230.9, 115.0)
- added C534: 160pF, C_Disc_D7.5mm_W5.0mm_P5.00mm, F.Cu at (236.5, 122.5)
- added C535: 91pF, C_Disc_D7.5mm_W5.0mm_P5.00mm, F.Cu at (237.4, 114.2)
- added C537: 51pF, C_Disc_D7.5mm_W5.0mm_P5.00mm, F.Cu at (258.6, 148.6)
- added C538: 160pF, C_Disc_D7.5mm_W5.0mm_P5.00mm, F.Cu at (254.9, 156.8)
- added C540: 24pF, C_Disc_D7.5mm_W5.0mm_P5.00mm, F.Cu at (256.7, 140.4)
- added C541: 91pF, C_Disc_D7.5mm_W5.0mm_P5.00mm, F.Cu at (272.1, 162.6)
- added C542: 62pF, C_Disc_D7.5mm_W5.0mm_P5.00mm, F.Cu at (256.7, 132.3)
- added C544: 15pF, C_Disc_D7.5mm_W5.0mm_P5.00mm, F.Cu at (272.1, 111.5)
- added C545: 110pF, C_Disc_D7.5mm_W5.0mm_P5.00mm, F.Cu at (255.6, 113.7)
- added C547: 6.2pF, C_Disc_D7.5mm_W5.0mm_P5.00mm, F.Cu at (272.1, 151.9)
- added C548: 62pF, C_Disc_D7.5mm_W5.0mm_P5.00mm, F.Cu at (272.1, 111.0)
- added L504: T94-2 24s, L_Toroid_T94_Vertical, F.Cu at (41.8, 99.0)
- added L515: T94-2 15s, L_Toroid_T94_Vertical, F.Cu at (118.3, 99.0)
- added L522: T68-2 12s, L_Toroid_T68_Vertical, F.Cu at (166.2, 99.0)
- added L525: T68-2 12s, L_Toroid_T68_Vertical, F.Cu at (185.2, 99.0)
- added L529: T68-2 10s, L_Toroid_T68_Vertical, F.Cu at (204.4, 99.0)
- added L532: T68-2 10s, L_Toroid_T68_Vertical, F.Cu at (223.5, 99.0)
- added L536: T50-6 9s, L_Toroid_T50_Vertical, F.Cu at (240.3, 99.0)
- added L539: T50-6 9s, L_Toroid_T50_Vertical, F.Cu at (254.5, 99.0)
- added L543, L546: T50-6 7s, L_Toroid_T50_Vertical, F.Cu at (267.1, 99.0)
- C110: value 10uF -> 100nF; footprint C_1206_3216Metric -> C_0603_1608Metric
- C502: value 3000pF -> 430pF
- C505: value 620pF -> 180pF
- C507: value 1000pF -> 820pF
- C509: value 620pF -> 220pF
- C510: value 330pF -> 1500pF
- C512: value 560pF -> 91pF
- C514: value 330pF -> 560pF
- C517: value 330pF -> 1000pF
- C519: value 200pF -> 56pF
- C520: value 120pF -> 560pF
- C524: value 120pF -> 430pF
- C527: value 110pF -> 270pF
- L501: value T94-2 25s -> T94-2 24s
- L508: value T94-2 15s -> T94-2 17s
- L511: value T68-2 13s -> T94-2 17s; footprint L_Toroid_T68_Vertical -> L_Toroid_T94_Vertical
- L518: value T68-2 10s -> T94-2 15s; footprint L_Toroid_T68_Vertical -> L_Toroid_T94_Vertical
- moved TP2 243.9 mm to (18.6, 122.3)
- moved TP12 162.5 mm to (99.8, 172.5)
- moved TP11 154.0 mm to (152.8, 24.1)
- moved TP10 140.3 mm to (91.6, 164.1)
- moved TP9 131.8 mm to (191.9, 13.1)
- moved TP4 98.5 mm to (22.9, 78.5)
- moved R690 89.9 mm to (240.2, 106.9)
- moved TP3 79.8 mm to (249.5, 70.6)
- moved TP8 58.3 mm to (101.9, 124.6)
- moved TP7 56.9 mm to (111.1, 72.6)
- moved TP13 38.4 mm to (96.0, 173.0)
- moved C512 33.6 mm to (100.7, 118.1)
- moved C527 31.0 mm to (198.8, 114.9)
- moved C520 29.7 mm to (157.3, 118.2)
- moved L518 28.7 mm to (143.8, 99.0), turned to 0 degrees
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Connections:
- C502 pad 1: N1_1 -> LF1_A
- C502 pad 2: GND -> N1_1
- C505 pad 1: LF2_A -> N1_1
- C505 pad 2: GND -> LF1_B
- C507 pad 1: N2_1 -> LF2_A
- C509 pad 1: LF2_B -> LF2_A
- C509 pad 2: GND -> N2_1
- C510 pad 1: LF3_A -> N2_1
- C512 pad 1: N3_1 -> N2_1
- C512 pad 2: GND -> LF2_B
- C514 pad 1: LF3_B -> LF3_A
- C517 pad 1: N4_1 -> N3_1
- C519 pad 1: LF4_B -> N3_1
- C519 pad 2: GND -> LF3_B
- C520 pad 1: LF5_A -> LF3_B
- C524 pad 1: LF5_B -> N4_1
- C527 pad 1: N6_1 -> LF4_B
- KL7 pad 14: PA_LPF_OUT -> LF7_A
- KL7 pad 24: PA_LPF_OUT -> LF7_B
- L508 pad 1: N2_1 -> LF2_A
- L508 pad 2: LF2_B -> N2_1
- L511 pad 1: LF3_A -> N2_1
- L511 pad 2: N3_1 -> LF2_B
- L518 pad 1: N4_1 -> N3_1
- L518 pad 2: LF4_B -> LF3_B

Commit message: Fit the filter bank and clear the overlaps
Board D's filter bank needs 285.6 mm of width with both inductors of
each band side by side, against about 236 mm available. Stacking them
vertically corrects the width and breaks the height: the strip
between the driver transformer and the relay row is 15.8 mm and a
stacked pair of T68 cores needs 37.7 mm.

Mapping the board in 10 mm bands gave the answer. Everything below
the relay row is the coupler and detector block at x above 250, while
the filter columns run from x 4 to 236. The space under them was
empty. The relay row moves from y 130 to 142 and its drivers from 155
to 172, with the filter block following. No board grew and the chain
stays in one row.

The separator never moves a part whose reference begins with U, J, T,
Y, L, Q, K or H, so two such parts overlapping cannot be separated
and the fix belongs in the placement rules. On A the XT60's courtyard
is 22.4 mm tall and snapped to the top edge, so it covered the
reverse-polarity MOSFET; the crystals and their inductors were placed
by the fallback and landed inside the PHY. All three now have
explicit positions.

The separator also gained a last resort: a movable part wedged so
that every push lands it in another part is relocated to the nearest
free position.

All three boards are at zero overlaps.
Parts:
- moved TP2 231.9 mm to (242.8, 63.0)
- moved TP11 156.7 mm to (91.6, 168.4)
- moved QL7 128.1 mm to (143.3, 155.0)
- moved C541 127.7 mm to (156.2, 108.9)
- moved L539 126.4 mm to (128.3, 106.2)
- moved KL7 125.0 mm to (139.6, 117.9)
- moved L543 124.0 mm to (143.3, 91.9)
- moved L546 124.0 mm to (143.3, 106.2)
- moved C544 121.8 mm to (152.7, 135.4)
- moved C537 120.0 mm to (139.7, 164.7)
- moved KL6 119.0 mm to (124.5, 117.9)
- moved QL6 119.0 mm to (128.3, 155.0)
- moved TP3 117.7 mm to (150.9, 6.35)
- moved D615 116.7 mm to (133.7, 145.7)
- moved C547 115.9 mm to (161.3, 117.8)
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Routing:
- net DRN_B: track 26.9 -> 0.00 mm
- net DRN_A: track 26.9 -> 0.00 mm
- net D2_GA_S: track 12.3 -> 0.00 mm
- net D2_GB_S: track 12.3 -> 0.00 mm
- net G13: track 11.5 -> 0.00 mm
- net G12: track 11.5 -> 0.00 mm
- net G11: track 11.5 -> 0.00 mm
- net G10: track 11.5 -> 0.00 mm
Other:
- board text removed: "​!! 50V - 100W RF - HEATSINK IS HOT !!"
- board text removed: "​12V->5V"
- board text removed: "​15/10m"
- board text removed: "​160m"
- board text removed: "​20/17m"
- board text removed: "​40/30m"
- board text removed: "​50V IN"
- board text removed: "​50V->12V"
- board text removed: "​6m"
- board text removed: "​80/60m"
- board text removed: "​ANT OUT"
- board text removed: "​BIAS INT 1-2"
- board text removed: "​BIAS INT 3-4"
- board text removed: "​BYPASS"
- board text removed: "​DET FWD"
- board text removed: "​DET REV"
- board text removed: "​DPD -> C"
- board text removed: "​DPD RELAY"
- board text removed: "​DRV CHOKE"
- board text removed: "​DRV IN XFMR"
- board text removed: "​FINAL 1"
- board text removed: "​FINAL 2"
- board text removed: "​FINAL 3"
- board text removed: "​FINAL 4"
- board text removed: "​FINAL CHOKE"
- board text removed: "​FINAL IN XFMR"
- board text removed: "​FORWARD"
- board text removed: "​FROM BOARD C"
- board text removed: "​HOLES UNPLATED - CHASSIS BOND ON BOARD C"
- board text removed: "​IDEAL DIODE"
- board text removed: "​INPUT TVS"
- board text removed: "​ISENSE 1"
- board text removed: "​ISENSE 2"
- board text removed: "​ISENSE 3"
- board text removed: "​ISENSE 4"
- board text removed: "​OUTPUT XFMR"
- board text removed: "​POWER AMPLIFIER - CLASS A 5..100W REV A"
- board text removed: "​REFLECTED"
- board text removed: "​REV POLARITY"
- board text removed: "​TO BOARD A"
- board text removed: "​TX IN <- A"

Commit message: Close the last overlaps and record the pass that undid the other
Board D reaches zero overlaps. Two remained after the relay row
moved: a T68 clipping the driver transformer by 1 x 2 mm, and two
2N7002 transistors two millimetres apart, which the separator was
never going to touch because both begin with Q.

One finding is left on D. Tracing a single capacitor through every
stage shows the mechanism:

  pcb_kur          121.2 mm from the chip
  placement          5.1 mm   correct
  separation        21.0 mm   pushed away
  decoupling pass   25.3 mm   handed to another chip

The placer puts the capacitor beside the pin that needs it, the
separator finds an overlap and moves it, and the decoupling pass then
reads it as the nearest free capacitor for somebody else. The chip
that began with a correct capacitor ends with none.

The two steps disagreed about what an overlap is: the pass used a
1.4 mm margin while the separator used its courtyard box. What one
called clear the other called a collision. The pass now uses the
separator's measure. Its guard against taking a chip's only capacitor
was also too broad, counting chips connected through a logic input
tied high; it now applies the same power_in test.

What remains is to decide which of the two passes owns the final
position.
Parts:
- moved TP2 185.7 mm to (70.4, 132.2)
- moved TP14 171.2 mm to (262.0, 143.8)
- moved TP15 170.3 mm to (257.7, 159.8)
- moved TP6 115.1 mm to (112.2, 21.7)
- moved C533 112.6 mm to (235.6, 111.2)
- moved C538 96.6 mm to (231.6, 122.8)
- moved C541 90.2 mm to (239.5, 143.7)
- moved C527 88.7 mm to (208.2, 167.9)
- moved C531 85.8 mm to (202.6, 168.4)
- moved C526 85.2 mm to (197.3, 179.9)
- moved C540 84.0 mm to (235.0, 135.4)
- moved C542 83.8 mm to (229.2, 130.9)
- moved C521 82.9 mm to (158.5, 135.3)
- moved C534 82.4 mm to (214.6, 171.7)
- moved TP7 81.9 mm to (111.1, 72.6)
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
Commit message: Name the copyright holder and stamp it into the generated files
The repository had three licence files and no statement of who owns
the work. The only record of authorship was the git author field.

Copyleft depends on that statement. GPL and CERN-OHL-S work because
the holder grants permission on condition of reciprocity; with no
holder named there is nobody to require it from a downstream user.
Naming the author keeps the design open rather than closing it.

kicad/telif.py is the single source. The line reaches the schematics
through their title block and not through the generators, because
every schematic file is rewritten on each build and a header placed in
a generator would disappear at the first regeneration. All 23
schematics carry it. 109 source files have SPDX headers, split by the
project's own table: generators and the layout chain are hardware
under CERN-OHL-S-2.0, HDL and the audit tools are software under
GPL-3.0-only.

Board C's inductors also move to footprints that match parts that can
be bought. All of them sat on 0805 pads. Of the values this design
needs, 33 to 220 nH are 0603 parts, 470 and 820 nH are 0805, and
everything from 1000 nH upward is 1210, which is 3.2 by 2.5 mm and
does not fit an 0805 land. 32 inductors could not have been soldered.

A symbol-against-footprint check cannot find this. Those two agreed
with each other; what was wrong was the body size of the real part
behind the footprint.
Parts:
- removed C505, C523: 180pF, C_Disc_D7.5mm_W5.0mm_P5.00mm
- removed C510: 1500pF, C_Disc_D7.5mm_W5.0mm_P5.00mm
- removed C514: 560pF, C_Disc_D7.5mm_W5.0mm_P5.00mm
- removed C519: 56pF, C_Disc_D7.5mm_W5.0mm_P5.00mm
- removed C528: 160pF, C_Disc_D7.5mm_W5.0mm_P5.00mm
- removed C537: 51pF, C_Disc_D7.5mm_W5.0mm_P5.00mm
- removed C541: 91pF, C_Disc_D7.5mm_W5.0mm_P5.00mm
- removed L504: T94-2 24s, L_Toroid_T94_Vertical
- removed L508, L511: T94-2 17s, L_Toroid_T94_Vertical
- removed L515, L518: T94-2 15s, L_Toroid_T94_Vertical
- removed L522, L525: T68-2 12s, L_Toroid_T68_Vertical
- removed L529: T68-2 10s, L_Toroid_T68_Vertical
- removed L536, L539: T50-6 9s, L_Toroid_T50_Vertical
- removed L543: T50-6 7s, L_Toroid_T50_Vertical
- added C504: 2700pF, C_Disc_D7.5mm_W5.0mm_P5.00mm, F.Cu at (46.5, 131.0)
- added C508: 1600pF, C_Disc_D7.5mm_W5.0mm_P5.00mm, F.Cu at (65.7, 129.1)
- added C511: 200pF, C_Disc_D7.5mm_W5.0mm_P5.00mm, F.Cu at (90.4, 131.9)
- added C515: 91pF, C_Disc_D7.5mm_W5.0mm_P5.00mm, F.Cu at (104.9, 128.7)
- added C518: 560pF, C_Disc_D7.5mm_W5.0mm_P5.00mm, F.Cu at (122.9, 127.2)
- added C522: 1000pF, C_Disc_D7.5mm_W5.0mm_P5.00mm, F.Cu at (147.6, 128.7)
- added C525: 3.6pF, C_1206_3216Metric, F.Cu at (157.4, 127.7)
- added C529: 160pF, C_Disc_D7.5mm_W5.0mm_P5.00mm, F.Cu at (177.3, 146.4)
- added C536: 160pF, C_Disc_D7.5mm_W5.0mm_P5.00mm, F.Cu at (182.6, 172.3)
- added C539: 6.8pF, C_1206_3216Metric, F.Cu at (198.0, 124.8)
- added C543: 3.6pF, C_1206_3216Metric, F.Cu at (218.3, 124.5)
- added C549: 160pF, C_Disc_D7.5mm_W5.0mm_P5.00mm, F.Cu at (229.2, 146.7)
- added C551: 22pF, C_Disc_D7.5mm_W5.0mm_P5.00mm, F.Cu at (235.0, 138.5)
- added C552: 1.6pF, C_1206_3216Metric, F.Cu at (237.8, 120.3)
- added C553: 91pF, C_Disc_D7.5mm_W5.0mm_P5.00mm, F.Cu at (249.0, 129.6)
- added C554: 62pF, C_Disc_D7.5mm_W5.0mm_P5.00mm, F.Cu at (214.1, 163.5)
- added C556: 13pF, C_Disc_D7.5mm_W5.0mm_P5.00mm, F.Cu at (229.3, 133.6)
- added C557: 1.1pF, C_1206_3216Metric, F.Cu at (228.0, 121.6)
- added C558: 110pF, C_Disc_D7.5mm_W5.0mm_P5.00mm, F.Cu at (237.7, 130.2)
- added C560: 5.1pF, C_Disc_D7.5mm_W5.0mm_P5.00mm, F.Cu at (243.3, 128.2)
- added C561: 1.2pF, C_1206_3216Metric, F.Cu at (253.1, 125.0)
- added C562: 62pF, C_Disc_D7.5mm_W5.0mm_P5.00mm, F.Cu at (257.7, 132.2)
- added L505: T94-2 24s, L_Toroid_T94_Vertical, F.Cu at (42.0, 108.0)
- added L510: T94-2 17s, L_Toroid_T94_Vertical, F.Cu at (68.1, 108.0)
- added L514: T94-2 17s, L_Toroid_T94_Vertical, F.Cu at (93.6, 108.0)
- added L519: T94-2 15s, L_Toroid_T94_Vertical, F.Cu at (119.6, 108.0)
- added L523: T94-2 15s, L_Toroid_T94_Vertical, F.Cu at (145.1, 108.0)
- added L528: T68-2 12s, L_Toroid_T68_Vertical, F.Cu at (167.9, 98.5)
- added L537: T68-2 10s, L_Toroid_T68_Vertical, F.Cu at (187.5, 98.5)
- added L541: T68-2 10s, L_Toroid_T68_Vertical, F.Cu at (187.5, 117.5)
- added L550: T50-6 9s, L_Toroid_T50_Vertical, F.Cu at (204.9, 115.2)
- added L555: T50-6 7s, L_Toroid_T50_Vertical, F.Cu at (219.8, 100.9)
- added L559: T50-6 7s, L_Toroid_T50_Vertical, F.Cu at (219.8, 115.2)
- C110: value 100nF -> 10uF; footprint C_0603_1608Metric -> C_1206_3216Metric
- C502: value 430pF -> 360pF
- C503: value 2700pF -> 56pF; footprint C_Disc_D7.5mm_W5.0mm_P5.00mm -> C_1206_3216Metric
- C506: value 1600pF -> 180pF
- C507: value 820pF -> 4.7pF; footprint C_Disc_D7.5mm_W5.0mm_P5.00mm -> C_1206_3216Metric
- C509: value 220pF -> 820pF
- C512: value 91pF -> 15pF; footprint C_Disc_D7.5mm_W5.0mm_P5.00mm -> C_1206_3216Metric
- C513: value 820pF -> 1500pF
- C516: value 120pF -> 4.7pF; footprint C_Disc_D7.5mm_W5.0mm_P5.00mm -> C_1206_3216Metric
- C517: value 1000pF -> 820pF
- C520: value 560pF -> 120pF
- C521: value 270pF -> 3pF; footprint C_Disc_D7.5mm_W5.0mm_P5.00mm -> C_1206_3216Metric
- C524: value 430pF -> 51pF
- C526: value 75pF -> 560pF
- C530: value 68pF -> 12pF; footprint C_Disc_D7.5mm_W5.0mm_P5.00mm -> C_1206_3216Metric
- C531: value 270pF -> 430pF
- C533: value 30pF -> 75pF
- C534: value 160pF -> 1.6pF; footprint C_Disc_D7.5mm_W5.0mm_P5.00mm -> C_1206_3216Metric
- C535: value 91pF -> 270pF
- C538: value 160pF -> 62pF
- C540: value 24pF -> 270pF
- C542: value 62pF -> 27pF
- C544: value 15pF -> 160pF
- C545: value 110pF -> 91pF
- C547: value 6.2pF -> 51pF
- C548: value 62pF -> 2.2pF; footprint C_Disc_D7.5mm_W5.0mm_P5.00mm -> C_1206_3216Metric
- L532: value T68-2 10s -> T68-2 12s
- L546: value T50-6 7s -> T50-6 9s
- moved TP13 138.8 mm to (197.4, 29.7)
- moved TP12 130.9 mm to (178.9, 28.9)
- moved TP3 122.1 mm to (257.6, 138.6)
- moved TP6 118.6 mm to (69.3, 132.3)
- moved TP4 88.8 mm to (39.2, 175.7)
- moved R99 80.4 mm to (21.6, 71.0)
- moved C533 71.9 mm to (196.4, 171.5)
- moved TP9 67.1 mm to (165.9, 74.9)
- moved TP8 65.6 mm to (100.3, 132.2)
- moved C527 58.5 mm to (158.5, 136.9)
- moved C547 57.7 mm to (215.0, 171.6)
- moved TP7 56.7 mm to (83.9, 122.4)
- moved C538 53.7 mm to (196.5, 163.4)
- moved C545 50.6 mm to (202.1, 163.4)
- moved C534 49.3 mm to (200.5, 124.4)
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Connections:
- C503 pad 1: N1_1 -> LF1_A
- C503 pad 2: GND -> N1_1
- C506 pad 1: LF1_B -> N1_1
- C506 pad 2: GND -> LF1_B
- C507 pad 1: LF2_A -> N1_1
- C507 pad 2: GND -> LF1_B
- C509 pad 2: N2_1 -> GND
- C512 pad 1: N2_1 -> LF2_A
- C512 pad 2: LF2_B -> N2_1
- C513 pad 1: LF2_B -> N2_1
- C516 pad 1: LF3_A -> N2_1
- C516 pad 2: N3_1 -> LF2_B
- C517 pad 1: N3_1 -> LF2_B
- C520 pad 1: LF3_B -> LF3_A
- C520 pad 2: GND -> N3_1
- C521 pad 1: LF4_A -> LF3_A
- C521 pad 2: GND -> N3_1
- C524 pad 1: N4_1 -> N3_1
- C524 pad 2: GND -> LF3_B
- C526 pad 1: N4_1 -> LF3_B
- C526 pad 2: LF4_B -> GND
- C527 pad 1: LF4_B -> LF4_A
- C530 pad 1: LF5_A -> LF4_A
- C530 pad 2: N5_1 -> N4_1
- C531 pad 1: N5_1 -> N4_1
- C533 pad 1: N5_1 -> N4_1
- C533 pad 2: LF5_B -> LF4_B
- C534 pad 1: LF5_B -> N4_1
- C534 pad 2: GND -> LF4_B
- C535 pad 1: LF6_A -> LF4_B
- C538 pad 1: N6_1 -> LF5_A
- C538 pad 2: GND -> N5_1
- C540 pad 1: N6_1 -> N5_1
- C540 pad 2: LF6_B -> GND
- C542 pad 1: LF7_A -> N5_1
- C542 pad 2: GND -> LF5_B
- C544 pad 1: LF7_A -> LF5_B
- C544 pad 2: N7_1 -> GND
- C545 pad 1: N7_1 -> LF6_A
- C547 pad 1: N7_1 -> LF6_A
- C547 pad 2: LF7_B -> N6_1
- C548 pad 1: LF7_B -> LF6_A
- C548 pad 2: GND -> N6_1
- L532 pad 1: N5_1 -> N4_1
- L532 pad 2: LF5_B -> LF4_B
- L546 pad 1: N7_1 -> LF6_A
- L546 pad 2: LF7_B -> N6_1
Routing:
- net D2_GA_S: track 0.00 -> 12.3 mm
- net D2_GB_S: track 0.00 -> 12.3 mm
- net G13: track 0.00 -> 11.5 mm
- net G12: track 0.00 -> 11.5 mm
- net G11: track 0.00 -> 11.5 mm
- net G10: track 0.00 -> 11.5 mm
Other:
- board text added: "​!! 50V - 100W RF - HEATSINK IS HOT !!"
- board text added: "​12V->5V"
- board text added: "​15/10m"
- board text added: "​160m"
- board text added: "​20/17m"
- board text added: "​40/30m"
- board text added: "​50V IN"
- board text added: "​50V->12V"
- board text added: "​6m"
- board text added: "​80/60m"
- board text added: "​ANT OUT"
- board text added: "​BIAS INT 1-2"
- board text added: "​BIAS INT 3-4"
- board text added: "​BYPASS"
- board text added: "​DET FWD"
- board text added: "​DET REV"
- board text added: "​DPD -> C"
- board text added: "​DPD RELAY"
- board text added: "​DRV CHOKE"
- board text added: "​DRV IN XFMR"
- board text added: "​FINAL 1"
- board text added: "​FINAL 2"
- board text added: "​FINAL 3"
- board text added: "​FINAL 4"
- board text added: "​FINAL CHOKE"
- board text added: "​FINAL IN XFMR"
- board text added: "​FORWARD"
- board text added: "​FROM BOARD C"
- board text added: "​HOLES UNPLATED - CHASSIS BOND ON BOARD C"
- board text added: "​IDEAL DIODE"
- board text added: "​INPUT TVS"
- board text added: "​ISENSE 1"
- board text added: "​ISENSE 2"
- board text added: "​ISENSE 3"
- board text added: "​ISENSE 4"
- board text added: "​OUTPUT XFMR"
- board text added: "​POWER AMPLIFIER - CLASS A 5..100W REV A"
- board text added: "​REFLECTED"
- board text added: "​REV POLARITY"
- board text added: "​TO BOARD A"
- board text added: "​TX IN <- A"
