File: hardware/kicad/A_main/02_clock.kicad_sch (KiCad schematic)
At the start: 29 parts, among them U15 ADCLK846BCPZ, U16 SN65LVDS2DBVR, U17 SN65LVDS2DBVR, U18 SN65LVDS2DBVR, Y10 ABLNO-V-80.000MHZ

Commit message: Update the ARDC package and record the simulation results
The package had drifted from the boards again: board C's BOM was 45
lines out of date and D's 46, and the schematic PDFs predated both
filter redesigns.

The verification document gains a section on circuit simulation. Every
check before it asks which pin joins which net; none of them can say
whether a capacitor's value is correct. That section holds the
measurements for both redesigns and, separately, the three faults the
simulation tools had themselves: a source divider that made every
insertion loss 6 dB too pessimistic, an E12 rounding helper that
multiplied instead of dividing, and an inductor loss computed at a
fixed 1 MHz.

Two entries in the status were wrong. Gateware timing is closed, with
all five clocks above target rather than two below. Decoupling
placement is corrected. In their place: the remaining overlaps at the
time of writing, five points that still need datasheet confirmation,
and the stock status of the new filter values, which could not be
queried and should be checked before ordering.
Parts:
- removed C210 (x2), C211 (x2): 100nF, Capacitor_SMD:C_0603_1608Metric, symbol Device:C
- added C210 (x2), C211 (x2): 100nF, Capacitor_SMD:C_0603_1608Metric, symbol Device:C
Connections:
- net +3V3: now also C210.1, C211.1
- net BUFCLK_N: now also C211.1
- net BUFCLK_P: now also C210.2
- net CLK80_DIV: now also C210.1
- net GND: now also C210.2, C211.2, C211.2

Commit message: Give each regulator the part number its rail needs
A fixed-output LDO carries its voltage in the part number. If the
number is wrong the schematic does not change: the netlist is correct,
ERC is clean, DRC is clean, and the rail comes up at the wrong
voltage.

U3 was specified as TPS7A2033. The last two digits are the output, so
33 is 3.3 V and 18 is 1.8 V. Its output feeds +1V8, which supplies the
FPGA's bank 6 and 3 VCCIO across twenty pads. The wiring was correct
and only the part number was wrong.

The six ADP150 regulators all carried the value "ADP150" and collapsed
into one BOM line under one code, which is the 2.5 V version. Their
outputs are 1.8, 1.8, 1.8, 2.5, 3.3 and 3.3 V. That line would have
put 2.5 V on both ADC supplies, and the AD9251 has an absolute maximum
of 2.0 V on AVDD. Each rail now names its own variant and the BOM has
separate lines.

regulator_denetim checks this class. It reads the voltage from the
part number, reads it from the rail name and compares them. It also
requires an LDO to have an input higher than its output by at least
the dropout voltage.
Parts:
- removed C210 (x2), C211 (x2): 100nF, Capacitor_SMD:C_0603_1608Metric, symbol Device:C
- added C210 (x2), C211 (x2): 100nF, Capacitor_SMD:C_0603_1608Metric, symbol Device:C
Connections:
- net +3V3: now also C210.1, C211.1
- net BUFCLK_N: now also C211.1
- net BUFCLK_P: now also C210.2
- net CLK80_DIV: now also C210.1
- net GND: now also C210.2, C211.2, C211.2
