File: hardware/kicad/A_main/03_adc.kicad_sch (KiCad schematic)
At the start: 59 parts, among them J20 SMA A1, J21 SMA B1, J22 SMA A2, J23 SMA B2, T1 ADT1-1WT+, T2 ADT1-1WT+, T3 ADT1-1WT+, T4 ADT1-1WT+, U10 LFE5U-25F-7BG256I, U20 AD9251BCPZ-80, U21 AD9251BCPZ-80

Commit message: Connect the pads that had no net
A symbol pin number must agree with the footprint pad number. If the
numbers do not agree, the net goes nowhere. The netlist removes it
and gives no message. ERC examines the schematic and sees a wire. DRC
does not count an unconnected pad as a violation. All three boards
showed zero ERC violations while 31 pads had no net.

Two of these faults stopped a board.

The footprint of the Ethernet PHY was for a different part. The
project used QFN-48 6x6 mm with 0.4 mm pitch. The RTL8211F(I)-CG is
WQFN-40-EP 5x5 mm. You cannot solder the part to that pad pattern.

The 25 MHz crystal had a 2-pin symbol on a 4-pad footprint. On a 3225
crystal the terminals are the diagonal pads 1 and 3. Pads 2 and 4 are
the metal can. XO went to pad 2. There was no crystal between XI and
XO, and thus neither PHY could make a clock.

The paddle of the AD9251 was pin 0 in the symbol and pad 65 in the
footprint. The paddle of the PE4312 was Pad against pad 21. The gas
discharge tubes had one electrode unconnected, because
Device:GDT_2Pin uses pins 1 and 3 but the varistor footprint uses
pads 1 and 2. A local footprint with pads 1 and 3 corrects this.

ped_denetim.py finds these faults on the board. yap.sh runs it before
the DSN export. The chain stops if a pad has no net.

The DSN export also changed. It declared In1 and In4 as power layers
but did not export the copper on them. The router thus believed that
the two ground planes were empty. It routed the 289 pins of GND as
traces on the signal layers. The planes now go out as conduction
areas.
Connections:
- net GND: now also U20.65 (GND), U21.65 (GND); no longer U20.0 (GND), U21.0 (GND)

Commit message: Correct the clearance test for the pre-routed traces
The clearance test used a circle for each pad. The radius was
max(width, height)/2. The corner of a rectangle is at
hypot(width, height)/2 from the center. The test thus made the pad
smaller than it is. On the 2.5 x 4.5 mm gate pad of a TO-247 the
difference is 2.250 mm against 2.574 mm.

The DRN_A trace was on the gate pad of Q10 with an overlap of 35 um.
This is a short circuit between the 50 V drain rail and the gate of a
100 W device. The search that finds the tee offset accepted this
route. The overlap is at a corner and 35 um wide. You cannot see it
on a plot.

The test now uses the real shape of the pad and the collision test of
pcbnew. It also uses the 300 um clearance and not only an overlap. A
trace that is 50 um from a pad is also not possible to manufacture.

Board D was built again. No trace is below 300 um and the smallest
gap is 0.537 mm. Boards A and C were correct.
Parts:
- removed C303, C307, C311, C315: 22pF, Capacitor_SMD:C_0603_1608Metric, symbol Device:C
- removed C316, C319: 1uF, Capacitor_SMD:C_0603_1608Metric, symbol Device:C
- removed C318, C321: 100nF, Capacitor_SMD:C_0603_1608Metric, symbol Device:C
- removed C400, C401, C402, C403, C404, C405, C406, C407, C408, C409, C410, C411, C412, C413, C414, C415, C420, C421, C422, C423, C424, C425, C426, C427: 100nF, Capacitor_SMD:C_0402_1005Metric, symbol Device:C
- removed C430, C431: 10uF, Capacitor_SMD:C_0402_1005Metric, symbol Device:C
- removed J20: SMA A1, Connector_Coaxial:SMA_Amphenol_132289_EdgeMount, symbol Connector:Conn_Coaxial
- removed J21: SMA B1, Connector_Coaxial:SMA_Amphenol_132289_EdgeMount, symbol Connector:Conn_Coaxial
- removed J22: SMA A2, Connector_Coaxial:SMA_Amphenol_132289_EdgeMount, symbol Connector:Conn_Coaxial
- removed J23: SMA B2, Connector_Coaxial:SMA_Amphenol_132289_EdgeMount, symbol Connector:Conn_Coaxial
- removed R300, R304, R308, R312: 49.9R 1%, Resistor_SMD:R_0603_1608Metric, symbol Device:R
- removed R301, R302, R305, R306, R309, R310, R313, R314: 33R 1%, Resistor_SMD:R_0603_1608Metric, symbol Device:R
- removed R317, R320: 10k 1%, Resistor_SMD:R_0603_1608Metric, symbol Device:R
- removed T1, T2, T3, T4: ADT1-1WT+, RF_Mini-Circuits:Mini-Circuits_CD542_H2.84mm, symbol dogrudan-sdr:ADT1-1WT
- removed U10: LFE5U-25F-7BG256I, Package_BGA:BGA-256_14.0x14.0mm_Layout16x16_P0.8mm_Ball0.45mm_Pad0.32mm_NSMD, symbol dogrudan-sdr:ECP5-BGA256
- removed U20, U21: AD9251BCPZ-80, Package_DFN_QFN:QFN-64-1EP_9x9mm_P0.5mm_EP4.7x4.7mm, symbol dogrudan-sdr:AD9251
Connections:
- no-connect marks 44 -> 0
Other:
- note added: "ADC x2 AD9251 x2 cogullamali, ADT1-1WT x4, banka 6 Baglantilar: ../NETLIST.md"
- note removed: "AD9251 ANALOG + SAAT — birim 1"
- note removed: "ANALOG ON UC — kanal basina bir trafo"
- note removed: "AVDD 8 pin x 2 cip = 16 adet 100nF + 2 adet toplu 10uF DRVDD 4 pin x 2 cip = 8 adet 100nF AVDD kondansatorleri ANALOG toprak adasinda, DRVDD'ninkiler dijital tarafta. Ikisini karistirmak ADC'nin gurultu tabanini yukseltir — bu kartta o taban aletin butun degeri."
- note removed: "AYRISTIRMA — pin basina, 0402"
- note removed: "BANKA 6 TAM DOLU: 32/32. ADC1 14 veri + DCO + OR = 16 ADC2 14 veri + DCO + OR = 16 Marj yok. Buraya bir sinyal daha gerekirse OR bayraklarindan biri feda edilir (FPGA'da doygunluk zaten tespit edilebiliyor). ** PIN ATAMASI GECICI ** — asagidaki eslesme banka 6'nin PL pinlerini sirayla dagitiyor. DCO hatlari SAAT-YETENEKLI pine dusmeli; hangi toplarin PCLK oldugu Lattice pinout CSV'sinden alinip b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"
- note removed: "COGULLAMA ACIK (SPI'dan). Cip basina 15 hat @160 MHz SDR, 30 hat @80 MHz yerine. Iki gerekce: 1. pin butcesi — cogullamasiz iki cip 60 pin, tutmuyor 2. GURULTU — 30 yerine 15 anahtarlanan hat, analog ucun yaninda IKI CIP DE BANKA 6'DA. Ayni bankada olmalari zamanlama eslesmesi ve faz uyumu icin sart. DCO saat-yetenekli pine gidecek (Lattice pinout'undan secilecek). Kanal sirasi (once A mi B mi) S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"
- note removed: "DIJITAL CIKIS — birim 2, cogullamali"
- note removed: "FPGA BANKA 6 — verinin gittigi yer"
- note removed: "GUC VE KONTROL — birim 4"
- note removed: "KANAL B CIKISLARI — birim 3, COGULLAMA MODUNDA BOSTA"
- note removed: "RC AGI BANDA GORE DEGISIYOR — AD9251 Tablo 9: 0-70 MHz giris R seri 33R, C dif 22 pF 70-200 MHz giris R seri 125R, C dif ACIK (takilmiyor) Bu alet hem tabanbant hem alt-ornekleme yapiyor, tek deger ikisine birden uymuyor. Sematikte 33R + 22pF cizili (HF/6m kullanimi). VHF/UHF alt-ornekleme icin ayni ayak izlerine 125R takilip C sokuluyor. Hepsi 0603, kart degismiyor — hangi bandda calisilacagi mo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"
- note removed: "SAAT: ADCLK_U20_P/N ve ADCLK_U21_P/N, 02_clock'taki ADCLK846'nin 1 ve 2 numarali cikislari. LVDS, dogrudan baglaniyor (AD9251 saat girisi PECL/LVDS/1.8V CMOS kabul ediyor). IKI YOL ES UZUNLUKTA CEKILECEK."
- note removed: "SENSE (56) DOGRUDAN AGND'ye: dahili 1.0 V referans secilir. VREF (55) 1uF ile AGND'ye. RBIAS (58) 10k %1 — %5 direnc olcek hatasi yapar, tam deger onemli. VCM CIPE OZEL: U20'ninki A1/B1 trafolarina, U21'inki A2/B2'ye. Ortak baglamak iki cikisi paralel etmek olurdu. Pin 0 = exposed paddle, cipin TEK toprak baglantisi. Termal via dizisiyle dogrudan toprak duzlemine — datasheet 'must be soldered'."
- note removed: "SMA (C kartindan gelen filtreli RF) -> ADT1-1WT+ 1:1 -> VIN cifti Orta uc VCM'e: ortak mod 0.9 V. Giris kapasitansi 6 pF. VIN cifti ES BOY, SIKI CIFT, KISA — dort kanalin faz uyumu buradaki simetriye bagli."
- note removed: "SPI: SDIO ve SCLK ORTAK, ~CSB cip basina ayri (banka 0). ~OEB dogrudan AGND'ye — cikislar hep acik, kontrol edilecek bir sey yok. ** ADC_SYNC IKI CIPE DE ORTAK VE ES UZUNLUKTA ** Iki ADC'nin ic bolucusunu ayni anda sifirliyor. Dort kanalin faz uyumu — yani bu aletin butun ayirt edici ozelligi: gurultu iptali, yon bulma, isin sekillendirme — bu tek hattin simetrisine bagli. Yol uzunluklari esitlen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"

Commit message: Correct the schematic faults that ERC cannot find
An agent examined the three schematics against the datasheets. ERC
reported zero violations before and after this work. None of these
faults are visible to ERC.

The comparator for the external 10 MHz reference was in shutdown. The
SHDN pin of the TLV3501 went to +3V3. Sixteen DRV8833 devices had VCP
and VINT unconnected. Without the charge pump none of the 28 filter
relays can latch. Seven regulators had no decoupling capacitor within
18 mm to 94 mm. On board D the nearest +12V capacitor to an LM358 was
227 mm away on a 275 mm board.

The PE4312 devices had no series 10k resistor on pin 3. The datasheet
makes this necessary for the attenuation accuracy. Their exposed pad
was 2.6 mm against 2.15 mm. The BOM did not give the load capacitance
of the crystal. This work added 60 parts and changed 4 footprints.

The worst fault was in the tool chain. lib/gen_symbols.py still made
the old pin numbers. The five corrections went into the symbol
library by hand and not into its generator. A new library would have
removed all of them.

The thermal vias are now a decision from the measured clearance and
the dissipation. This work removed them from the PE4312, the RTL8211F
and the ADCLK846. They stay on the DRV8833 and on the LM5164, which
is a 1 W buck converter.

Two checks are new. sema_denetim compares the pin names with the
nets. netlist_denetim locks 22 pin-to-net expectations from the
datasheets and does not need a board.

The boards were built again with these corrections. The chain now
adds the test points: 10 on board A, 7 on board C and 15 on board D.
Each board has 3 fiducials. Every pad has a net.
Parts:
- added C303, C307, C311, C315: 22pF, Capacitor_SMD:C_0603_1608Metric, symbol Device:C
- added C316, C319: 1uF, Capacitor_SMD:C_0603_1608Metric, symbol Device:C
- added C318, C321: 100nF, Capacitor_SMD:C_0603_1608Metric, symbol Device:C
- added C400, C401, C402, C403, C404, C405, C406, C407, C408, C409, C410, C411, C412, C413, C414, C415, C420, C421, C422, C423, C424, C425, C426, C427: 100nF, Capacitor_SMD:C_0402_1005Metric, symbol Device:C
- added C430, C431: 10uF, Capacitor_SMD:C_0402_1005Metric, symbol Device:C
- added J20: SMA A1, Connector_Coaxial:SMA_Amphenol_132289_EdgeMount, symbol Connector:Conn_Coaxial
- added J21: SMA B1, Connector_Coaxial:SMA_Amphenol_132289_EdgeMount, symbol Connector:Conn_Coaxial
- added J22: SMA A2, Connector_Coaxial:SMA_Amphenol_132289_EdgeMount, symbol Connector:Conn_Coaxial
- added J23: SMA B2, Connector_Coaxial:SMA_Amphenol_132289_EdgeMount, symbol Connector:Conn_Coaxial
- added R300, R304, R308, R312: 49.9R 1%, Resistor_SMD:R_0603_1608Metric, symbol Device:R
- added R301, R302, R305, R306, R309, R310, R313, R314: 33R 1%, Resistor_SMD:R_0603_1608Metric, symbol Device:R
- added R317, R320: 10k 1%, Resistor_SMD:R_0603_1608Metric, symbol Device:R
- added T1, T2, T3, T4: ADT1-1WT+, RF_Mini-Circuits:Mini-Circuits_CD542_H2.84mm, symbol dogrudan-sdr:ADT1-1WT
- added U10: LFE5U-25F-7BG256I, Package_BGA:BGA-256_14.0x14.0mm_Layout16x16_P0.8mm_Ball0.45mm_Pad0.32mm_NSMD, symbol dogrudan-sdr:ECP5-BGA256
- added U20, U21: AD9251BCPZ-80, Package_DFN_QFN:QFN-64-1EP_9x9mm_P0.5mm_EP4.7x4.7mm, symbol dogrudan-sdr:AD9251
Connections:
- new net +1V8: U10.J6 (VCCIO6_1), U10.J7 (VCCIO6_2)
- new net +1V8_A: C400.1, C401.1, C402.1, C403.1, C404.1, C405.1, C406.1, C407.1, C408.1, C409.1, C410.1, C411.1, C412.1, C413.1, C414.1, C415.1, C430.1, C431.1, U20.49 (AVDD), U20.50 (AVDD), U20.53 (AVDD), U20.54 (AVDD), U20.59 (AVDD), U20.60 (AVDD), U20.63 (AVDD), U20.64 (AVDD), U21.49 (AVDD), U21.50 (AVDD), U21.53 (AVDD), U21.54 (AVDD), U21.59 (AVDD), U21.60 (AVDD), U21.63 (AVDD), U21.64 (AVDD)
- new net +1V8_D: C420.1, C421.1, C422.1, C423.1, C424.1, C425.1, C426.1, C427.1, U20.10 (DRVDD), U20.19 (DRVDD), U20.28 (DRVDD), U20.37 (DRVDD), U21.10 (DRVDD), U21.19 (DRVDD), U21.28 (DRVDD), U21.37 (DRVDD)
- new net ADC1_D0: U10.M6 (PL47A), U20.27 (D0A)
- new net ADC1_D1: U10.N1 (PL32A), U20.29 (D1A)
- new net ADC1_D10: U10.L3 (PL32C), U20.39 (D10A)
- new net ADC1_D11: U10.L2 (PL26B), U20.40 (D11A)
- new net ADC1_D12: U10.L1 (PL26A), U20.41 (D12A)
- new net ADC1_D13: U10.K5 (PL29B), U20.42 (D13A)
- new net ADC1_D2: U10.N3 (PL35D), U20.30 (D2A)
- new net ADC1_D3: U10.N4 (PL38A), U20.31 (D3A)
- new net ADC1_D4: U10.P1 (PL35A), U20.32 (D4A)
- new net ADC1_D5: U10.M5 (PL44C), U20.33 (D5A)
- new net ADC1_D6: U10.M4 (PL35C), U20.34 (D6A)
- new net ADC1_D7: U10.M3 (PL32D), U20.35 (D7A)
- new net ADC1_D8: U10.L5 (PL29D), U20.36 (D8A)
- new net ADC1_D9: U10.L4 (PL29C), U20.38 (D9A)
- new net ADC1_DCO: U10.M1 (PL26C), U20.24 (DCOA)
- new net ADC1_OR: U10.K4 (PL29A), U20.43 (ORA)
- new net ADC1_nCSB: U20.46 (~{CSB})
- new net ADC2_D0: U10.R1 (PL35B), U21.27 (D0A)
- new net ADC2_D1: U10.P2 (PL32B), U21.29 (D1A)
- new net ADC2_D10: U10.N5 (PL44D), U21.39 (D10A)
- new net ADC2_D11: U10.P5 (PL47D), U21.40 (D11A)
- new net ADC2_D12: U10.R5 (PL44A), U21.41 (D12A)
- new net ADC2_D13: U10.N6 (PL47B), U21.42 (D13A)
- new net ADC2_D2: U10.R2 (PL38C), U21.30 (D2A)
- new net ADC2_D3: U10.T2 (PL38D), U21.31 (D3A)
- new net ADC2_D4: U10.P3 (PL38B), U21.32 (D4A)
- new net ADC2_D5: U10.R3 (PL41B), U21.33 (D5A)
- new net ADC2_D6: U10.T3 (PL41D), U21.34 (D6A)
- new net ADC2_D7: U10.P4 (PL41A), U21.35 (D7A)
- new net ADC2_D8: U10.R4 (PL41C), U21.36 (D8A)
- new net ADC2_D9: U10.T4 (PL44B), U21.38 (D9A)
- new net ADC2_DCO: U10.M2 (PL26D), U21.24 (DCOA)
- new net ADC2_OR: U10.P6 (PL47C), U21.43 (ORA)
- new net ADC2_nCSB: U21.46 (~{CSB})
- new net ADCLK_U20_N: U20.2 (CLK-)
- new net ADCLK_U20_P: U20.1 (CLK+)
- new net ADCLK_U21_N: U21.2 (CLK-)
- new net ADCLK_U21_P: U21.1 (CLK+)
- new net ADC_SCLK: U20.45 (SCLK/DFS), U21.45 (SCLK/DFS)
- new net ADC_SDIO: U20.44 (SDIO/DCS), U21.44 (SDIO/DCS)
- new net ADC_SYNC: U20.3 (SYNC), U21.3 (SYNC)
- new net GND: C316.2, C318.2, C319.2, C321.2, C400.2, C401.2, C402.2, C403.2, C404.2, C405.2, C406.2, C407.2, C408.2, C409.2, C410.2, C411.2, C412.2, C413.2, C414.2, C415.2, C420.2, C421.2, C422.2, C423.2, C424.2, C425.2, C426.2, C427.2, C430.2, C431.2, J20.2 (Ext), J21.2 (Ext), J22.2 (Ext), J23.2 (Ext), R300.2, R304.2, R308.2, R312.2, R317.2, R320.2, T1.1 (PRI), T2.1 (PRI), T3.1 (PRI), T4.1 (PRI), U20.47 (~{OEB}), U20.48 (PDWN), U20.56 (SENSE), U20.65 (GND), U21.47 (~{OEB}), U21.48 (PDWN), U21.56 (SENSE), U21.65 (GND)
- new net RBIAS_U20: R317.1, U20.58 (RBIAS)
- new net RBIAS_U21: R320.1, U21.58 (RBIAS)
- new net RF_A1: J20.1 (In), R300.1, T1.3 (PRI_DOT)
- new net RF_A2: J22.1 (In), R308.1, T3.3 (PRI_DOT)
- new net RF_B1: J21.1 (In), R304.1, T2.3 (PRI_DOT)
- new net RF_B2: J23.1 (In), R312.1, T4.3 (PRI_DOT)
- new net SEC_A1_N: R302.1, T1.4 (SEC)
- new net SEC_A1_P: R301.1, T1.6 (SEC_DOT)
- new net SEC_A2_N: R310.1, T3.4 (SEC)
- new net SEC_A2_P: R309.1, T3.6 (SEC_DOT)
- new net SEC_B1_N: R306.1, T2.4 (SEC)
- new net SEC_B1_P: R305.1, T2.6 (SEC_DOT)
- new net SEC_B2_N: R314.1, T4.4 (SEC)
- new net SEC_B2_P: R313.1, T4.6 (SEC_DOT)
- new net VCM_U20: C318.1, T1.2 (SEC_CT), T2.2 (SEC_CT), U20.57 (VCM)
- new net VCM_U21: C321.1, T3.2 (SEC_CT), T4.2 (SEC_CT), U21.57 (VCM)
- new net VIN_A1_N: C303.2, R302.2, U20.52 (VIN-A)
- new net VIN_A1_P: C303.1, R301.2, U20.51 (VIN+A)
- new net VIN_A2_N: C311.2, R310.2, U21.52 (VIN-A)
- new net VIN_A2_P: C311.1, R309.2, U21.51 (VIN+A)
- new net VIN_B1_N: C307.2, R306.2, U20.61 (VIN-B)
- new net VIN_B1_P: C307.1, R305.2, U20.62 (VIN+B)
- new net VIN_B2_N: C315.2, R314.2, U21.61 (VIN-B)
- new net VIN_B2_P: C315.1, R313.2, U21.62 (VIN+B)
- new net VREF_U20: C316.1, U20.55 (VREF)
- new net VREF_U21: C319.1, U21.55 (VREF)
- no-connect marks 0 -> 44
Other:
- note added: "AD9251 ANALOG + SAAT — birim 1"
- note added: "ANALOG ON UC — kanal basina bir trafo"
- note added: "AVDD 8 pin x 2 cip = 16 adet 100nF + 2 adet toplu 10uF DRVDD 4 pin x 2 cip = 8 adet 100nF AVDD kondansatorleri ANALOG toprak adasinda, DRVDD'ninkiler dijital tarafta. Ikisini karistirmak ADC'nin gurultu tabanini yukseltir — bu kartta o taban aletin butun degeri."
- note added: "AYRISTIRMA — pin basina, 0402"
- note added: "BANKA 6 TAM DOLU: 32/32. ADC1 14 veri + DCO + OR = 16 ADC2 14 veri + DCO + OR = 16 Marj yok. Buraya bir sinyal daha gerekirse OR bayraklarindan biri feda edilir (FPGA'da doygunluk zaten tespit edilebiliyor). ** PIN ATAMASI GECICI ** — asagidaki eslesme banka 6'nin PL pinlerini sirayla dagitiyor. DCO hatlari SAAT-YETENEKLI pine dusmeli; hangi toplarin PCLK oldugu Lattice pinout CSV'sinden alinip b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"
- note added: "COGULLAMA ACIK (SPI'dan). Cip basina 15 hat @160 MHz SDR, 30 hat @80 MHz yerine. Iki gerekce: 1. pin butcesi — cogullamasiz iki cip 60 pin, tutmuyor 2. GURULTU — 30 yerine 15 anahtarlanan hat, analog ucun yaninda IKI CIP DE BANKA 6'DA. Ayni bankada olmalari zamanlama eslesmesi ve faz uyumu icin sart. DCO saat-yetenekli pine gidecek (Lattice pinout'undan secilecek). Kanal sirasi (once A mi B mi) S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"
- note added: "DIJITAL CIKIS — birim 2, cogullamali"
- note added: "FPGA BANKA 6 — verinin gittigi yer"
- note added: "GUC VE KONTROL — birim 4"
- note added: "KANAL B CIKISLARI — birim 3, COGULLAMA MODUNDA BOSTA"
- note added: "RC AGI BANDA GORE DEGISIYOR — AD9251 Tablo 9: 0-70 MHz giris R seri 33R, C dif 22 pF 70-200 MHz giris R seri 125R, C dif ACIK (takilmiyor) Bu alet hem tabanbant hem alt-ornekleme yapiyor, tek deger ikisine birden uymuyor. Sematikte 33R + 22pF cizili (HF/6m kullanimi). VHF/UHF alt-ornekleme icin ayni ayak izlerine 125R takilip C sokuluyor. Hepsi 0603, kart degismiyor — hangi bandda calisilacagi mo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"
- note added: "SAAT: ADCLK_U20_P/N ve ADCLK_U21_P/N, 02_clock'taki ADCLK846'nin 1 ve 2 numarali cikislari. LVDS, dogrudan baglaniyor (AD9251 saat girisi PECL/LVDS/1.8V CMOS kabul ediyor). IKI YOL ES UZUNLUKTA CEKILECEK."
- note added: "SENSE (56) DOGRUDAN AGND'ye: dahili 1.0 V referans secilir. VREF (55) 1uF ile AGND'ye. RBIAS (58) 10k %1 — %5 direnc olcek hatasi yapar, tam deger onemli. VCM CIPE OZEL: U20'ninki A1/B1 trafolarina, U21'inki A2/B2'ye. Ortak baglamak iki cikisi paralel etmek olurdu. Pin 0 = exposed paddle, cipin TEK toprak baglantisi. Termal via dizisiyle dogrudan toprak duzlemine — datasheet 'must be soldered'."
- note added: "SMA (C kartindan gelen filtreli RF) -> ADT1-1WT+ 1:1 -> VIN cifti Orta uc VCM'e: ortak mod 0.9 V. Giris kapasitansi 6 pF. VIN cifti ES BOY, SIKI CIFT, KISA — dort kanalin faz uyumu buradaki simetriye bagli."
- note added: "SPI: SDIO ve SCLK ORTAK, ~CSB cip basina ayri (banka 0). ~OEB dogrudan AGND'ye — cikislar hep acik, kontrol edilecek bir sey yok. ** ADC_SYNC IKI CIPE DE ORTAK VE ES UZUNLUKTA ** Iki ADC'nin ic bolucusunu ayni anda sifirliyor. Dort kanalin faz uyumu — yani bu aletin butun ayirt edici ozelligi: gurultu iptali, yon bulma, isin sekillendirme — bu tek hattin simetrisine bagli. Yol uzunluklari esitlen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"
- note removed: "ADC x2 AD9251 x2 cogullamali, ADT1-1WT x4, banka 6 Baglantilar: ../NETLIST.md"
