File: hardware/kicad/A_main/05_sdram.kicad_sch (KiCad schematic)
At the start: 10 parts, among them U10 LFE5U-25F-7BG256I, U50 W9825G6KH-6I

Commit message: Correct the clearance test for the pre-routed traces
The clearance test used a circle for each pad. The radius was
max(width, height)/2. The corner of a rectangle is at
hypot(width, height)/2 from the center. The test thus made the pad
smaller than it is. On the 2.5 x 4.5 mm gate pad of a TO-247 the
difference is 2.250 mm against 2.574 mm.

The DRN_A trace was on the gate pad of Q10 with an overlap of 35 um.
This is a short circuit between the 50 V drain rail and the gate of a
100 W device. The search that finds the tee offset accepted this
route. The overlap is at a corner and 35 um wide. You cannot see it
on a plot.

The test now uses the real shape of the pad and the collision test of
pcbnew. It also uses the 300 um clearance and not only an overlap. A
trace that is 50 um from a pad is also not possible to manufacture.

Board D was built again. No trace is below 300 um and the smallest
gap is 0.537 mm. Boards A and C were correct.
Parts:
- removed C500, C501, C502, C503, C504, C505: 100nF, Capacitor_SMD:C_0603_1608Metric, symbol Device:C
- removed C506: 10uF, Capacitor_SMD:C_0603_1608Metric, symbol Device:C
- removed R550: 22R, Resistor_SMD:R_0603_1608Metric, symbol Device:R
- removed U10: LFE5U-25F-7BG256I, Package_BGA:BGA-256_14.0x14.0mm_Layout16x16_P0.8mm_Ball0.45mm_Pad0.32mm_NSMD, symbol dogrudan-sdr:ECP5-BGA256
- removed U50: W9825G6KH-6I, Package_SO:TSOP-II-54_22.2x10.16mm_P0.8mm, symbol dogrudan-sdr:W9825G6KH
Connections:
- no-connect marks 1 -> 0
Other:
- note added: "SDRAM W9825G6KH-6I 32MB, banka 7 + 0 Baglantilar: ../NETLIST.md"
- note removed: "ADRES VE KOMUT — birim 2"
- note removed: "BANKA 0'a TASAN 7 SINYAL"
- note removed: "BANKA 7 TAM DOLU: 16 DQ + 9 adres + 6 komut + CLK = 32/32. VERI YOLU VE STROBE TEK BANKADA. Zamanlama acisindan onemli olan bu: aynı banka = ayni IO gerilimi, ayni surucu gecikmesi, ayni sicaklik davranisi. Adresin bir kismini bankaya sigmadigi icin banka 0'a tasidik — adres hatlarinin skew'i komut cevriminde tolere ediliyor, veri yolununki edilmiyor."
- note removed: "CLK hattinda 22R SERI sonlandirma, FPGA cikisina yakin. Tek yuk oldugu icin seri sonlandirma yetiyor; yansimasi kaynaga donunce sonuyor. 166 MHz'de yol uzunlugu farki setup marjini yiyor — CLK ile DQ grubunu es boy cek."
- note removed: "FPGA BANKA 7 — veri yolu"
- note removed: "GUC"
- note removed: "Patlama yakalama icin. ECP5'in dahili blok RAM'i 1008 kbit = 126 KB, tam hizda 0.79 ms eder — meteor olayinin sadece on kenarini yakalar. 32 MB / 160 MB/s = 200 ms. 250 kat. DDR3 DEGIL, SDR. Kasten: DDR3'un fly-by yonlendirmesi, ODT'si ve kalibrasyonu rev A'ya agir yuk. SDR tek cip, duz yonlendirme, LiteDRAM destekliyor."
- note removed: "SAAT SONLANDIRMA"
- note removed: "SDRAM — W9825G6KH-6I, 32 MB"
- note removed: "SD_A9, SD_A10, SD_A11, SD_A12, SD_BA0, SD_BA1, SD_UDQM ECP5 sembolunun banka 0 birimi BU SAYFADA DEGIL, 08_control'de. KiCad'de cok birimli bir sembolun her birimi projede BIR KEZ yerlestirilebiliyor; birimi buraya da koyunca kalan 17 pini 'baglanmamis' diye isaretledi. Sinyaller etiketle gidiyor, cizim 08_control'de kapaniyor. Neden banka 0'a tasti: banka 7'nin 32 pini DQ + 9 adres + komut ile d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"
- note removed: "VDD ve VDDQ ayni +3V3 rayindan. Ayristirma: her VDD/VDDQ ciftine bir 100nF (alti adet) + toplu 10uF. 166 MHz'de akim adimlari keskin; kondansatorler bacaga en yakin, viasi dogrudan duzleme."
- note removed: "VERI YOLU — birim 1, banka 7"

Commit message: Correct the schematic faults that ERC cannot find
An agent examined the three schematics against the datasheets. ERC
reported zero violations before and after this work. None of these
faults are visible to ERC.

The comparator for the external 10 MHz reference was in shutdown. The
SHDN pin of the TLV3501 went to +3V3. Sixteen DRV8833 devices had VCP
and VINT unconnected. Without the charge pump none of the 28 filter
relays can latch. Seven regulators had no decoupling capacitor within
18 mm to 94 mm. On board D the nearest +12V capacitor to an LM358 was
227 mm away on a 275 mm board.

The PE4312 devices had no series 10k resistor on pin 3. The datasheet
makes this necessary for the attenuation accuracy. Their exposed pad
was 2.6 mm against 2.15 mm. The BOM did not give the load capacitance
of the crystal. This work added 60 parts and changed 4 footprints.

The worst fault was in the tool chain. lib/gen_symbols.py still made
the old pin numbers. The five corrections went into the symbol
library by hand and not into its generator. A new library would have
removed all of them.

The thermal vias are now a decision from the measured clearance and
the dissipation. This work removed them from the PE4312, the RTL8211F
and the ADCLK846. They stay on the DRV8833 and on the LM5164, which
is a 1 W buck converter.

Two checks are new. sema_denetim compares the pin names with the
nets. netlist_denetim locks 22 pin-to-net expectations from the
datasheets and does not need a board.

The boards were built again with these corrections. The chain now
adds the test points: 10 on board A, 7 on board C and 15 on board D.
Each board has 3 fiducials. Every pad has a net.
Parts:
- added C500, C501, C502, C503, C504, C505: 100nF, Capacitor_SMD:C_0603_1608Metric, symbol Device:C
- added C506: 10uF, Capacitor_SMD:C_0603_1608Metric, symbol Device:C
- added R550: 22R, Resistor_SMD:R_0603_1608Metric, symbol Device:R
- added U10: LFE5U-25F-7BG256I, Package_BGA:BGA-256_14.0x14.0mm_Layout16x16_P0.8mm_Ball0.45mm_Pad0.32mm_NSMD, symbol dogrudan-sdr:ECP5-BGA256
- added U50: W9825G6KH-6I, Package_SO:TSOP-II-54_22.2x10.16mm_P0.8mm, symbol dogrudan-sdr:W9825G6KH
Connections:
- new net +3V3: C500.1, C501.1, C502.1, C503.1, C504.1, C505.1, C506.1, U10.H6 (VCCIO7_1), U10.H7 (VCCIO7_2), U50.1 (VDD), U50.14 (VDD), U50.27 (VDD), U50.3 (VDDQ), U50.43 (VDDQ), U50.49 (VDDQ), U50.9 (VDDQ)
- new net GND: C500.2, C501.2, C502.2, C503.2, C504.2, C505.2, C506.2, U50.12 (VSSQ), U50.28 (VSS), U50.41 (VSS), U50.46 (VSSQ), U50.52 (VSSQ), U50.54 (VSS), U50.6 (VSSQ)
- new net SD_A0: U10.E2 (PL8B), U50.23 (A0)
- new net SD_A1: U10.F2 (PL11C), U50.24 (A1)
- new net SD_A10: U50.22 (A10)
- new net SD_A11: U50.35 (A11)
- new net SD_A12: U50.36 (A12)
- new net SD_A2: U10.G2 (PL14B), U50.25 (A2)
- new net SD_A3: U10.H2 (PL20B), U50.26 (A3)
- new net SD_A4: U10.G4 (PL11B), U50.29 (A4)
- new net SD_A5: U10.H4 (PL17B), U50.30 (A5)
- new net SD_A6: U10.F5 (PL8D), U50.31 (A6)
- new net SD_A7: U10.G5 (PL11A), U50.32 (A7)
- new net SD_A8: U10.H5 (PL17A), U50.33 (A8)
- new net SD_A9: U50.34 (A9)
- new net SD_BA0: U50.20 (BA0)
- new net SD_BA1: U50.21 (BA1)
- new net SD_CKE: U10.J5 (PL17D), U50.37 (CKE)
- new net SD_CLK: R550.2, U50.38 (CLK)
- new net SD_CLK_FPGA: R550.1, U10.K1 (PL23C)
- new net SD_DQ0: U10.B1 (PL2A), U50.2 (DQ0)
- new net SD_DQ1: U10.C1 (PL5A), U50.4 (DQ1)
- new net SD_DQ10: U10.D3 (PL2D), U50.45 (DQ10)
- new net SD_DQ11: U10.E3 (PL5C), U50.47 (DQ11)
- new net SD_DQ12: U10.F3 (PL5D), U50.48 (DQ12)
- new net SD_DQ13: U10.G3 (PL14C), U50.50 (DQ13)
- new net SD_DQ14: U10.H3 (PL14D), U50.51 (DQ14)
- new net SD_DQ15: U10.F4 (PL8C), U50.53 (DQ15)
- new net SD_DQ2: U10.D1 (PL8A), U50.5 (DQ2)
- new net SD_DQ3: U10.E1 (PL11D), U50.7 (DQ3)
- new net SD_DQ4: U10.F1 (PL14A), U50.8 (DQ4)
- new net SD_DQ5: U10.G1 (PL20A), U50.10 (DQ5)
- new net SD_DQ6: U10.B2 (PL2B), U50.11 (DQ6)
- new net SD_DQ7: U10.C2 (PL5B), U50.13 (DQ7)
- new net SD_DQ8: U10.K2 (PL23D), U50.42 (DQ8)
- new net SD_DQ9: U10.C3 (PL2C), U50.44 (DQ9)
- new net SD_LDQM: U10.K3 (PL20D), U50.15 (LDQM)
- new net SD_UDQM: U50.39 (UDQM)
- new net SD_nCAS: U10.J3 (PL20C), U50.17 (~{CAS})
- new net SD_nCS: U10.J1 (PL23A), U50.19 (~{CS})
- new net SD_nRAS: U10.J2 (PL23B), U50.18 (~{RAS})
- new net SD_nWE: U10.J4 (PL17C), U50.16 (~{WE})
- no-connect marks 0 -> 1
Other:
- note added: "ADRES VE KOMUT — birim 2"
- note added: "BANKA 0'a TASAN 7 SINYAL"
- note added: "BANKA 7 TAM DOLU: 16 DQ + 9 adres + 6 komut + CLK = 32/32. VERI YOLU VE STROBE TEK BANKADA. Zamanlama acisindan onemli olan bu: aynı banka = ayni IO gerilimi, ayni surucu gecikmesi, ayni sicaklik davranisi. Adresin bir kismini bankaya sigmadigi icin banka 0'a tasidik — adres hatlarinin skew'i komut cevriminde tolere ediliyor, veri yolununki edilmiyor."
- note added: "CLK hattinda 22R SERI sonlandirma, FPGA cikisina yakin. Tek yuk oldugu icin seri sonlandirma yetiyor; yansimasi kaynaga donunce sonuyor. 166 MHz'de yol uzunlugu farki setup marjini yiyor — CLK ile DQ grubunu es boy cek."
- note added: "FPGA BANKA 7 — veri yolu"
- note added: "GUC"
- note added: "Patlama yakalama icin. ECP5'in dahili blok RAM'i 1008 kbit = 126 KB, tam hizda 0.79 ms eder — meteor olayinin sadece on kenarini yakalar. 32 MB / 160 MB/s = 200 ms. 250 kat. DDR3 DEGIL, SDR. Kasten: DDR3'un fly-by yonlendirmesi, ODT'si ve kalibrasyonu rev A'ya agir yuk. SDR tek cip, duz yonlendirme, LiteDRAM destekliyor."
- note added: "SAAT SONLANDIRMA"
- note added: "SDRAM — W9825G6KH-6I, 32 MB"
- note added: "SD_A9, SD_A10, SD_A11, SD_A12, SD_BA0, SD_BA1, SD_UDQM ECP5 sembolunun banka 0 birimi BU SAYFADA DEGIL, 08_control'de. KiCad'de cok birimli bir sembolun her birimi projede BIR KEZ yerlestirilebiliyor; birimi buraya da koyunca kalan 17 pini 'baglanmamis' diye isaretledi. Sinyaller etiketle gidiyor, cizim 08_control'de kapaniyor. Neden banka 0'a tasti: banka 7'nin 32 pini DQ + 9 adres + komut ile d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"
- note added: "VDD ve VDDQ ayni +3V3 rayindan. Ayristirma: her VDD/VDDQ ciftine bir 100nF (alti adet) + toplu 10uF. 166 MHz'de akim adimlari keskin; kondansatorler bacaga en yakin, viasi dogrudan duzleme."
- note added: "VERI YOLU — birim 1, banka 7"
- note removed: "SDRAM W9825G6KH-6I 32MB, banka 7 + 0 Baglantilar: ../NETLIST.md"
