File: hardware/kicad/A_main/06_ethernet.kicad_sch (KiCad schematic)
At the start: 55 parts, among them J40 HR911130A, J41 HR911130A, U10 LFE5U-25F-7BG256I, U40 RTL8211FI-CG, U41 RTL8211FI-CG, Y610 25MHz, Y626 25MHz

Commit message: Connect the pads that had no net
A symbol pin number must agree with the footprint pad number. If the
numbers do not agree, the net goes nowhere. The netlist removes it
and gives no message. ERC examines the schematic and sees a wire. DRC
does not count an unconnected pad as a violation. All three boards
showed zero ERC violations while 31 pads had no net.

Two of these faults stopped a board.

The footprint of the Ethernet PHY was for a different part. The
project used QFN-48 6x6 mm with 0.4 mm pitch. The RTL8211F(I)-CG is
WQFN-40-EP 5x5 mm. You cannot solder the part to that pad pattern.

The 25 MHz crystal had a 2-pin symbol on a 4-pad footprint. On a 3225
crystal the terminals are the diagonal pads 1 and 3. Pads 2 and 4 are
the metal can. XO went to pad 2. There was no crystal between XI and
XO, and thus neither PHY could make a clock.

The paddle of the AD9251 was pin 0 in the symbol and pad 65 in the
footprint. The paddle of the PE4312 was Pad against pad 21. The gas
discharge tubes had one electrode unconnected, because
Device:GDT_2Pin uses pins 1 and 3 but the varistor footprint uses
pads 1 and 2. A local footprint with pads 1 and 3 corrects this.

ped_denetim.py finds these faults on the board. yap.sh runs it before
the DSN export. The chain stops if a pad has no net.

The DSN export also changed. It declared In1 and In4 as power layers
but did not export the copper on them. The router thus believed that
the two ground planes were empty. It routed the 289 pins of GND as
traces on the signal layers. The planes now go out as conduction
areas.
Parts:
- removed Y610, Y626: 25MHz, Crystal:Crystal_SMD_3225-4Pin_3.2x2.5mm, symbol Device:Crystal
- added R692: 0R, Resistor_SMD:R_0603_1608Metric, symbol Device:R
- added Y610, Y626: 25MHz, Crystal:Crystal_SMD_3225-4Pin_3.2x2.5mm, symbol Device:Crystal_GND24
- U40, U41: footprint Package_DFN_QFN:QFN-48-1EP_6x6mm_P0.4mm_EP4.6x4.6mm -> Package_DFN_QFN:QFN-40-1EP_5x5mm_P0.4mm_EP3.6x3.6mm_ThermalVias
Connections:
- net CHASSIS: now also J40.SH1 (SHIELD), J40.SH2 (SHIELD), J40.SH3 (SHIELD), J40.SH4 (SHIELD), J41.SH1 (SHIELD), J41.SH2 (SHIELD), J41.SH3 (SHIELD), J41.SH4 (SHIELD), R692.1
- net GND: now also R692.2, Y610.2 (G), Y610.4 (G), Y626.2 (G), Y626.4 (G)
- net PHY1_XI: now also Y610.1
- net PHY1_XO: now also Y610.3
- net PHY2_XI: now also Y626.1
- net PHY2_XO: now also Y626.3
Other:
- note added: "SASE BAGI — RJ45 kalkani ve orta uc dugumu CHASSIS'te; CHASSIS topraga TEK NOKTADAN, R692 (0R) ile bagli. Montaj delikleri bu kartta KAPLAMASIZ: sase referansi C kartinda, orada anten konnektorlerinin dibindeki delik kaplamali ve GND'de. Iki karttan da kasaya baglanirsa toprak dongusu olusur."

Commit message: Remove the pads that have no copper from the DSN export
The router reported the same 220 clearance violations in each pass.
At the same time the number of unrouted connections decreased. The
violations were thus in the input and not in the routing.

The -1EP footprints of KiCad put four paste apertures on the exposed
pad. These apertures stop full paste coverage and they have no copper
layer. The DSN export put them on the top copper layer. The image of
U51 in the DSN had 21 pins: 17 correct pins and four unconnected
copper islands in the exposed pad. These islands are always in
conflict with the pad and they close the area below it.

The export now removes a pad that has no copper layer. The image of
U51 has 17 pins. The violations on board D decreased from 220 to 152.
Parts:
- Y610, Y626: value 25MHz -> 25MHz CL12pF

Commit message: Correct the clearance test for the pre-routed traces
The clearance test used a circle for each pad. The radius was
max(width, height)/2. The corner of a rectangle is at
hypot(width, height)/2 from the center. The test thus made the pad
smaller than it is. On the 2.5 x 4.5 mm gate pad of a TO-247 the
difference is 2.250 mm against 2.574 mm.

The DRN_A trace was on the gate pad of Q10 with an overlap of 35 um.
This is a short circuit between the 50 V drain rail and the gate of a
100 W device. The search that finds the tee offset accepted this
route. The overlap is at a corner and 35 um wide. You cannot see it
on a plot.

The test now uses the real shape of the pad and the collision test of
pcbnew. It also uses the 300 um clearance and not only an overlap. A
trace that is 50 um from a pad is also not possible to manufacture.

Board D was built again. No trace is below 300 um and the smallest
gap is 0.537 mm. Boards A and C were correct.
Parts:
- removed C607, C623: 10uF X5R, Capacitor_SMD:C_0603_1608Metric, symbol Device:C
- removed C611, C612, C627, C628: 18pF, Capacitor_SMD:C_0603_1608Metric, symbol Device:C
- removed C615, C631: 100nF 2kV, Capacitor_SMD:C_0603_1608Metric, symbol Device:C
- removed C700, C701, C702, C703, C704, C705, C706, C707, C720, C721, C722, C723, C724, C725, C726, C727: 100nF, Capacitor_SMD:C_0402_1005Metric, symbol Device:C
- removed J40, J41: HR911130A, dogrudan-sdr:RJ45_Hanrun_HR911130A, symbol dogrudan-sdr:HR911130A
- removed L606, L622: 4.7uH, Inductor_SMD:L_0805_2012Metric, symbol Device:L
- removed R600, R601, R602, R603, R604, R605, R616, R617, R618, R619, R620, R621: 1k, Resistor_SMD:R_0603_1608Metric, symbol Device:R
- removed R608, R624: 2.2k 1%, Resistor_SMD:R_0603_1608Metric, symbol Device:R
- removed R609, R625: 10k, Resistor_SMD:R_0603_1608Metric, symbol Device:R
- removed R613, R614, R629, R630: 330R, Resistor_SMD:R_0603_1608Metric, symbol Device:R
- removed R690: 1.5k, Resistor_SMD:R_0603_1608Metric, symbol Device:R
- removed R691, R692: 0R, Resistor_SMD:R_0603_1608Metric, symbol Device:R
- removed U10: LFE5U-25F-7BG256I, Package_BGA:BGA-256_14.0x14.0mm_Layout16x16_P0.8mm_Ball0.45mm_Pad0.32mm_NSMD, symbol dogrudan-sdr:ECP5-BGA256
- removed U40, U41: RTL8211FI-CG, Package_DFN_QFN:QFN-40-1EP_5x5mm_P0.4mm_EP3.6x3.6mm_ThermalVias, symbol dogrudan-sdr:RTL8211F
- removed Y610, Y626: 25MHz CL12pF, Crystal:Crystal_SMD_3225-4Pin_3.2x2.5mm, symbol Device:Crystal_GND24
Connections:
- no-connect marks 2 -> 0
Other:
- note added: "Ethernet x2 RTL8211F x2 + HR911105A x2, banka 3 Baglantilar: ../NETLIST.md"
- note removed: "** PARCA DEGISTI: HR911105A -> HR911130A ** (veri sayfasi geldi) Veri sayfasi geldi ve HR911105A'nin kapaginda 'for 10/100Base-T NIC Applications' yaziyor. Semasinda SADECE IKI cift sargi var (TD, RD); gigabit DORT cift ister. O parcayla iki GbE portu 100 Mbit'e duserdi — aletin veri borusu on kat daralirdi, 4 kanal IQ akisi imkansiz. HR911130A ayni ailenin gigabit uyesi: LCSC C54408, $1.58, 6005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"
- note removed: "AYRISTIRMA — PHY basina"
- note removed: "Asagi cekilen strap'ler GND_STRAP uzerinden 0R ile toprakta. Tek noktadan ayrilabiliyor: adres catismasi cikarsa direnc sokulup baska kombinasyon denenir."
- note removed: "BANKA 3: 24 RGMII + 2 reset + 2 kesme + MDC/MDIO = 30/32. Iki pin bos — bu kartta tek marj burasi. VCCIO3 = +1V8, PHY'nin DVDD_RG'siyle ayni. UZUNLUK ESLEME: TXC ile TXD[3:0]+TXCTL grubu +-5 mm; RXC ile RXD grubu ayni. Gruplar ARASI esleme gerekmiyor — RGMII kaynak-senkron, her yon kendi saatini tasiyor. TXC/RXC saat-yetenekli pine dusmeli, liste Lattice pinout'undan yeniden siralanacak."
- note removed: "Cip basina: AVDD33 (11, 40) ve DVDD33 (29) -> 3 x 100nF @+3V3 AVDD10 (3, 8, 38) ve DVDD10 (21) -> 4 x 100nF @PHYn_1V0 DVDD_RG (28) -> 1 x 100nF @+1V8 Artı REG_OUT cikisindaki 10uF X5R (yukarida). ** Y5V KULLANMA ** — datasheet s.46-53."
- note removed: "ETHERNET x2 — RTL8211FI-CG, RGMII, banka 3"
- note removed: "FPGA BANKA 3 — RGMII x2"
- note removed: "Iki bagimsiz gigabit arayuz. Sahada tek kablo yeterli; labda biri ham IQ akisi, digeri kontrol/telemetri — akislar birbirinin gecikmesini bozmuyor."
- note removed: "MDC ve MDIO iki PHY'da ORTAK. Adresler strap ile ayrilmis: PHY-1 = 0, PHY-2 = 1. MDIO acik drenaj, 1.5k ile 1.8 V'a cekiliyor. Cekme direnci DVDD_RG seviyesinde olmali (1.8 V), 3.3 V DEGIL."
- note removed: "MDIO ORTAK YOL"
- note removed: "REG_OUT BOBINI — datasheet s.46-53 PHY'nin dahili anahtarlamali regulatoru 1.0 V rayini kendi uretiyor; bobin ve cikis kondansatoru DISARIDA. 4.7uH + 10uF X5R. ** Y5V KULLANMA ** — datasheet dalgalanma olcumlerinde acikca uyariyor; Y5V'nin DC bias altinda kapasitesi cokuyor."
- note removed: "SAAT: PHY BASINA AYRI KRISTAL 25 MHz X322525MOB4SI, LCSC C9006. Iki PHY'a tek kristal paylastirmak denenmedi — her PHY'nin kendi osilator devresi var, paylasim yuk kapasitesini bozar. 5 kurusluk parca icin risk alinmiyor. CLKOUT (35) bosta."
- note removed: "SASE BAGI — RJ45 kalkani ve orta uc dugumu CHASSIS'te; CHASSIS topraga TEK NOKTADAN, R692 (0R) ile bagli. Montaj delikleri bu kartta KAPLAMASIZ: sase referansi C kartinda, orada anten konnektorlerinin dibindeki delik kaplamali ve GND'de. Iki karttan da kasaya baglanirsa toprak dongusu olusur."
- note removed: "STRAP DIRENCLERI 1k (NETLIST.md §5.2) Bu alti bacak hem RGMII verisi hem reset anindaki strap. TXDLY / RXDLY yukari -> 2 ns ic gecikmeyi PHY uretiyor, FPGA tarafinda gecikme kurmaya gerek yok PHYAD0 PHY-2'de yukari -> adresler 0 ve 1 PLLOFF asagi -> ALDPS'te PLL acik kalsin 1k: RGMII sinyal butunlugunu bozmayacak kadar yuksek, strap'i belirleyecek kadar dusuk. 100R olsa surucuyu yorardi, 10k olsa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"

Commit message: Correct the schematic faults that ERC cannot find
An agent examined the three schematics against the datasheets. ERC
reported zero violations before and after this work. None of these
faults are visible to ERC.

The comparator for the external 10 MHz reference was in shutdown. The
SHDN pin of the TLV3501 went to +3V3. Sixteen DRV8833 devices had VCP
and VINT unconnected. Without the charge pump none of the 28 filter
relays can latch. Seven regulators had no decoupling capacitor within
18 mm to 94 mm. On board D the nearest +12V capacitor to an LM358 was
227 mm away on a 275 mm board.

The PE4312 devices had no series 10k resistor on pin 3. The datasheet
makes this necessary for the attenuation accuracy. Their exposed pad
was 2.6 mm against 2.15 mm. The BOM did not give the load capacitance
of the crystal. This work added 60 parts and changed 4 footprints.

The worst fault was in the tool chain. lib/gen_symbols.py still made
the old pin numbers. The five corrections went into the symbol
library by hand and not into its generator. A new library would have
removed all of them.

The thermal vias are now a decision from the measured clearance and
the dissipation. This work removed them from the PE4312, the RTL8211F
and the ADCLK846. They stay on the DRV8833 and on the LM5164, which
is a 1 W buck converter.

Two checks are new. sema_denetim compares the pin names with the
nets. netlist_denetim locks 22 pin-to-net expectations from the
datasheets and does not need a board.

The boards were built again with these corrections. The chain now
adds the test points: 10 on board A, 7 on board C and 15 on board D.
Each board has 3 fiducials. Every pad has a net.
Parts:
- added C607, C623: 10uF X5R, Capacitor_SMD:C_0603_1608Metric, symbol Device:C
- added C611, C612, C627, C628: 18pF, Capacitor_SMD:C_0603_1608Metric, symbol Device:C
- added C615, C631: 100nF 2kV, Capacitor_SMD:C_0603_1608Metric, symbol Device:C
- added C700, C701, C702, C703, C704, C705, C706, C707, C720, C721, C722, C723, C724, C725, C726, C727: 100nF, Capacitor_SMD:C_0402_1005Metric, symbol Device:C
- added J40, J41: HR911130A, dogrudan-sdr:RJ45_Hanrun_HR911130A, symbol dogrudan-sdr:HR911130A
- added L606, L622: 4.7uH, Inductor_SMD:L_0805_2012Metric, symbol Device:L
- added R600, R601, R602, R603, R604, R605, R616, R617, R618, R619, R620, R621: 1k, Resistor_SMD:R_0603_1608Metric, symbol Device:R
- added R608, R624: 2.2k 1%, Resistor_SMD:R_0603_1608Metric, symbol Device:R
- added R609, R625: 10k, Resistor_SMD:R_0603_1608Metric, symbol Device:R
- added R613, R614, R629, R630: 330R, Resistor_SMD:R_0603_1608Metric, symbol Device:R
- added R690: 1.5k, Resistor_SMD:R_0603_1608Metric, symbol Device:R
- added R691, R692: 0R, Resistor_SMD:R_0603_1608Metric, symbol Device:R
- added U10: LFE5U-25F-7BG256I, Package_BGA:BGA-256_14.0x14.0mm_Layout16x16_P0.8mm_Ball0.45mm_Pad0.32mm_NSMD, symbol dogrudan-sdr:ECP5-BGA256
- added U40, U41: RTL8211FI-CG, Package_DFN_QFN:QFN-40-1EP_5x5mm_P0.4mm_EP3.6x3.6mm, symbol dogrudan-sdr:RTL8211F
- added Y610, Y626: 25MHz CL12pF, Crystal:Crystal_SMD_3225-4Pin_3.2x2.5mm, symbol Device:Crystal_GND24
Connections:
- new net +1V8: C707.1, C727.1, R602.1, R603.1, R616.1, R618.1, R619.1, R690.1, U10.K11 (VCCIO3_1), U10.L11 (VCCIO3_2), U40.28 (DVDD_RG), U41.28 (DVDD_RG)
- new net +3V3: C700.1, C701.1, C702.1, C720.1, C721.1, C722.1, R609.1, R613.1, R614.1, R625.1, R629.1, R630.1, U40.11 (AVDD33), U40.29 (DVDD33), U40.40 (AVDD33), U41.11 (AVDD33), U41.29 (DVDD33), U41.40 (AVDD33)
- new net CHASSIS: C615.2, C631.2, J40.10 (CHS), J40.SH1 (SHIELD), J40.SH2 (SHIELD), J40.SH3 (SHIELD), J40.SH4 (SHIELD), J41.10 (CHS), J41.SH1 (SHIELD), J41.SH2 (SHIELD), J41.SH3 (SHIELD), J41.SH4 (SHIELD), R692.1
- new net GND: C607.2, C611.2, C612.2, C623.2, C627.2, C628.2, C700.2, C701.2, C702.2, C703.2, C704.2, C705.2, C706.2, C707.2, C720.2, C721.2, C722.2, C723.2, C724.2, C725.2, C726.2, C727.2, R608.2, R624.2, R691.2, R692.2, U40.41 (GND), U41.41 (GND), Y610.2 (G), Y610.4 (G), Y626.2 (G), Y626.4 (G)
- new net GND_STRAP: R600.2, R601.2, R604.2, R605.2, R617.2, R620.2, R621.2, R691.1
- new net LED_DATA: U10.T15 (PR38D)
- new net LED_TX: U10.T14 (PR41D)
- new net MDC: U10.R16 (PR35B), U40.13 (MDC), U41.13 (MDC)
- new net MDIO: R690.2, U10.T13 (PR44B), U40.14 (MDIO), U41.14 (MDIO)
- new net PHY1_1V0: C607.1, C703.1, C704.1, C705.1, C706.1, L606.2, U40.21 (DVDD10), U40.3 (AVDD10), U40.38 (AVDD10), U40.8 (AVDD10)
- new net PHY1_CFGEXT: R609.2, U40.32 (LED0/CFG_EXT)
- new net PHY1_CT: C615.1, J40.1 (CT_COM)
- new net PHY1_LED1: J40.12 (LEDG_K), U40.33 (LED1/CFG_LDO0)
- new net PHY1_LED1_A: J40.11 (LEDG_A), R613.2
- new net PHY1_LED2: J40.13 (LEDY_K), U40.34 (LED2/CFG_LDO1)
- new net PHY1_LED2_A: J40.14 (LEDY_A), R614.2
- new net PHY1_MDI0N: J40.3 (MDI0-), U40.2 (MDIN0)
- new net PHY1_MDI0P: J40.2 (MDI0+), U40.1 (MDIP0)
- new net PHY1_MDI1N: J40.7 (MDI1-), U40.5 (MDIN1)
- new net PHY1_MDI1P: J40.4 (MDI1+), U40.4 (MDIP1)
- new net PHY1_MDI2N: J40.6 (MDI2-), U40.7 (MDIN2)
- new net PHY1_MDI2P: J40.5 (MDI2+), U40.6 (MDIP2)
- new net PHY1_MDI3N: J40.9 (MDI3-), U40.10 (MDIN3)
- new net PHY1_MDI3P: J40.8 (MDI3+), U40.9 (MDIP3)
- new net PHY1_REGOUT: L606.1, U40.30 (REG_OUT)
- new net PHY1_RSET: R608.1, U40.39 (RSET)
- new net PHY1_RXC: R605.1, U10.L16 (PR26A), U40.27 (RXC/PHYAD1)
- new net PHY1_RXCTL: R604.1, U10.K12 (PR29B), U40.26 (RXCTL/PHYAD2)
- new net PHY1_RXD0: R603.2, U10.K13 (PR29A), U40.25 (RXD0/RXDLY)
- new net PHY1_RXD1: R602.2, U10.M13 (PR35C), U40.24 (RXD1/TXDLY)
- new net PHY1_RXD2: R601.1, U10.M14 (PR32D), U40.23 (RXD2/PLLOFF)
- new net PHY1_RXD3: R600.1, U10.N16 (PR32A), U40.22 (RXD3/PHYAD0)
- new net PHY1_TXC: U10.L15 (PR26B), U40.20 (TXC)
- new net PHY1_TXCTL: U10.M12 (PR44C), U40.19 (TXCTL)
- new net PHY1_TXD0: U10.L12 (PR29D), U40.18 (TXD0)
- new net PHY1_TXD1: U10.L13 (PR29C), U40.17 (TXD1)
- new net PHY1_TXD2: U10.L14 (PR32C), U40.16 (TXD2)
- new net PHY1_TXD3: U10.M11 (PR47A), U40.15 (TXD3)
- new net PHY1_XI: C611.1, U40.36 (XTAL_IN), Y610.1
- new net PHY1_XO: C612.1, U40.37 (XTAL_OUT/EXT_CLK), Y610.3
- new net PHY1_nINT: U10.R14 (PR41B), U40.31 (~{INTB}/~{PMEB})
- new net PHY1_nRST: U10.R12 (PR44A), U40.12 (~{PHYRSTB})
- new net PHY2_1V0: C623.1, C723.1, C724.1, C725.1, C726.1, L622.2, U41.21 (DVDD10), U41.3 (AVDD10), U41.38 (AVDD10), U41.8 (AVDD10)
- new net PHY2_CFGEXT: R625.2, U41.32 (LED0/CFG_EXT)
- new net PHY2_CT: C631.1, J41.1 (CT_COM)
- new net PHY2_LED1: J41.12 (LEDG_K), U41.33 (LED1/CFG_LDO0)
- new net PHY2_LED1_A: J41.11 (LEDG_A), R629.2
- new net PHY2_LED2: J41.13 (LEDY_K), U41.34 (LED2/CFG_LDO1)
- new net PHY2_LED2_A: J41.14 (LEDY_A), R630.2
- new net PHY2_MDI0N: J41.3 (MDI0-), U41.2 (MDIN0)
- new net PHY2_MDI0P: J41.2 (MDI0+), U41.1 (MDIP0)
- new net PHY2_MDI1N: J41.7 (MDI1-), U41.5 (MDIN1)
- new net PHY2_MDI1P: J41.4 (MDI1+), U41.4 (MDIP1)
- new net PHY2_MDI2N: J41.6 (MDI2-), U41.7 (MDIN2)
- new net PHY2_MDI2P: J41.5 (MDI2+), U41.6 (MDIP2)
- new net PHY2_MDI3N: J41.9 (MDI3-), U41.10 (MDIN3)
- new net PHY2_MDI3P: J41.8 (MDI3+), U41.9 (MDIP3)
- new net PHY2_REGOUT: L622.1, U41.30 (REG_OUT)
- new net PHY2_RSET: R624.1, U41.39 (RSET)
- new net PHY2_RXC: R621.1, U10.M16 (PR26C), U41.27 (RXC/PHYAD1)
- new net PHY2_RXCTL: R620.1, U10.P16 (PR35A), U41.26 (RXCTL/PHYAD2)
- new net PHY2_RXD0: R619.2, U10.P15 (PR32B), U41.25 (RXD0/RXDLY)
- new net PHY2_RXD1: R618.2, U10.P14 (PR38B), U41.24 (RXD1/TXDLY)
- new net PHY2_RXD2: R617.1, U10.N14 (PR35D), U41.23 (RXD2/PLLOFF)
- new net PHY2_RXD3: R616.2, U10.P13 (PR41A), U41.22 (RXD3/PHYAD0)
- new net PHY2_TXC: U10.M15 (PR26D), U41.20 (TXC)
- new net PHY2_TXCTL: U10.N13 (PR38A), U41.19 (TXCTL)
- new net PHY2_TXD0: U10.P12 (PR47D), U41.18 (TXD0)
- new net PHY2_TXD1: U10.N12 (PR44D), U41.17 (TXD1)
- new net PHY2_TXD2: U10.P11 (PR47C), U41.16 (TXD2)
- new net PHY2_TXD3: U10.N11 (PR47B), U41.15 (TXD3)
- new net PHY2_XI: C627.1, U41.36 (XTAL_IN), Y626.1
- new net PHY2_XO: C628.1, U41.37 (XTAL_OUT/EXT_CLK), Y626.3
- new net PHY2_nINT: U10.R15 (PR38C), U41.31 (~{INTB}/~{PMEB})
- new net PHY2_nRST: U10.R13 (PR41C), U41.12 (~{PHYRSTB})
- no-connect marks 0 -> 2
Other:
- note added: "** PARCA DEGISTI: HR911105A -> HR911130A ** (veri sayfasi geldi) Veri sayfasi geldi ve HR911105A'nin kapaginda 'for 10/100Base-T NIC Applications' yaziyor. Semasinda SADECE IKI cift sargi var (TD, RD); gigabit DORT cift ister. O parcayla iki GbE portu 100 Mbit'e duserdi — aletin veri borusu on kat daralirdi, 4 kanal IQ akisi imkansiz. HR911130A ayni ailenin gigabit uyesi: LCSC C54408, $1.58, 6005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"
- note added: "AYRISTIRMA — PHY basina"
- note added: "Asagi cekilen strap'ler GND_STRAP uzerinden 0R ile toprakta. Tek noktadan ayrilabiliyor: adres catismasi cikarsa direnc sokulup baska kombinasyon denenir."
- note added: "BANKA 3: 24 RGMII + 2 reset + 2 kesme + MDC/MDIO = 30/32. Iki pin bos — bu kartta tek marj burasi. VCCIO3 = +1V8, PHY'nin DVDD_RG'siyle ayni. UZUNLUK ESLEME: TXC ile TXD[3:0]+TXCTL grubu +-5 mm; RXC ile RXD grubu ayni. Gruplar ARASI esleme gerekmiyor — RGMII kaynak-senkron, her yon kendi saatini tasiyor. TXC/RXC saat-yetenekli pine dusmeli, liste Lattice pinout'undan yeniden siralanacak."
- note added: "Cip basina: AVDD33 (11, 40) ve DVDD33 (29) -> 3 x 100nF @+3V3 AVDD10 (3, 8, 38) ve DVDD10 (21) -> 4 x 100nF @PHYn_1V0 DVDD_RG (28) -> 1 x 100nF @+1V8 Artı REG_OUT cikisindaki 10uF X5R (yukarida). ** Y5V KULLANMA ** — datasheet s.46-53."
- note added: "ETHERNET x2 — RTL8211FI-CG, RGMII, banka 3"
- note added: "FPGA BANKA 3 — RGMII x2"
- note added: "Iki bagimsiz gigabit arayuz. Sahada tek kablo yeterli; labda biri ham IQ akisi, digeri kontrol/telemetri — akislar birbirinin gecikmesini bozmuyor."
- note added: "MDC ve MDIO iki PHY'da ORTAK. Adresler strap ile ayrilmis: PHY-1 = 0, PHY-2 = 1. MDIO acik drenaj, 1.5k ile 1.8 V'a cekiliyor. Cekme direnci DVDD_RG seviyesinde olmali (1.8 V), 3.3 V DEGIL."
- note added: "MDIO ORTAK YOL"
- note added: "REG_OUT BOBINI — datasheet s.46-53 PHY'nin dahili anahtarlamali regulatoru 1.0 V rayini kendi uretiyor; bobin ve cikis kondansatoru DISARIDA. 4.7uH + 10uF X5R. ** Y5V KULLANMA ** — datasheet dalgalanma olcumlerinde acikca uyariyor; Y5V'nin DC bias altinda kapasitesi cokuyor."
- note added: "SAAT: PHY BASINA AYRI KRISTAL 25 MHz X322525MOB4SI, LCSC C9006. Iki PHY'a tek kristal paylastirmak denenmedi — her PHY'nin kendi osilator devresi var, paylasim yuk kapasitesini bozar. 5 kurusluk parca icin risk alinmiyor. CLKOUT (35) bosta."
- note added: "SASE BAGI — RJ45 kalkani ve orta uc dugumu CHASSIS'te; CHASSIS topraga TEK NOKTADAN, R692 (0R) ile bagli. Montaj delikleri bu kartta KAPLAMASIZ: sase referansi C kartinda, orada anten konnektorlerinin dibindeki delik kaplamali ve GND'de. Iki karttan da kasaya baglanirsa toprak dongusu olusur."
- note added: "STRAP DIRENCLERI 1k (NETLIST.md §5.2) Bu alti bacak hem RGMII verisi hem reset anindaki strap. TXDLY / RXDLY yukari -> 2 ns ic gecikmeyi PHY uretiyor, FPGA tarafinda gecikme kurmaya gerek yok PHYAD0 PHY-2'de yukari -> adresler 0 ve 1 PLLOFF asagi -> ALDPS'te PLL acik kalsin 1k: RGMII sinyal butunlugunu bozmayacak kadar yuksek, strap'i belirleyecek kadar dusuk. 100R olsa surucuyu yorardi, 10k olsa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"
- note removed: "Ethernet x2 RTL8211F x2 + HR911105A x2, banka 3 Baglantilar: ../NETLIST.md"
