File: hardware/kicad/A_main/01_power.kicad_sch (KiCad schematic)
At the start: 42 parts, among them J1 XT60, Q1 DMP3098L, U1 TPS62130, U2 TPS62130, U3 TPS7A2018, U4 ADP150-1.8, U5 ADP150-1.8, U6 ADP150-3.3, U7 ADP150-3.3, U8 ADP150-2.5, U9 ADP150-1.8

Commit message: Name the copyright holder and stamp it into the generated files
The repository had three licence files and no statement of who owns
the work. The only record of authorship was the git author field.

Copyleft depends on that statement. GPL and CERN-OHL-S work because
the holder grants permission on condition of reciprocity; with no
holder named there is nobody to require it from a downstream user.
Naming the author keeps the design open rather than closing it.

kicad/telif.py is the single source. The line reaches the schematics
through their title block and not through the generators, because
every schematic file is rewritten on each build and a header placed in
a generator would disappear at the first regeneration. All 23
schematics carry it. 109 source files have SPDX headers, split by the
project's own table: generators and the layout chain are hardware
under CERN-OHL-S-2.0, HDL and the audit tools are software under
GPL-3.0-only.

Board C's inductors also move to footprints that match parts that can
be bought. All of them sat on 0805 pads. Of the values this design
needs, 33 to 220 nH are 0603 parts, 470 and 820 nH are 0805, and
everything from 1000 nH upward is 1210, which is 3.2 by 2.5 mm and
does not fit an 0805 land. 32 inductors could not have been soldered.

A symbol-against-footprint check cannot find this. Those two agreed
with each other; what was wrong was the body size of the real part
behind the footprint.
Parts:
- removed U6, U7: ADP150-3.3, Package_TO_SOT_SMD:TSOT-23-5, symbol dogrudan-sdr:ADP150
- added FB6, FB7: ferrit 600R, Inductor_SMD:L_0603_1608Metric, symbol Device:L
- C18, C20: value 1uF -> 10uF
- C19, C21: value 1uF -> 100nF
Connections:
- net +3V3: now also FB6.1, FB7.1; no longer C18.1, C20.1
- net +3V3_A: now also C20.1, FB7.2
- net +3V3_CLK: now also C18.1, FB6.2
- no-connect marks 9 -> 7
Other:
- note added: "DAC AVDD FERRIT, LDO DEGIL"
- note added: "FB6 (+3V3_CLK) VCXO zincirinin beslemesi, FB7 (+3V3_A) DAC AVDD. Once LDO'ydular: giris +3V3, cikis 3.3 V — bir regulator kendi giris gerilimini uretemez. Ferrit + 10 uF, 2.5 MHz'te ayni bastirmayi veriyor. Besleme gurultusu DOGRUDAN faz gurultusune donusuyor — manset spec burada."
- note added: "GIRIS VE KORUMA — NETLIST.md §9 9-17 V aku ya da tezgah kaynagi. Ters polarite sahada bir kere olur, yeter. UST SINIR 18 DEGIL 17 V. TPS62130 veri sayfasi (SLVSBC3F) tablo 7.3: onerilen calisma araligi 3-17 V; mutlak azami 20 V. 18 V yazan bir tasarimda parca veri sayfasi disinda kosuyor ve TVS de tutmuyor — SMBJ20A 20 V'ta bloke, yani 18 V'u kirpmiyor. 4S lipo (16.8 V dolu) sinirin altinda kaliy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"
- note added: "VCXO zinciri FERRIT, LDO DEGIL"
- note removed: "DAC AVDD"
- note removed: "GIRIS VE KORUMA — NETLIST.md §9 9-18 V aku ya da tezgah kaynagi. Ters polarite sahada bir kere olur, yeter."
- note removed: "U6 (+3V3_CLK) VCXO'nun TEK beslemesi. Ferrit boncuk, ayri toprak adasi. Besleme gurultusu DOGRUDAN faz gurultusune donusuyor — manset spec burada."
- note removed: "VCXO — TEK besleme, FERRIT"
